File: unused.kicad_sch (KiCad schematic)
At the start: 2 parts, among them U19 SN74ALS04 (КР1533ЛН1), U40 IN74ALS00N (КР1533ЛА3)

Commit message: 20 march version
Added 2nd list, working on the third
Parts:
- removed unit 2 of U19
- removed U40: IN74ALS00N (КР1533ЛА3), Package_DIP:DIP-14_W7.62mm_Socket_LongPads, symbol 74xx:74LS00
Connections:
- no-connect marks 13 -> 8
Changed lines of the file:
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@@
   (no_connect (at 46.99 76.835))
   (no_connect (at 46.99 62.865))
-  (no_connect (at 57.15 29.21))
-  (no_connect (at 72.39 31.75))
   (no_connect (at 72.39 47.625))
   (no_connect (at 72.39 62.865))
-  (no_connect (at 46.99 47.625))
   (no_connect (at 31.75 62.865))
   (no_connect (at 57.15 62.865))
   (no_connect (at 57.15 47.625))
-  (no_connect (at 31.75 47.625))
   (no_connect (at 31.75 76.835))
-  (no_connect (at 57.15 34.29))
   (symbol (lib_id "74xx:74LS04") (at 64.77 47.625 0) (unit 3)
     (in_bom yes) (on_board yes)
@@
       (effects (font (size 1.27 1.27)) hide)
     )
-    (pin "1")
-    (pin "2")
-    (pin "3")
-    (pin "4")
-    (pin "5")
-    (pin "6")
-    (pin "8")
-    (pin "9")
-    (pin "10")
-    (pin "11")
-    (pin "12")
-    (pin "13")
-    (pin "14")
-    (pin "7")
-  )
-  (symbol (lib_id "74xx:74LS00") (at 64.77 31.75 0) (unit 2)
-    (in_bom yes) (on_board yes)
-    (property "Reference" "U40" (id 0) (at 64.77 31.75 0))
-    (property "Value" "IN74ALS00N (КР1533ЛА3)" (id 1) (at 64.77 24.765 0))
-    (property "Footprint" "Package_DIP:DIP-14_W7.62mm_Socket_LongPads" (id 2) (at 64.77 31.75 0)
-      (effects (font (size 1.27 1.27)) hide)
-    )
-    (property "Datasheet" "http://www.ti.com/lit/gpn/sn74ls00" (id 3) (at 64.77 31.75 0)
-      (effects (font (size 1.27 1.27)) hide)
-    )
-    (pin "1")
-    (pin "2")
-    (pin "3")
-    (pin "4")
-    (pin "5")
-    (pin "6")
-    (pin "10")
-    (pin "8")
-    (pin "9")
-    (pin "11")
-    (pin "12")
-    (pin "13")
-    (pin "14")
-    (pin "7")
-  )
-  (symbol (lib_id "74xx:74LS04") (at 39.37 47.625 0) (unit 2)
-    (in_bom yes) (on_board yes)
-    (property "Reference" "U19" (id 0) (at 38.735 47.625 0))
-    (property "Value" "SN74ALS04 (КР1533ЛН1)" (id 1) (at 39.37 41.275 0))
-    (property "Footprint" "Package_DIP:DIP-14_W7.62mm_Socket_LongPads" (id 2) (at 39.37 47.625 0)
-      (effects (font (size 1.27 1.27)) hide)
-    )
-    (property "Datasheet" "http://www.ti.com/lit/gpn/sn74LS04" (id 3) (at 39.37 47.625 0)
-      (effects (font (size 1.27 1.27)) hide)
-    )

Commit message: March 21st update
Parts:
- removed unit 3 of U19
- removed unit 5 of U19
Connections:
- no-connect marks 8 -> 4
Changed lines of the file:
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@@
   (no_connect (at 46.99 76.835))
   (no_connect (at 46.99 62.865))
-  (no_connect (at 72.39 47.625))
-  (no_connect (at 72.39 62.865))
   (no_connect (at 31.75 62.865))
-  (no_connect (at 57.15 62.865))
-  (no_connect (at 57.15 47.625))
   (no_connect (at 31.75 76.835))
-  (symbol (lib_id "74xx:74LS04") (at 64.77 47.625 0) (unit 3)
-    (in_bom yes) (on_board yes)
-    (property "Reference" "U19" (id 0) (at 64.135 47.625 0))
-    (property "Value" "SN74ALS04 (КР1533ЛН1)" (id 1) (at 64.77 41.275 0))
-    (property "Footprint" "Package_DIP:DIP-14_W7.62mm_Socket_LongPads" (id 2) (at 64.77 47.625 0)
-      (effects (font (size 1.27 1.27)) hide)
-    )
-    (property "Datasheet" "http://www.ti.com/lit/gpn/sn74LS04" (id 3) (at 64.77 47.625 0)
-      (effects (font (size 1.27 1.27)) hide)
-    )
-    (pin "1")
-    (pin "2")
-    (pin "3")
-    (pin "4")
-    (pin "5")
-    (pin "6")
-    (pin "8")
-    (pin "9")
-    (pin "10")
-    (pin "11")
-    (pin "12")
-    (pin "13")
-    (pin "14")
-    (pin "7")
-  )
   (symbol (lib_id "74xx:74LS04") (at 39.37 76.835 0) (unit 6)
     (in_bom yes) (on_board yes)
@@
       (effects (font (size 1.27 1.27)) hide)
     )
-    (pin "1")
-    (pin "2")
-    (pin "3")
-    (pin "4")
-    (pin "5")
-    (pin "6")
-    (pin "8")
-    (pin "9")
-    (pin "10")
-    (pin "11")
-    (pin "12")
-    (pin "13")
-    (pin "14")
-    (pin "7")
-  )
-  (symbol (lib_id "74xx:74LS04") (at 64.77 62.865 0) (unit 5)
-    (in_bom yes) (on_board yes)
-    (property "Reference" "U19" (id 0) (at 64.135 62.865 0))
-    (property "Value" "SN74ALS04 (КР1533ЛН1)" (id 1) (at 64.77 56.515 0))
-    (property "Footprint" "Package_DIP:DIP-14_W7.62mm_Socket_LongPads" (id 2) (at 64.77 62.865 0)
-      (effects (font (size 1.27 1.27)) hide)
-    )
-    (property "Datasheet" "http://www.ti.com/lit/gpn/sn74LS04" (id 3) (at 64.77 62.865 0)
-      (effects (font (size 1.27 1.27)) hide)
-    )

Commit message: March 22nd additions
Parts:
- removed unit 6 of U19
Connections:
- no-connect marks 4 -> 2
Changed lines of the file:
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@@
     (comment 2 "Евстафьев")
   )
-  (no_connect (at 46.99 76.835))
   (no_connect (at 46.99 62.865))
   (no_connect (at 31.75 62.865))
-  (no_connect (at 31.75 76.835))
-  (symbol (lib_id "74xx:74LS04") (at 39.37 76.835 0) (unit 6)
-    (in_bom yes) (on_board yes)
-    (property "Reference" "U19" (id 0) (at 38.735 76.835 0))
-    (property "Value" "SN74ALS04 (КР1533ЛН1)" (id 1) (at 39.37 70.485 0))
-    (property "Footprint" "Package_DIP:DIP-14_W7.62mm_Socket_LongPads" (id 2) (at 39.37 76.835 0)
-      (effects (font (size 1.27 1.27)) hide)
-    )
-    (property "Datasheet" "http://www.ti.com/lit/gpn/sn74LS04" (id 3) (at 39.37 76.835 0)
-      (effects (font (size 1.27 1.27)) hide)
-    )
-    (pin "1")
-    (pin "2")
-    (pin "3")
-    (pin "4")
-    (pin "5")
-    (pin "6")
-    (pin "8")
-    (pin "9")
-    (pin "10")
-    (pin "11")
-    (pin "12")
-    (pin "13")
-    (pin "14")
-    (pin "7")
-  )
   (symbol (lib_id "74xx:74LS04") (at 39.37 62.865 0) (unit 4)
     (in_bom yes) (on_board yes)

Commit message: March 22nd update 2
Parts:
- removed U19: SN74ALS04 (КР1533ЛН1), Package_DIP:DIP-14_W7.62mm_Socket_LongPads, symbol 74xx:74LS04
Connections:
- no-connect marks 2 -> 0
Changed lines of the file:
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@@
     (comment 2 "Евстафьев")
   )
-  (no_connect (at 46.99 62.865))
-  (no_connect (at 31.75 62.865))
-  (symbol (lib_id "74xx:74LS04") (at 39.37 62.865 0) (unit 4)
-    (in_bom yes) (on_board yes)
-    (property "Reference" "U19" (id 0) (at 38.735 62.865 0))
-    (property "Value" "SN74ALS04 (КР1533ЛН1)" (id 1) (at 39.37 56.515 0))
-    (property "Footprint" "Package_DIP:DIP-14_W7.62mm_Socket_LongPads" (id 2) (at 39.37 62.865 0)
-      (effects (font (size 1.27 1.27)) hide)
-    )
-    (property "Datasheet" "http://www.ti.com/lit/gpn/sn74LS04" (id 3) (at 39.37 62.865 0)
-      (effects (font (size 1.27 1.27)) hide)
-    )
-    (pin "1")
-    (pin "2")
-    (pin "3")
-    (pin "4")
-    (pin "5")
-    (pin "6")
-    (pin "8")
-    (pin "9")
-    (pin "10")
-    (pin "11")
-    (pin "12")
-    (pin "13")
-    (pin "14")
-    (pin "7")
-  )
 )
