File: ROM.kicad_sch (KiCad schematic)
At the start: 5 parts, among them U19 SN74ALS04 (КР1533ЛН1), U70 27C64, U71 27C64, U75 IN74ALS32N (КР1533ЛЛ1)

Commit message: March 26th update
Parts:
- U19, U75: footprint Package_DIP:DIP-14_W7.62mm_Socket_LongPads -> Package_DIP:DIP-14_W7.62mm_Socket
- U70, U71: footprint Package_DIP:DIP-28_W15.24mm_Socket_LongPads -> Package_DIP:DIP-28_W15.24mm_Socket
Changed lines of the file:
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@@
     (property "Reference" "U19" (id 0) (at 149.225 163.83 0))
     (property "Value" "SN74ALS04 (КР1533ЛН1)" (id 1) (at 149.86 168.91 0))
-    (property "Footprint" "Package_DIP:DIP-14_W7.62mm_Socket_LongPads" (id 2) (at 149.86 163.83 0)
+    (property "Footprint" "Package_DIP:DIP-14_W7.62mm_Socket" (id 2) (at 149.86 163.83 0)
       (effects (font (size 1.27 1.27)) hide)
     )
@@
     (property "Reference" "U75" (id 0) (at 168.91 142.875 0))
     (property "Value" "IN74ALS32N (КР1533ЛЛ1)" (id 1) (at 168.91 135.89 0))
-    (property "Footprint" "Package_DIP:DIP-14_W7.62mm_Socket_LongPads" (id 2) (at 168.91 142.875 0)
+    (property "Footprint" "Package_DIP:DIP-14_W7.62mm_Socket" (id 2) (at 168.91 142.875 0)
       (effects (font (size 1.27 1.27)) hide)
     )
@@
       (effects (font (size 1.27 1.27)) (justify left))
     )
-    (property "Footprint" "Package_DIP:DIP-28_W15.24mm_Socket_LongPads" (id 2) (at 130.175 83.82 0)
+    (property "Footprint" "Package_DIP:DIP-28_W15.24mm_Socket" (id 2) (at 130.175 83.82 0)
       (effects (font (size 1.27 1.27)) hide)
     )
@@
       (effects (font (size 1.27 1.27)) (justify left))
     )
-    (property "Footprint" "Package_DIP:DIP-28_W15.24mm_Socket_LongPads" (id 2) (at 189.865 83.82 0)
+    (property "Footprint" "Package_DIP:DIP-28_W15.24mm_Socket" (id 2) (at 189.865 83.82 0)
       (effects (font (size 1.27 1.27)) hide)
     )
@@
     (property "Reference" "U75" (id 0) (at 177.8 158.115 0))
     (property "Value" "IN74ALS32N (КР1533ЛЛ1)" (id 1) (at 177.8 151.765 0))
-    (property "Footprint" "Package_DIP:DIP-14_W7.62mm_Socket_LongPads" (id 2) (at 177.8 158.115 0)
+    (property "Footprint" "Package_DIP:DIP-14_W7.62mm_Socket" (id 2) (at 177.8 158.115 0)
       (effects (font (size 1.27 1.27)) hide)
     )
