File: ROM.kicad_sch (KiCad schematic)
At the start: 5 parts, among them U19 SN74ALS04 (КР1533ЛН1), U70 27C64, U71 27C64, U75 IN74ALS32N (КР1533ЛЛ1)

Commit message: Version 1.0 schematics and PCB complete
Parts:
- JP2: symbol Jumper:Jumper_3_Open -> Delta_s_m_Lib:Jumper_3_Open
- U19: symbol 74xx:74LS04 -> Delta_s_m_Lib:74LS04
- U70, U71: symbol Memory_EPROM:27C128 -> Delta_s_m_Lib:27C128
- U75: symbol 74xx:74LS32 -> Delta_s_m_Lib:74LS32
Changed lines of the file:
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@@
     )
   )
-  (symbol (lib_id "74xx:74LS04") (at 149.86 163.83 0) (unit 1)
+  (symbol (lib_id "Delta_s_m_Lib:74LS04") (at 149.86 163.83 0) (unit 1)
     (in_bom yes) (on_board yes) (dnp no)
     (property "Reference" "U19" (at 149.225 163.83 0)
@@
     )
   )
-  (symbol (lib_id "74xx:74LS32") (at 168.91 142.875 0) (mirror x) (unit 1)
+  (symbol (lib_id "Delta_s_m_Lib:74LS32") (at 168.91 142.875 0) (mirror x) (unit 1)
     (in_bom yes) (on_board yes) (dnp no)
     (property "Reference" "U75" (at 168.91 142.875 0)
@@
     )
   )
-  (symbol (lib_id "Memory_EPROM:27C128") (at 130.175 83.82 0) (unit 1)
+  (symbol (lib_id "Delta_s_m_Lib:27C128") (at 130.175 83.82 0) (unit 1)
     (in_bom yes) (on_board yes) (dnp no) (fields_autoplaced)
     (property "Reference" "U70" (at 132.1944 52.705 0)
@@
     )
   )
-  (symbol (lib_id "Memory_EPROM:27C128") (at 189.865 83.82 0) (unit 1)
+  (symbol (lib_id "Delta_s_m_Lib:27C128") (at 189.865 83.82 0) (unit 1)
     (in_bom yes) (on_board yes) (dnp no) (fields_autoplaced)
     (property "Reference" "U71" (at 191.8844 52.705 0)
@@
     )
   )
-  (symbol (lib_id "74xx:74LS32") (at 177.8 158.115 0) (mirror x) (unit 4)
+  (symbol (lib_id "Delta_s_m_Lib:74LS32") (at 177.8 158.115 0) (mirror x) (unit 4)
     (in_bom yes) (on_board yes) (dnp no)
     (property "Reference" "U75" (at 177.8 158.115 0)
@@
     )
   )
-  (symbol (lib_id "Jumper:Jumper_3_Open") (at 135.89 149.225 0) (unit 1)
+  (symbol (lib_id "Delta_s_m_Lib:Jumper_3_Open") (at 135.89 149.225 0) (unit 1)
     (in_bom yes) (on_board yes) (dnp no) (fields_autoplaced)
     (property "Reference" "JP2" (at 135.89 142.875 0)

Commit message: Version 1.2 update
Parts:
- JP2: footprint Connector_PinHeader_2.54mm:PinHeader_1x03_P2.54mm_Vertical -> Delta_sm_lib:PinHeader_1x03_P2.54mm_Vertical
- U19, U75: footprint Package_DIP:DIP-14_W7.62mm_Socket -> Delta_sm_lib:DIP-14_W7.62mm_Socket
- U70, U71: footprint Package_DIP:DIP-28_W15.24mm_Socket -> Delta_sm_lib:DIP-28_W15.24mm_Socket
Changed lines of the file:
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@@
       (effects (font (size 1.27 1.27)))
     )
-    (property "Footprint" "Package_DIP:DIP-14_W7.62mm_Socket" (at 149.86 163.83 0)
+    (property "Footprint" "Delta_sm_lib:DIP-14_W7.62mm_Socket" (at 149.86 163.83 0)
       (effects (font (size 1.27 1.27)) hide)
     )
@@
       (effects (font (size 1.27 1.27)))
     )
-    (property "Footprint" "Package_DIP:DIP-14_W7.62mm_Socket" (at 168.91 142.875 0)
+    (property "Footprint" "Delta_sm_lib:DIP-14_W7.62mm_Socket" (at 168.91 142.875 0)
       (effects (font (size 1.27 1.27)) hide)
     )
@@
       (effects (font (size 1.27 1.27)) (justify left))
     )
-    (property "Footprint" "Package_DIP:DIP-28_W15.24mm_Socket" (at 130.175 83.82 0)
+    (property "Footprint" "Delta_sm_lib:DIP-28_W15.24mm_Socket" (at 130.175 83.82 0)
       (effects (font (size 1.27 1.27)) hide)
     )
@@
       (effects (font (size 1.27 1.27)) (justify left))
     )
-    (property "Footprint" "Package_DIP:DIP-28_W15.24mm_Socket" (at 189.865 83.82 0)
+    (property "Footprint" "Delta_sm_lib:DIP-28_W15.24mm_Socket" (at 189.865 83.82 0)
       (effects (font (size 1.27 1.27)) hide)
     )
@@
       (effects (font (size 1.27 1.27)))
     )
-    (property "Footprint" "Package_DIP:DIP-14_W7.62mm_Socket" (at 177.8 158.115 0)
+    (property "Footprint" "Delta_sm_lib:DIP-14_W7.62mm_Socket" (at 177.8 158.115 0)
       (effects (font (size 1.27 1.27)) hide)
     )
@@
       (effects (font (size 1.27 1.27)))
     )
-    (property "Footprint" "Connector_PinHeader_2.54mm:PinHeader_1x03_P2.54mm_Vertical" (at 135.89 149.225 0)
-      (effects (font (size 1.27 1.27)) hide)
-    )
+    (property "Footprint" "Delta_sm_lib:PinHeader_1x03_P2.54mm_Vertical" (at 135.89 149.225 0)
+      (effects (font (size 1.27 1.27)) hide)
+    )

Commit message: Update 1.2, additional pins
Parts:
- added U76: 27C256, Delta_sm_lib:DIP-28_W15.24mm_Socket, symbol Memory_EPROM:27C256
Changed lines of the file:
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@@
+    )
+  )
+  (symbol (lib_id "Memory_EPROM:27C256") (at 75.565 83.185 0) (unit 1)
+    (in_bom yes) (on_board yes) (dnp no) (fields_autoplaced)
+    (property "Reference" "U76" (at 77.5209 53.34 0)
+      (effects (font (size 1.27 1.27)) (justify left))
+    )
+    (property "Value" "27C256" (at 77.5209 55.88 0)
+      (effects (font (size 1.27 1.27)) (justify left))
+    )
+    (property "Footprint" "Delta_sm_lib:DIP-28_W15.24mm_Socket" (at 75.565 83.185 0)
+      (effects (font (size 1.27 1.27)) hide)
+    )
+    (property "Datasheet" "http://ww1.microchip.com/downloads/en/DeviceDoc/doc0014.pdf" (at 75.565 83.185 0)
+      (effects (font (size 1.27 1.27)) hide)
+    )
+    (pin "1")
+    (pin "10")
+    (pin "11")
+    (pin "12")
+    (pin "13")
+    (pin "14")
+    (pin "15")
+    (pin "16")
+    (pin "17")
+    (pin "18")
+    (pin "19")
+    (pin "2")
+    (pin "20")
+    (pin "21")
+    (pin "22")
+    (pin "23")
+    (pin "24")
+    (pin "25")
+    (pin "26")
+    (pin "27")
+    (pin "28")
+    (pin "3")
+    (pin "4")
+    (pin "5")
+    (pin "6")
+    (pin "7")
+    (pin "8")
+    (pin "9")
+    (instances
+      (project "delta48m"
+        (path "/31325de8-16cf-4c6f-92cf-6f5a8aaa6830/9648d2dd-c41a-4075-97f8-828436d6d430"
+          (reference "U76") (unit 1)
+        )
+      )
     )
   )

Commit message: Topology for version 1.2
Parts:
- removed U70: 27C64, Delta_sm_lib:DIP-28_W15.24mm_Socket, symbol Delta_s_m_Lib:27C128
- added J14: Conn_01x02, Connector_PinHeader_2.54mm:PinHeader_1x02_P2.54mm_Vertical, symbol Connector_Generic:Conn_01x02
- added R3: 4.7K, Delta_sm_lib:R_Axial_DIN0207_L6.3mm_D2.5mm_P10.16mm_Horizontal, symbol Delta_s_m_Lib:R
- added SW2: SW_SPST, Delta_sm_lib:onoffswitch, symbol Switch:SW_SPST
- renumbered U76 to U70
Connections:
- net +5V: now also U70.28 (VCC), R3.1
- net A0: now also U70.10 (A0)
- net A1: now also U70.9 (A1)
- net A10: now also U70.21 (A10)
- net A11: now also U70.23 (A11)
- net A12: now also U70.2 (A12)
- net A13: now also U70.26 (A13)
- net A2: now also U70.8 (A2)
- net A3: now also U70.7 (A3)
- net A4: now also U70.6 (A4)
- net A5: now also U70.5 (A5)
- net A6: now also U70.4 (A6)
- net A7: now also U70.3 (A7)
- net A8: now also U70.25 (A8)
- net A9: now also U70.24 (A9)
- net D0: now also U70.11 (D0)
- net D1: now also U70.12 (D1)
- net D2: now also U70.13 (D2)
- net D3: now also U70.15 (D3)
- net D4: now also U70.16 (D4)
- net D5: now also U70.17 (D5)
- net D6: now also U70.18 (D6)
- net D7: now also U70.19 (D7)
- net GND: now also U70.14 (GND), J14.1 (Pin_1), SW2.2 (B)
- net OE0L: now also U70.22 (~{OE})
- net ЧТПЗУL: now also U70.20 (~{CE})
- net Extra_A14: now reaches U70.27 (A14)
- net Extra_A14: now also J14.2 (Pin_2), R3.2, SW2.1 (A)
- no-connect marks 4 -> 3
Other:
- moved on the sheet: U70
