File: cpu.kicad_sch (KiCad schematic)
At the start: 1 part, among them U69 Z80CPU

Commit message: March 22nd - 3rd edition
List 3 is complete
Other:
- title: (none) -> Центральный процессор
Changed lines of the file:
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@@
   (paper "A4")
   (title_block
+    (title "Центральный процессор")
     (comment 2 "Евстафьев")
   )

Commit message: March 24th - First Edition of PCB
Parts:
- U69: footprint Package_DIP:DIP-40_W25.4mm_Socket_LongPads -> Package_DIP:DIP-40_W15.24mm_Socket_LongPads
Changed lines of the file:
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@@
       (effects (font (size 1.27 1.27)) (justify left))
     )
-    (property "Footprint" "Package_DIP:DIP-40_W25.4mm_Socket_LongPads" (id 2) (at 144.145 75.565 0)
+    (property "Footprint" "Package_DIP:DIP-40_W15.24mm_Socket_LongPads" (id 2) (at 144.145 75.565 0)
       (effects (font (size 1.27 1.27)) hide)
     )

Commit message: March 26th update
Parts:
- U69: footprint Package_DIP:DIP-40_W15.24mm_Socket_LongPads -> Package_DIP:DIP-40_W15.24mm_Socket
Changed lines of the file:
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@@
       (effects (font (size 1.27 1.27)) (justify left))
     )
-    (property "Footprint" "Package_DIP:DIP-40_W15.24mm_Socket_LongPads" (id 2) (at 144.145 75.565 0)
+    (property "Footprint" "Package_DIP:DIP-40_W15.24mm_Socket" (id 2) (at 144.145 75.565 0)
       (effects (font (size 1.27 1.27)) hide)
     )
