File: cpu.kicad_sch (KiCad schematic)
At the start: 1 part, among them U69 Z80CPU

Commit message: Version 1.0 schematics and PCB complete
Parts:
- U69: symbol CPU:Z80CPU -> Delta_s_m_Lib:Z80CPU
Changed lines of the file:
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@@
     )
   )
-  (symbol (lib_id "CPU:Z80CPU") (at 144.145 85.725 0) (unit 1)
+  (symbol (lib_id "Delta_s_m_Lib:Z80CPU") (at 144.145 85.725 0) (unit 1)
     (in_bom yes) (on_board yes) (dnp no) (fields_autoplaced)
     (property "Reference" "U69" (at 146.1644 46.355 0)

Commit message: Version 1.2 update
Parts:
- U69: footprint Package_DIP:DIP-40_W15.24mm_Socket -> Delta_sm_lib:DIP-40_W15.24mm_Socket
Changed lines of the file:
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@@
       (effects (font (size 1.27 1.27)) (justify left))
     )
-    (property "Footprint" "Package_DIP:DIP-40_W15.24mm_Socket" (at 144.145 75.565 0)
+    (property "Footprint" "Delta_sm_lib:DIP-40_W15.24mm_Socket" (at 144.145 75.565 0)
       (effects (font (size 1.27 1.27)) hide)
     )
