File: ramd31d38.kicad_sch (KiCad schematic)
At the start: 18 parts, among them U22 74LS257 (КР1533КП11А), U25 74LS257 (КР1533КП11А), U31 RU5D1, U32 RU5D1, U33 RU5D1, U34 RU5D1, U35 RU5D1, U36 RU5D1, U37 RU5D1, U38 RU5D1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

Commit message: March 22nd - 3rd edition
List 3 is complete
Parts:
- gave numbers to parts that had none: 1
Changed lines of the file:
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@@
   (symbol (lib_id "Jumper:Jumper_3_Bridged12") (at 35.56 113.03 90) (mirror x) (unit 1)
     (in_bom yes) (on_board yes)
-    (property "Reference" "JP?" (id 0) (at 33.02 111.7599 90)
+    (property "Reference" "JP1" (id 0) (at 33.02 111.7599 90)
       (effects (font (size 1.27 1.27)) (justify left))
     )

Commit message: March 23rd First pre-alpha
First time ZERO errors and 93 warnings. Schematics are done, now to deal with warnings and footprints.
Parts:
- C21, C22: footprint (none) -> Capacitor_THT:C_Disc_D7.0mm_W2.5mm_P5.00mm
- R16, R22, R23: footprint (none) -> Resistor_THT:R_Axial_DIN0207_L6.3mm_D2.5mm_P10.16mm_Horizontal
Changed lines of the file:
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@@
 (kicad_sch (version 20211123) (generator eeschema)
-  (paper "A3")
+  (paper "A4")
   (title_block
     (comment 2 "Евстафьев")
@@
     (property "Reference" "R23" (id 0) (at 101.6 152.4 90))
     (property "Value" "240" (id 1) (at 101.6 154.94 90))
-    (property "Footprint" "" (id 2) (at 101.6 160.528 90)
+    (property "Footprint" "Resistor_THT:R_Axial_DIN0207_L6.3mm_D2.5mm_P10.16mm_Horizontal" (id 2) (at 101.6 160.528 90)
       (effects (font (size 1.27 1.27)) hide)
     )
@@
       (effects (font (size 1.27 1.27)) (justify left))
     )
-    (property "Footprint" "" (id 2) (at 84.1502 182.245 0)
+    (property "Footprint" "Capacitor_THT:C_Disc_D7.0mm_W2.5mm_P5.00mm" (id 2) (at 84.1502 182.245 0)
       (effects (font (size 1.27 1.27)) hide)
     )
@@
       (effects (font (size 1.27 1.27)) (justify left))
     )
-    (property "Footprint" "" (id 2) (at 97.4852 182.245 0)
+    (property "Footprint" "Capacitor_THT:C_Disc_D7.0mm_W2.5mm_P5.00mm" (id 2) (at 97.4852 182.245 0)
       (effects (font (size 1.27 1.27)) hide)
     )
@@
       (effects (font (size 1.27 1.27)) (justify left))
     )
-    (property "Footprint" "" (id 2) (at 84.582 163.83 90)
+    (property "Footprint" "Resistor_THT:R_Axial_DIN0207_L6.3mm_D2.5mm_P10.16mm_Horizontal" (id 2) (at 84.582 163.83 90)
       (effects (font (size 1.27 1.27)) hide)
     )
@@
       (effects (font (size 1.27 1.27)) (justify left))
     )
-    (property "Footprint" "" (id 2) (at 33.782 101.6 90)
-      (effects (font (size 1.27 1.27)) hide)
-    )
+    (property "Footprint" "Resistor_THT:R_Axial_DIN0207_L6.3mm_D2.5mm_P10.16mm_Horizontal" (id 2) (at 33.782 101.6 90)
+      (effects (font (size 1.27 1.27)) hide)
+    )

Commit message: March 24th Second Update
Parts:
- U22: symbol 74xx:74LS257 -> w_connectors:74LS257_(КР1533КП11А)_U22
- U25: symbol 74xx:74LS257 -> w_connectors:74LS257_(КР1533КП11А)_U25
Changed lines of the file:
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@@
     (pin "7")
   )
-  (symbol (lib_name "74LS257_1") (lib_id "74xx:74LS257") (at 68.58 48.895 0) (unit 1)
+  (symbol (lib_id "w_connectors:74LS257_(КР1533КП11А)_U22") (at 68.58 48.895 0) (unit 1)
     (in_bom yes) (on_board yes) (fields_autoplaced)
     (property "Reference" "U22" (id 0) (at 70.5994 26.035 0)
@@
     (pin "2")
   )
-  (symbol (lib_name "74LS257_1") (lib_id "74xx:74LS257") (at 68.58 102.87 0) (unit 1)
+  (symbol (lib_id "w_connectors:74LS257_(КР1533КП11А)_U25") (at 68.58 102.87 0) (unit 1)
     (in_bom yes) (on_board yes) (fields_autoplaced)
     (property "Reference" "U25" (id 0) (at 70.5994 80.01 0)

Commit message: March 26th update
Parts:
- U22, U25, U31, U32, U33, U34, U35, U36, U37, U38: footprint Package_DIP:DIP-16_W7.62mm_Socket_LongPads -> Package_DIP:DIP-16_W7.62mm_Socket
- U39, U40: footprint Package_DIP:DIP-14_W7.62mm_Socket_LongPads -> Package_DIP:DIP-14_W7.62mm_Socket
Changed lines of the file:
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@@
     (property "Reference" "U38" (id 0) (at 266.065 107.95 0))
     (property "Value" "RU5D1" (id 1) (at 266.065 110.49 0))
-    (property "Footprint" "Package_DIP:DIP-16_W7.62mm_Socket_LongPads" (id 2) (at 253.365 95.885 0)
+    (property "Footprint" "Package_DIP:DIP-16_W7.62mm_Socket" (id 2) (at 253.365 95.885 0)
       (effects (font (size 1.27 1.27)) hide)
     )
@@
     (property "Reference" "U34" (id 0) (at 266.065 55.245 0))
     (property "Value" "RU5D1" (id 1) (at 266.065 57.785 0))
-    (property "Footprint" "Package_DIP:DIP-16_W7.62mm_Socket_LongPads" (id 2) (at 253.365 42.545 0)
+    (property "Footprint" "Package_DIP:DIP-16_W7.62mm_Socket" (id 2) (at 253.365 42.545 0)
       (effects (font (size 1.27 1.27)) hide)
     )
@@
     (property "Reference" "U31" (id 0) (at 142.875 55.245 0))
     (property "Value" "RU5D1" (id 1) (at 142.875 57.785 0))
-    (property "Footprint" "Package_DIP:DIP-16_W7.62mm_Socket_LongPads" (id 2) (at 130.175 42.545 0)
+    (property "Footprint" "Package_DIP:DIP-16_W7.62mm_Socket" (id 2) (at 130.175 42.545 0)
       (effects (font (size 1.27 1.27)) hide)
     )
@@
     (property "Reference" "U40" (id 0) (at 49.53 146.685 0))
     (property "Value" "IN74ALS00N (КР1533ЛА3)" (id 1) (at 49.53 139.7 0))
-    (property "Footprint" "Package_DIP:DIP-14_W7.62mm_Socket_LongPads" (id 2) (at 49.53 146.685 0)
+    (property "Footprint" "Package_DIP:DIP-14_W7.62mm_Socket" (id 2) (at 49.53 146.685 0)
       (effects (font (size 1.27 1.27)) hide)
     )
@@
       (effects (font (size 1.27 1.27)) (justify left))
     )
-    (property "Footprint" "Package_DIP:DIP-16_W7.62mm_Socket_LongPads" (id 2) (at 68.58 48.895 0)
+    (property "Footprint" "Package_DIP:DIP-16_W7.62mm_Socket" (id 2) (at 68.58 48.895 0)
       (effects (font (size 1.27 1.27)) hide)
     )
@@
     (property "Reference" "U40" (id 0) (at 77.47 144.145 0))
     (property "Value" "IN74ALS00N (КР1533ЛА3)" (id 1) (at 77.47 137.795 0))
-    (property "Footprint" "Package_DIP:DIP-14_W7.62mm_Socket_LongPads" (id 2) (at 77.47 144.145 0)
+    (property "Footprint" "Package_DIP:DIP-14_W7.62mm_Socket" (id 2) (at 77.47 144.145 0)
       (effects (font (size 1.27 1.27)) hide)
     )
@@
     (property "Reference" "U32" (id 0) (at 183.515 56.515 0))
     (property "Value" "RU5D1" (id 1) (at 183.515 59.055 0))
-    (property "Footprint" "Package_DIP:DIP-16_W7.62mm_Socket_LongPads" (id 2) (at 170.815 42.545 0)
+    (property "Footprint" "Package_DIP:DIP-16_W7.62mm_Socket" (id 2) (at 170.815 42.545 0)
       (effects (font (size 1.27 1.27)) hide)
     )
@@
     (property "Reference" "U39" (id 0) (at 49.53 163.195 0))
     (property "Value" "IN74ALS32N (КР1533ЛЛ1)" (id 1) (at 50.8 156.21 0))
-    (property "Footprint" "Package_DIP:DIP-14_W7.62mm_Socket_LongPads" (id 2) (at 49.53 163.195 0)
+    (property "Footprint" "Package_DIP:DIP-14_W7.62mm_Socket" (id 2) (at 49.53 163.195 0)
       (effects (font (size 1.27 1.27)) hide)
     )
@@
     (property "Reference" "U39" (id 0) (at 102.235 146.685 0))
     (property "Value" "IN74ALS32N (КР1533ЛЛ1)" (id 1) (at 101.6 140.335 0))
-    (property "Footprint" "Package_DIP:DIP-14_W7.62mm_Socket_LongPads" (id 2) (at 101.6 146.685 0)
+    (property "Footprint" "Package_DIP:DIP-14_W7.62mm_Socket" (id 2) (at 101.6 146.685 0)
       (effects (font (size 1.27 1.27)) hide)
     )
@@
     (property "Reference" "U39" (id 0) (at 49.53 179.705 0))
     (property "Value" "IN74ALS32N (КР1533ЛЛ1)" (id 1) (at 49.53 173.355 0))
-    (property "Footprint" "Package_DIP:DIP-14_W7.62mm_Socket_LongPads" (id 2) (at 49.53 179.705 0)
+    (property "Footprint" "Package_DIP:DIP-14_W7.62mm_Socket" (id 2) (at 49.53 179.705 0)
       (effects (font (size 1.27 1.27)) hide)
     )
@@
     (property "Reference" "U33" (id 0) (at 226.06 55.88 0))
     (property "Value" "RU5D1" (id 1) (at 226.06 58.42 0))
-    (property "Footprint" "Package_DIP:DIP-16_W7.62mm_Socket_LongPads" (id 2) (at 212.725 42.545 0)
+    (property "Footprint" "Package_DIP:DIP-16_W7.62mm_Socket" (id 2) (at 212.725 42.545 0)
       (effects (font (size 1.27 1.27)) hide)
     )
@@
       (effects (font (size 1.27 1.27)) (justify left))
     )
-    (property "Footprint" "Package_DIP:DIP-16_W7.62mm_Socket_LongPads" (id 2) (at 68.58 102.87 0)
+    (property "Footprint" "Package_DIP:DIP-16_W7.62mm_Socket" (id 2) (at 68.58 102.87 0)
       (effects (font (size 1.27 1.27)) hide)
     )
@@
     (property "Reference" "U36" (id 0) (at 183.515 107.315 0))
     (property "Value" "RU5D1" (id 1) (at 183.515 109.855 0))
-    (property "Footprint" "Package_DIP:DIP-16_W7.62mm_Socket_LongPads" (id 2) (at 170.815 95.885 0)
+    (property "Footprint" "Package_DIP:DIP-16_W7.62mm_Socket" (id 2) (at 170.815 95.885 0)
       (effects (font (size 1.27 1.27)) hide)
     )
@@
     (property "Reference" "U37" (id 0) (at 225.425 107.315 0))
     (property "Value" "RU5D1" (id 1) (at 225.425 109.855 0))
-    (property "Footprint" "Package_DIP:DIP-16_W7.62mm_Socket_LongPads" (id 2) (at 212.725 95.885 0)
+    (property "Footprint" "Package_DIP:DIP-16_W7.62mm_Socket" (id 2) (at 212.725 95.885 0)
       (effects (font (size 1.27 1.27)) hide)
     )
@@
     (property "Reference" "U35" (id 0) (at 142.875 107.95 0))
     (property "Value" "RU5D1" (id 1) (at 142.875 110.49 0))
-    (property "Footprint" "Package_DIP:DIP-16_W7.62mm_Socket_LongPads" (id 2) (at 130.175 95.885 0)
+    (property "Footprint" "Package_DIP:DIP-16_W7.62mm_Socket" (id 2) (at 130.175 95.885 0)
       (effects (font (size 1.27 1.27)) hide)
     )
@@
     (property "Reference" "U39" (id 0) (at 113.03 168.91 0))
     (property "Value" "IN74ALS32N (КР1533ЛЛ1)" (id 1) (at 112.395 161.925 0))
-    (property "Footprint" "Package_DIP:DIP-14_W7.62mm_Socket_LongPads" (id 2) (at 112.395 168.91 0)
-      (effects (font (size 1.27 1.27)) hide)
-    )
+    (property "Footprint" "Package_DIP:DIP-14_W7.62mm_Socket" (id 2) (at 112.395 168.91 0)
+      (effects (font (size 1.27 1.27)) hide)
+    )
