File: ramd31d38.kicad_sch (KiCad schematic)
At the start: 18 parts, among them U22 74LS257 (КР1533КП11А), U25 74LS257 (КР1533КП11А), U31 RU5D1, U32 RU5D1, U33 RU5D1, U34 RU5D1, U35 RU5D1, U36 RU5D1, U37 RU5D1, U38 RU5D1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

Commit message: Update ramd31d38.kicad_sch
Other:
- note added: "Select upper or lower part of RU5"
Changed lines of the file:
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@@
     (stroke (width 0) (type default))
+  )
+  (text "Select upper or lower part of RU5" (at 27.94 121.92 90)
+    (effects (font (size 1.27 1.27)) (justify left bottom))
   )
   (global_label "A5" (shape input) (at 55.88 97.79 180) (fields_autoplaced)

Commit message: Version 1.0 schematics and PCB complete
Parts:
- C21, C22: symbol Device:C -> Delta_s_m_Lib:C
- JP1: symbol Jumper:Jumper_3_Bridged12 -> Delta_s_m_Lib:Jumper_3_Bridged12
- R16, R22, R23: symbol Device:R -> Delta_s_m_Lib:R
- U22: symbol w_connectors:74LS257_(КР1533КП11А)_U22 -> Delta_s_m_Lib:74LS257_(КР1533КП11А)_U22
- U25: symbol w_connectors:74LS257_(КР1533КП11А)_U25 -> Delta_s_m_Lib:74LS257_(КР1533КП11А)_U25
- U31, U32, U33, U34, U37, U38: symbol w_connectors:RU5D1 -> Delta_s_m_Lib:RU5D1
- U35: symbol w_connectors:RU5D1 -> Delta_s_m_Lib:RU5D1_5
- U36: symbol w_connectors:RU5D1 -> Delta_s_m_Lib:RU5D1_6
- U39: symbol 74xx:74LS32 -> Delta_s_m_Lib:74LS32
- U40: symbol 74xx:74LS00 -> Delta_s_m_Lib:74LS00
Changed lines of the file:
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@@
     )
   )
-  (symbol (lib_id "Device:R") (at 101.6 158.75 90) (unit 1)
+  (symbol (lib_id "Delta_s_m_Lib:R") (at 101.6 158.75 90) (unit 1)
     (in_bom yes) (on_board yes) (dnp no) (fields_autoplaced)
     (property "Reference" "R23" (at 101.6 152.4 90)
@@
     )
   )
-  (symbol (lib_id "Jumper:Jumper_3_Bridged12") (at 35.56 113.03 90) (mirror x) (unit 1)
+  (symbol (lib_id "Delta_s_m_Lib:Jumper_3_Bridged12") (at 35.56 113.03 90) (mirror x) (unit 1)
     (in_bom yes) (on_board yes) (dnp no)
     (property "Reference" "JP1" (at 33.02 111.7599 90)
@@
     )
   )
-  (symbol (lib_id "Device:C") (at 83.185 178.435 0) (unit 1)
+  (symbol (lib_id "Delta_s_m_Lib:C") (at 83.185 178.435 0) (unit 1)
     (in_bom yes) (on_board yes) (dnp no) (fields_autoplaced)
     (property "Reference" "C21" (at 86.36 177.1649 0)
@@
     )
   )
-  (symbol (lib_id "w_connectors:RU5D1") (at 262.255 104.775 0) (unit 1)
+  (symbol (lib_id "Delta_s_m_Lib:RU5D1") (at 262.255 104.775 0) (unit 1)
     (in_bom yes) (on_board yes) (dnp no)
     (property "Reference" "U38" (at 266.065 107.95 0)
@@
     )
   )
-  (symbol (lib_id "w_connectors:RU5D1") (at 262.255 51.435 0) (unit 1)
+  (symbol (lib_id "Delta_s_m_Lib:RU5D1") (at 262.255 51.435 0) (unit 1)
     (in_bom yes) (on_board yes) (dnp no)
     (property "Reference" "U34" (at 266.065 55.245 0)
@@
     )
   )
-  (symbol (lib_id "w_connectors:RU5D1") (at 139.065 51.435 0) (unit 1)
+  (symbol (lib_id "Delta_s_m_Lib:RU5D1") (at 139.065 51.435 0) (unit 1)
     (in_bom yes) (on_board yes) (dnp no)
     (property "Reference" "U31" (at 142.875 55.245 0)
@@
     )
   )
-  (symbol (lib_id "74xx:74LS00") (at 49.53 146.685 0) (mirror x) (unit 4)
+  (symbol (lib_id "Delta_s_m_Lib:74LS00") (at 49.53 146.685 0) (mirror x) (unit 4)
     (in_bom yes) (on_board yes) (dnp no)
     (property "Reference" "U40" (at 49.53 146.685 0)
@@
     )
   )
-  (symbol (lib_id "w_connectors:74LS257_(КР1533КП11А)_U22") (at 68.58 48.895 0) (unit 1)
+  (symbol (lib_id "Delta_s_m_Lib:74LS257_(КР1533КП11А)_U22") (at 68.58 48.895 0) (unit 1)
     (in_bom yes) (on_board yes) (dnp no) (fields_autoplaced)
     (property "Reference" "U22" (at 70.5994 26.035 0)
@@
     )
   )
-  (symbol (lib_id "74xx:74LS00") (at 77.47 144.145 0) (unit 3)
+  (symbol (lib_id "Delta_s_m_Lib:74LS00") (at 77.47 144.145 0) (unit 3)
     (in_bom yes) (on_board yes) (dnp no)
     (property "Reference" "U40" (at 77.47 144.145 0)
@@
     )
   )
-  (symbol (lib_id "w_connectors:RU5D1") (at 179.705 51.435 0) (unit 1)
+  (symbol (lib_id "Delta_s_m_Lib:RU5D1") (at 179.705 51.435 0) (unit 1)
     (in_bom yes) (on_board yes) (dnp no)
     (property "Reference" "U32" (at 183.515 56.515 0)
@@
     )
   )
-  (symbol (lib_id "74xx:74LS32") (at 49.53 163.195 0) (unit 4)
+  (symbol (lib_id "Delta_s_m_Lib:74LS32") (at 49.53 163.195 0) (unit 4)
     (in_bom yes) (on_board yes) (dnp no)
     (property "Reference" "U39" (at 49.53 163.195 0)
@@
     )
   )
-  (symbol (lib_id "74xx:74LS32") (at 101.6 146.685 0) (unit 1)
+  (symbol (lib_id "Delta_s_m_Lib:74LS32") (at 101.6 146.685 0) (unit 1)
     (in_bom yes) (on_board yes) (dnp no)
     (property "Reference" "U39" (at 102.235 146.685 0)
@@
     )
   )
-  (symbol (lib_id "74xx:74LS32") (at 49.53 179.705 0) (unit 2)
+  (symbol (lib_id "Delta_s_m_Lib:74LS32") (at 49.53 179.705 0) (unit 2)
     (in_bom yes) (on_board yes) (dnp no)
     (property "Reference" "U39" (at 49.53 179.705 0)
@@
     )
   )
-  (symbol (lib_id "w_connectors:RU5D1") (at 221.615 51.435 0) (unit 1)
+  (symbol (lib_id "Delta_s_m_Lib:RU5D1") (at 221.615 51.435 0) (unit 1)
     (in_bom yes) (on_board yes) (dnp no)
     (property "Reference" "U33" (at 226.06 55.88 0)
@@
     )
   )
-  (symbol (lib_id "Device:C") (at 96.52 178.435 0) (unit 1)
+  (symbol (lib_id "Delta_s_m_Lib:C") (at 96.52 178.435 0) (unit 1)
     (in_bom yes) (on_board yes) (dnp no) (fields_autoplaced)
     (property "Reference" "C22" (at 99.695 177.1649 0)
@@
     )
   )
-  (symbol (lib_id "w_connectors:74LS257_(КР1533КП11А)_U25") (at 68.58 102.87 0) (unit 1)
+  (symbol (lib_id "Delta_s_m_Lib:74LS257_(КР1533КП11А)_U25") (at 68.58 102.87 0) (unit 1)
     (in_bom yes) (on_board yes) (dnp no) (fields_autoplaced)
     (property "Reference" "U25" (at 70.5994 80.01 0)
@@
     )
   )
-  (symbol (lib_name "RU5D1_6") (lib_id "w_connectors:RU5D1") (at 179.705 104.775 0) (unit 1)
+  (symbol (lib_name "RU5D1_6") (lib_id "Delta_s_m_Lib:RU5D1_6") (at 179.705 104.775 0) (unit 1)
     (in_bom yes) (on_board yes) (dnp no)
     (property "Reference" "U36" (at 183.515 107.315 0)
@@
     )
   )
-  (symbol (lib_id "w_connectors:RU5D1") (at 221.615 104.775 0) (unit 1)
+  (symbol (lib_id "Delta_s_m_Lib:RU5D1") (at 221.615 104.775 0) (unit 1)
     (in_bom yes) (on_board yes) (dnp no)
     (property "Reference" "U37" (at 225.425 107.315 0)
@@
     )
   )
-  (symbol (lib_id "Device:R") (at 86.36 163.83 0) (unit 1)
+  (symbol (lib_id "Delta_s_m_Lib:R") (at 86.36 163.83 0) (unit 1)
     (in_bom yes) (on_board yes) (dnp no) (fields_autoplaced)
     (property "Reference" "R22" (at 88.265 162.5599 0)
@@
     )
   )
-  (symbol (lib_name "RU5D1_5") (lib_id "w_connectors:RU5D1") (at 139.065 104.775 0) (unit 1)
+  (symbol (lib_name "RU5D1_5") (lib_id "Delta_s_m_Lib:RU5D1_5") (at 139.065 104.775 0) (unit 1)
     (in_bom yes) (on_board yes) (dnp no)
     (property "Reference" "U35" (at 142.875 107.95 0)
@@
     )
   )
-  (symbol (lib_id "Device:R") (at 35.56 101.6 0) (unit 1)
+  (symbol (lib_id "Delta_s_m_Lib:R") (at 35.56 101.6 0) (unit 1)
     (in_bom yes) (on_board yes) (dnp no) (fields_autoplaced)
     (property "Reference" "R16" (at 37.465 100.3299 0)
@@
     )
   )
-  (symbol (lib_id "74xx:74LS32") (at 112.395 168.91 0) (mirror x) (unit 3)
+  (symbol (lib_id "Delta_s_m_Lib:74LS32") (at 112.395 168.91 0) (mirror x) (unit 3)
     (in_bom yes) (on_board yes) (dnp no)
     (property "Reference" "U39" (at 113.03 168.91 0)

Commit message: Version 1.2 update
Parts:
- C21, C22: footprint Capacitor_THT:C_Disc_D7.0mm_W2.5mm_P5.00mm -> Delta_sm_lib:C_Disc_D7.0mm_W2.5mm_P5.00mm
- JP1: footprint Connector_PinHeader_2.54mm:PinHeader_1x03_P2.54mm_Vertical -> Delta_sm_lib:PinHeader_1x03_P2.54mm_Vertical
- R16, R22, R23: footprint Resistor_THT:R_Axial_DIN0207_L6.3mm_D2.5mm_P10.16mm_Horizontal -> Delta_sm_lib:R_Axial_DIN0207_L6.3mm_D2.5mm_P10.16mm_Horizontal
- U22, U25, U31, U32, U33, U34, U35, U36, U37, U38: footprint Package_DIP:DIP-16_W7.62mm_Socket -> Delta_sm_lib:DIP-16_W7.62mm_Socket
- U39, U40: footprint Package_DIP:DIP-14_W7.62mm_Socket -> Delta_sm_lib:DIP-14_W7.62mm_Socket
Changed lines of the file:
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@@
       (effects (font (size 1.27 1.27)))
     )
-    (property "Footprint" "Resistor_THT:R_Axial_DIN0207_L6.3mm_D2.5mm_P10.16mm_Horizontal" (at 101.6 160.528 90)
+    (property "Footprint" "Delta_sm_lib:R_Axial_DIN0207_L6.3mm_D2.5mm_P10.16mm_Horizontal" (at 101.6 160.528 90)
       (effects (font (size 1.27 1.27)) hide)
     )
@@
       (effects (font (size 1.27 1.27)) (justify left))
     )
-    (property "Footprint" "Connector_PinHeader_2.54mm:PinHeader_1x03_P2.54mm_Vertical" (at 35.56 113.03 0)
+    (property "Footprint" "Delta_sm_lib:PinHeader_1x03_P2.54mm_Vertical" (at 35.56 113.03 0)
       (effects (font (size 1.27 1.27)) hide)
     )
@@
       (effects (font (size 1.27 1.27)) (justify left))
     )
-    (property "Footprint" "Capacitor_THT:C_Disc_D7.0mm_W2.5mm_P5.00mm" (at 84.1502 182.245 0)
+    (property "Footprint" "Delta_sm_lib:C_Disc_D7.0mm_W2.5mm_P5.00mm" (at 84.1502 182.245 0)
       (effects (font (size 1.27 1.27)) hide)
     )
@@
       (effects (font (size 1.27 1.27)))
     )
-    (property "Footprint" "Package_DIP:DIP-16_W7.62mm_Socket" (at 253.365 95.885 0)
+    (property "Footprint" "Delta_sm_lib:DIP-16_W7.62mm_Socket" (at 253.365 95.885 0)
       (effects (font (size 1.27 1.27)) hide)
     )
@@
       (effects (font (size 1.27 1.27)))
     )
-    (property "Footprint" "Package_DIP:DIP-16_W7.62mm_Socket" (at 253.365 42.545 0)
+    (property "Footprint" "Delta_sm_lib:DIP-16_W7.62mm_Socket" (at 253.365 42.545 0)
       (effects (font (size 1.27 1.27)) hide)
     )
@@
       (effects (font (size 1.27 1.27)))
     )
-    (property "Footprint" "Package_DIP:DIP-16_W7.62mm_Socket" (at 130.175 42.545 0)
+    (property "Footprint" "Delta_sm_lib:DIP-16_W7.62mm_Socket" (at 130.175 42.545 0)
       (effects (font (size 1.27 1.27)) hide)
     )
@@
       (effects (font (size 1.27 1.27)))
     )
-    (property "Footprint" "Package_DIP:DIP-14_W7.62mm_Socket" (at 49.53 146.685 0)
+    (property "Footprint" "Delta_sm_lib:DIP-14_W7.62mm_Socket" (at 49.53 146.685 0)
       (effects (font (size 1.27 1.27)) hide)
     )
@@
       (effects (font (size 1.27 1.27)) (justify left))
     )
-    (property "Footprint" "Package_DIP:DIP-16_W7.62mm_Socket" (at 68.58 48.895 0)
+    (property "Footprint" "Delta_sm_lib:DIP-16_W7.62mm_Socket" (at 68.58 48.895 0)
       (effects (font (size 1.27 1.27)) hide)
     )
@@
       (effects (font (size 1.27 1.27)))
     )
-    (property "Footprint" "Package_DIP:DIP-14_W7.62mm_Socket" (at 77.47 144.145 0)
+    (property "Footprint" "Delta_sm_lib:DIP-14_W7.62mm_Socket" (at 77.47 144.145 0)
       (effects (font (size 1.27 1.27)) hide)
     )
@@
       (effects (font (size 1.27 1.27)))
     )
-    (property "Footprint" "Package_DIP:DIP-16_W7.62mm_Socket" (at 170.815 42.545 0)
+    (property "Footprint" "Delta_sm_lib:DIP-16_W7.62mm_Socket" (at 170.815 42.545 0)
       (effects (font (size 1.27 1.27)) hide)
     )
@@
       (effects (font (size 1.27 1.27)))
     )
-    (property "Footprint" "Package_DIP:DIP-14_W7.62mm_Socket" (at 49.53 163.195 0)
+    (property "Footprint" "Delta_sm_lib:DIP-14_W7.62mm_Socket" (at 49.53 163.195 0)
       (effects (font (size 1.27 1.27)) hide)
     )
@@
       (effects (font (size 1.27 1.27)))
     )
-    (property "Footprint" "Package_DIP:DIP-14_W7.62mm_Socket" (at 101.6 146.685 0)
+    (property "Footprint" "Delta_sm_lib:DIP-14_W7.62mm_Socket" (at 101.6 146.685 0)
       (effects (font (size 1.27 1.27)) hide)
     )
@@
       (effects (font (size 1.27 1.27)))
     )
-    (property "Footprint" "Package_DIP:DIP-14_W7.62mm_Socket" (at 49.53 179.705 0)
+    (property "Footprint" "Delta_sm_lib:DIP-14_W7.62mm_Socket" (at 49.53 179.705 0)
       (effects (font (size 1.27 1.27)) hide)
     )
@@
       (effects (font (size 1.27 1.27)))
     )
-    (property "Footprint" "Package_DIP:DIP-16_W7.62mm_Socket" (at 212.725 42.545 0)
+    (property "Footprint" "Delta_sm_lib:DIP-16_W7.62mm_Socket" (at 212.725 42.545 0)
       (effects (font (size 1.27 1.27)) hide)
     )
@@
       (effects (font (size 1.27 1.27)) (justify left))
     )
-    (property "Footprint" "Capacitor_THT:C_Disc_D7.0mm_W2.5mm_P5.00mm" (at 97.4852 182.245 0)
+    (property "Footprint" "Delta_sm_lib:C_Disc_D7.0mm_W2.5mm_P5.00mm" (at 97.4852 182.245 0)
       (effects (font (size 1.27 1.27)) hide)
     )
@@
       (effects (font (size 1.27 1.27)) (justify left))
     )
-    (property "Footprint" "Package_DIP:DIP-16_W7.62mm_Socket" (at 68.58 102.87 0)
+    (property "Footprint" "Delta_sm_lib:DIP-16_W7.62mm_Socket" (at 68.58 102.87 0)
       (effects (font (size 1.27 1.27)) hide)
     )
@@
       (effects (font (size 1.27 1.27)))
     )
-    (property "Footprint" "Package_DIP:DIP-16_W7.62mm_Socket" (at 170.815 95.885 0)
+    (property "Footprint" "Delta_sm_lib:DIP-16_W7.62mm_Socket" (at 170.815 95.885 0)
       (effects (font (size 1.27 1.27)) hide)
     )
@@
       (effects (font (size 1.27 1.27)))
     )
-    (property "Footprint" "Package_DIP:DIP-16_W7.62mm_Socket" (at 212.725 95.885 0)
+    (property "Footprint" "Delta_sm_lib:DIP-16_W7.62mm_Socket" (at 212.725 95.885 0)
       (effects (font (size 1.27 1.27)) hide)
     )
@@
       (effects (font (size 1.27 1.27)) (justify left))
     )
-    (property "Footprint" "Resistor_THT:R_Axial_DIN0207_L6.3mm_D2.5mm_P10.16mm_Horizontal" (at 84.582 163.83 90)
+    (property "Footprint" "Delta_sm_lib:R_Axial_DIN0207_L6.3mm_D2.5mm_P10.16mm_Horizontal" (at 84.582 163.83 90)
       (effects (font (size 1.27 1.27)) hide)
     )
@@
       (effects (font (size 1.27 1.27)))
     )
-    (property "Footprint" "Package_DIP:DIP-16_W7.62mm_Socket" (at 130.175 95.885 0)
+    (property "Footprint" "Delta_sm_lib:DIP-16_W7.62mm_Socket" (at 130.175 95.885 0)
       (effects (font (size 1.27 1.27)) hide)
     )
@@
       (effects (font (size 1.27 1.27)) (justify left))
     )
-    (property "Footprint" "Resistor_THT:R_Axial_DIN0207_L6.3mm_D2.5mm_P10.16mm_Horizontal" (at 33.782 101.6 90)
+    (property "Footprint" "Delta_sm_lib:R_Axial_DIN0207_L6.3mm_D2.5mm_P10.16mm_Horizontal" (at 33.782 101.6 90)
       (effects (font (size 1.27 1.27)) hide)
     )
@@
       (effects (font (size 1.27 1.27)))
     )
-    (property "Footprint" "Package_DIP:DIP-14_W7.62mm_Socket" (at 112.395 168.91 0)
-      (effects (font (size 1.27 1.27)) hide)
-    )
+    (property "Footprint" "Delta_sm_lib:DIP-14_W7.62mm_Socket" (at 112.395 168.91 0)
+      (effects (font (size 1.27 1.27)) hide)
+    )
