File: external.kicad_sch (KiCad schematic)
At the start: 47 parts, among them J5 Keyboard Connector, J6 Joystick 1, J7 Joystick 2, Q7 BC547B, Q8 BC547B, U66 SN74ALS175N (КР1533ТМ8), U67 8282 (КР580ИР82), U68 КР556РТ2, U72 КР556РТ2, U73 SN74ALS08 (КР1533ЛИ1)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

Commit message: March 26th update
Parts:
- J6, J7: footprint (none) -> w_conn_av:DIN-7-Variable
- U66: footprint Package_DIP:DIP-16_W7.62mm_Socket_LongPads -> Package_DIP:DIP-16_W7.62mm_Socket
- U67: footprint Package_DIP:DIP-20_W7.62mm_Socket_LongPads -> Package_DIP:DIP-20_W7.62mm_Socket
- U68, U72: footprint Package_DIP:DIP-28_W15.24mm_Socket_LongPads -> Package_DIP:DIP-28_W15.24mm_Socket
- U73, U74: footprint Package_DIP:DIP-14_W7.62mm_Socket_LongPads -> Package_DIP:DIP-14_W7.62mm_Socket
Changed lines of the file:
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@@
       (effects (font (size 1.27 1.27)) (justify left))
     )
-    (property "Footprint" "Package_DIP:DIP-14_W7.62mm_Socket_LongPads" (id 2) (at 63.5 215.265 0)
+    (property "Footprint" "Package_DIP:DIP-14_W7.62mm_Socket" (id 2) (at 63.5 215.265 0)
       (effects (font (size 1.27 1.27)) hide)
     )
@@
     (property "Reference" "U74" (id 0) (at 63.5 164.465 0))
     (property "Value" "SN74ALS08 (КР1533ЛИ1)" (id 1) (at 65.405 159.385 0))
-    (property "Footprint" "Package_DIP:DIP-14_W7.62mm_Socket_LongPads" (id 2) (at 63.5 164.465 0)
+    (property "Footprint" "Package_DIP:DIP-14_W7.62mm_Socket" (id 2) (at 63.5 164.465 0)
       (effects (font (size 1.27 1.27)) hide)
     )
@@
     (property "Reference" "U74" (id 0) (at 63.5 85.725 0))
     (property "Value" "SN74ALS08 (КР1533ЛИ1)" (id 1) (at 65.405 80.645 0))
-    (property "Footprint" "Package_DIP:DIP-14_W7.62mm_Socket_LongPads" (id 2) (at 63.5 85.725 0)
+    (property "Footprint" "Package_DIP:DIP-14_W7.62mm_Socket" (id 2) (at 63.5 85.725 0)
       (effects (font (size 1.27 1.27)) hide)
     )
@@
     (property "Reference" "J6" (id 0) (at 338.4551 201.295 0))
     (property "Value" "Joystick 1" (id 1) (at 338.4551 203.835 0))
-    (property "Footprint" "" (id 2) (at 338.455 193.04 0)
+    (property "Footprint" "w_conn_av:DIN-7-Variable" (id 2) (at 338.455 193.04 0)
       (effects (font (size 1.27 1.27)) hide)
     )
@@
       (effects (font (size 1.27 1.27)) (justify left))
     )
-    (property "Footprint" "Package_DIP:DIP-16_W7.62mm_Socket_LongPads" (id 2) (at 219.71 212.09 0)
+    (property "Footprint" "Package_DIP:DIP-16_W7.62mm_Socket" (id 2) (at 219.71 212.09 0)
       (effects (font (size 1.27 1.27)) hide)
     )
@@
       (effects (font (size 1.27 1.27)) (justify left))
     )
-    (property "Footprint" "Package_DIP:DIP-28_W15.24mm_Socket_LongPads" (id 2) (at 162.56 40.005 0)
+    (property "Footprint" "Package_DIP:DIP-28_W15.24mm_Socket" (id 2) (at 162.56 40.005 0)
       (effects (font (size 1.27 1.27)) hide)
     )
@@
     (property "Reference" "J7" (id 0) (at 338.4551 234.315 0))
     (property "Value" "Joystick 2" (id 1) (at 338.4551 236.855 0))
-    (property "Footprint" "" (id 2) (at 338.455 226.06 0)
+    (property "Footprint" "w_conn_av:DIN-7-Variable" (id 2) (at 338.455 226.06 0)
       (effects (font (size 1.27 1.27)) hide)
     )
@@
       (effects (font (size 1.27 1.27)) (justify left))
     )
-    (property "Footprint" "Package_DIP:DIP-28_W15.24mm_Socket_LongPads" (id 2) (at 188.595 126.365 0)
+    (property "Footprint" "Package_DIP:DIP-28_W15.24mm_Socket" (id 2) (at 188.595 126.365 0)
       (effects (font (size 1.27 1.27)) hide)
     )
@@
       (effects (font (size 1.27 1.27)) (justify left))
     )
-    (property "Footprint" "Package_DIP:DIP-20_W7.62mm_Socket_LongPads" (id 2) (at 241.935 79.375 0)
+    (property "Footprint" "Package_DIP:DIP-20_W7.62mm_Socket" (id 2) (at 241.935 79.375 0)
       (effects (font (size 1.27 1.27)) hide)
     )
@@
     (property "Reference" "U73" (id 0) (at 63.5 124.46 0))
     (property "Value" "SN74ALS08 (КР1533ЛИ1)" (id 1) (at 65.405 119.38 0))
-    (property "Footprint" "Package_DIP:DIP-14_W7.62mm_Socket_LongPads" (id 2) (at 63.5 124.46 0)
+    (property "Footprint" "Package_DIP:DIP-14_W7.62mm_Socket" (id 2) (at 63.5 124.46 0)
       (effects (font (size 1.27 1.27)) hide)
     )
@@
     (property "Reference" "U74" (id 0) (at 63.5 72.39 0))
     (property "Value" "SN74ALS08 (КР1533ЛИ1)" (id 1) (at 65.405 67.31 0))
-    (property "Footprint" "Package_DIP:DIP-14_W7.62mm_Socket_LongPads" (id 2) (at 63.5 72.39 0)
+    (property "Footprint" "Package_DIP:DIP-14_W7.62mm_Socket" (id 2) (at 63.5 72.39 0)
       (effects (font (size 1.27 1.27)) hide)
     )
@@
     (property "Reference" "U73" (id 0) (at 63.5 105.41 0))
     (property "Value" "SN74ALS08 (КР1533ЛИ1)" (id 1) (at 65.405 100.33 0))
-    (property "Footprint" "Package_DIP:DIP-14_W7.62mm_Socket_LongPads" (id 2) (at 63.5 105.41 0)
+    (property "Footprint" "Package_DIP:DIP-14_W7.62mm_Socket" (id 2) (at 63.5 105.41 0)
       (effects (font (size 1.27 1.27)) hide)
     )
@@
     (property "Reference" "U73" (id 0) (at 63.5 59.055 0))
     (property "Value" "SN74ALS08 (КР1533ЛИ1)" (id 1) (at 64.77 53.975 0))
-    (property "Footprint" "Package_DIP:DIP-14_W7.62mm_Socket_LongPads" (id 2) (at 63.5 59.055 0)
+    (property "Footprint" "Package_DIP:DIP-14_W7.62mm_Socket" (id 2) (at 63.5 59.055 0)
       (effects (font (size 1.27 1.27)) hide)
     )
@@
     (property "Reference" "U73" (id 0) (at 63.5 144.145 0))
     (property "Value" "SN74ALS08 (КР1533ЛИ1)" (id 1) (at 65.405 139.065 0))
-    (property "Footprint" "Package_DIP:DIP-14_W7.62mm_Socket_LongPads" (id 2) (at 63.5 144.145 0)
+    (property "Footprint" "Package_DIP:DIP-14_W7.62mm_Socket" (id 2) (at 63.5 144.145 0)
       (effects (font (size 1.27 1.27)) hide)
     )
@@
       (effects (font (size 1.27 1.27)) (justify left))
     )
-    (property "Footprint" "Package_DIP:DIP-14_W7.62mm_Socket_LongPads" (id 2) (at 78.74 215.265 0)
+    (property "Footprint" "Package_DIP:DIP-14_W7.62mm_Socket" (id 2) (at 78.74 215.265 0)
       (effects (font (size 1.27 1.27)) hide)
     )
@@
     (property "Reference" "U74" (id 0) (at 63.5 41.91 0))
     (property "Value" "SN74ALS08 (КР1533ЛИ1)" (id 1) (at 64.77 36.195 0))
-    (property "Footprint" "Package_DIP:DIP-14_W7.62mm_Socket_LongPads" (id 2) (at 63.5 41.91 0)
-      (effects (font (size 1.27 1.27)) hide)
-    )
+    (property "Footprint" "Package_DIP:DIP-14_W7.62mm_Socket" (id 2) (at 63.5 41.91 0)
+      (effects (font (size 1.27 1.27)) hide)
+    )

Commit message: 29th march 2023 Update 1
Connections:
- net at U66.14 (~{Q3}): no longer R55.2
- net at U66.7 (Q1): now also R55.2
Other:
- moved on the sheet: R55
Changed lines of the file:
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@@
   (no_connect (at 232.41 212.09))
   (no_connect (at 232.41 204.47))
+  (no_connect (at 232.41 219.71))
   (no_connect (at 232.41 209.55))
   (no_connect (at 207.645 163.195))
-  (no_connect (at 232.41 207.01))
   (no_connect (at 181.61 79.375))
   (wire (pts (xy 199.39 132.715) (xy 207.645 132.715))
@@
     (stroke (width 0) (type default) (color 0 0 0 0))
   )
-  (wire (pts (xy 232.41 219.71) (xy 233.68 219.71))
-    (stroke (width 0) (type default) (color 0 0 0 0))
-  )
   (wire (pts (xy 241.935 146.685) (xy 231.775 146.685))
     (stroke (width 0) (type default) (color 0 0 0 0))
@@
     (stroke (width 0) (type default) (color 0 0 0 0))
   )
+  (wire (pts (xy 232.41 207.01) (xy 238.125 207.01))
+    (stroke (width 0) (type default) (color 0 0 0 0))
+  )
   (wire (pts (xy 199.39 145.415) (xy 207.645 145.415))
     (stroke (width 0) (type default) (color 0 0 0 0))
@@
     (stroke (width 0) (type default) (color 0 0 0 0))
   )
+  (wire (pts (xy 238.125 207.01) (xy 238.125 219.71))
+    (stroke (width 0) (type default) (color 0 0 0 0))
+  )
   (wire (pts (xy 146.05 35.56) (xy 154.94 35.56))
     (stroke (width 0) (type default) (color 0 0 0 0))
@@
     (stroke (width 0) (type default) (color 0 0 0 0))
   )
-  (wire (pts (xy 241.3 219.71) (xy 247.015 219.71))
+  (wire (pts (xy 245.745 219.71) (xy 247.015 219.71))
     (stroke (width 0) (type default) (color 0 0 0 0))
   )
@@
     (pin "7")
   )
-  (symbol (lib_id "Device:R") (at 237.49 219.71 270) (unit 1)
-    (in_bom yes) (on_board yes)
-    (property "Reference" "R55" (id 0) (at 237.49 222.885 90))
-    (property "Value" "2.2K" (id 1) (at 237.49 219.71 90))
-    (property "Footprint" "Resistor_THT:R_Axial_DIN0207_L6.3mm_D2.5mm_P10.16mm_Horizontal" (id 2) (at 237.49 217.932 90)
-      (effects (font (size 1.27 1.27)) hide)
-    )
-    (property "Datasheet" "~" (id 3) (at 237.49 219.71 0)
-      (effects (font (size 1.27 1.27)) hide)
-    )
+  (symbol (lib_id "Device:R") (at 241.935 219.71 270) (unit 1)
+    (in_bom yes) (on_board yes)
+    (property "Reference" "R55" (id 0) (at 241.935 222.885 90))
+    (property "Value" "2.2K" (id 1) (at 241.935 219.71 90))
+    (property "Footprint" "Resistor_THT:R_Axial_DIN0207_L6.3mm_D2.5mm_P10.16mm_Horizontal" (id 2) (at 241.935 217.932 90)
+      (effects (font (size 1.27 1.27)) hide)
+    )
+    (property "Datasheet" "~" (id 3) (at 241.935 219.71 0)
+      (effects (font (size 1.27 1.27)) hide)
+    )
