File: delta48m.kicad_pcb (KiCad board)
At the start: 2 copper layers, 287 x 150 mm, 222 parts, among them J1 SNP, J2 DIN-7 Video, J3 DIN-5 Audio, J4 DIN-5 Power, J5 Keyboard Connector, J6 Joystick 1, J7 Joystick 2, Q1 BC547B, Q3 BC547B, Q4 BC547B, Q5 BC547B, Q6 BC547B, Q7 BC547B, Q8 BC547B, SW1 Reset button, U1 SN74ALS08 (КР1533ЛИ1), U10 SN74ALS08 (КР1533ЛИ1), U11 IN74ALS00N (КР1533ЛА3), U12 IN74ALS02N (КР1533ЛЕ1), U13 SN74ALS10 (КР1533ЛА4), U14 SN74ALS86N (КР1533ЛП5), U15 CD4520АN (К561ИЕ10A), U16 SN74ALS257N_(КР1533КП11А), U17 CD4520АN (К561ИЕ10A), U18 CD4011 (К561ЛА7), U19 SN74ALS04 (КР1533ЛН1), U2 SN74ALS04 (КР1533ЛН1), U20 SN74ALS74AN (КР1533ТМ2), U21 SN74ALS04 (КР1533ЛН1), U22 74LS257 (КР1533КП11А), U23 SN74ALS253N (КР1533КП12), U24 SN74ALS253N (КР1533КП12), U25 74LS257 (КР1533КП11А), U26 SN74ALS253N (КР1533КП12), U27 SN74ALS253N (КР1533КП12), U28 IN74ALS32N (КР1533ЛЛ1), U29 IN74ALS32N (КР1533ЛЛ1), U3 SN74ALS74AN (КР1533ТМ2), U30 IN74ALS02N (КР1533ЛЕ1), U31 RU5D1, U32 RU5D1, U33 RU5D1, U34 RU5D1, U35 RU5D1, U36 RU5D1, U37 RU5D1, U38 RU5D1, U39 IN74ALS32N (КР1533ЛЛ1), U4 SN74ALS193N_(КР1533ИЕ7), U40 IN74ALS00N (КР1533ЛА3), U41 2118 (КР565РУ6), U42 2118 (КР565РУ6), U43 2118 (КР565РУ6), U44 2118 (КР565РУ6), U45 2118 (КР565РУ6), U46 2118 (КР565РУ6), U47 2118 (КР565РУ6), U48 2118 (КР565РУ6), U49 SN74ALS04 (КР1533ЛН1), U5 СD4013АN_(К561ТМ2), U50 SN74ALS86N (КР1533ЛП5), U51 SN7486N (К155ЛП5), U52 SN74ALS175N (КР1533ТМ8), U53 SN74ALS153N (КР1533КП2), U54 SN74ALS298N (КР1533КП13), U55 74LS257 (КР1533КП11А), U56 SN74ALS175N (КР1533ТМ8), U57 SN74LS295N_(К555ИР16), U58 SN74LS295N_(К555ИР16), U59 SN74ALS175N (КР1533ТМ8), U6 CD4015A (К561ИР2), U60 SN74ALS153N (КР1533КП2), U61 SN74ALS298N (КР1533КП13), U62 74LS257 (КР1533КП11А), U63 SN74ALS175N (КР1533ТМ8), U64 SN74LS295N_(К555ИР16), U65 SN74LS295N_(К555ИР16), U66 SN74ALS175N (КР1533ТМ8), U67 8282 (КР580ИР82), U68 КР556РТ2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

Commit message: Video connector fix and labels
Parts:
- added H6: MountingHole_3.5mm, MountingHole:MountingHole_3.5mm, F.Cu at (112.3, 76.6)
- C14: value 4.7µF 15V -> 4.7µF 16V
- moved Log2 6.33 mm to (119.0, 77.2)
Connections:
- J2 pad 2: RED -> GND
- J2 pad 3: unconnected-(J2-Pad3) -> RED
- J2 pad 6: GND -> unconnected-(J2-Pad6)
Routing:
- net RED: track 22.2 -> 25.2 mm
- net GND: track 1873.4 -> 1870.9 mm
Other:
- board text added: "БПК {dblquote}Дельта-С{dblquote} Recreation Project Version 1.1 Board Design by MadCat, 2023 https://github.com/madcatse/Delta-S-M t.me/zx_delta_s https://www.youtube.com/@MadCatSE"
- board text removed: "БПК {dblquote}Дельта-С{dblquote} Recreation Project Version 1.0 Board Design by MadCat, 2023 https://github.com/madcatse/Delta-S-M t.me/zx_delta_s https://www.youtube.com/@MadCatSE"

Commit message: Update delta48m.kicad_pcb
Other:
- board text added: "+5V"
- board text added: "1 SYNC"
- board text added: "2 GND"
- board text added: "4 BLUE"
- board text added: "6 NC"
- board text added: "GREEN"
- board text added: "RED"
Changed lines of the file:
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@@
     (effects (font (size 2 2) (thickness 0.3)))
   )
+  (gr_text "+5V" (at 242.05 87.4) (layer "F.SilkS")
+    (effects (font (size 0.75 0.75) (thickness 0.15)))
+  )
   (gr_text "3" (at 178.439 81.56) (layer "F.SilkS")
     (effects (font (size 0.75 0.75) (thickness 0.15)))
@@
     (effects (font (size 0.75 0.75) (thickness 0.15)))
   )
-  (gr_text "5" (at 238.383 84.1) (layer "F.SilkS")
+  (gr_text "5" (at 236.25 85.7) (layer "F.SilkS")
     (effects (font (size 0.75 0.75) (thickness 0.15)))
   )
@@
     (effects (font (size 0.75 0.75) (thickness 0.15)))
   )
-  (gr_text "3" (at 240.923 81.56) (layer "F.SilkS")
+  (gr_text "3" (at 240.05 82.3) (layer "F.SilkS")
     (effects (font (size 0.75 0.75) (thickness 0.15)))
   )
@@
     (effects (font (size 0.75 0.75) (thickness 0.15)))
   )
+  (gr_text "RED" (at 241.95 82.3) (layer "F.SilkS")
+    (effects (font (size 0.75 0.75) (thickness 0.15)))
+  )
   (gr_text "2118 (КР565РУ6)" (at 204.093 209.068) (layer "F.SilkS")
     (effects (font (size 0.75 0.75) (thickness 0.15)))
@@
     (effects (font (size 0.75 0.75) (thickness 0.15)))
   )
-  (gr_text "6" (at 225.937 87.148) (layer "F.SilkS")
+  (gr_text "6 NC" (at 225.45 87.2) (layer "F.SilkS")
     (effects (font (size 0.75 0.75) (thickness 0.15)))
   )
@@
     (effects (font (size 0.75 0.75) (thickness 0.15)))
   )
-  (gr_text "1" (at 225.937 81.56) (layer "F.SilkS")
+  (gr_text "1 SYNC" (at 225.65 82.2) (layer "F.SilkS")
     (effects (font (size 0.75 0.75) (thickness 0.15)))
   )
@@
     (effects (font (size 0.75 0.75) (thickness 0.15)))
   )
-  (gr_text "2" (at 233.303 81.56) (layer "F.SilkS")
+  (gr_text "2 GND" (at 233.303 81.56) (layer "F.SilkS")
     (effects (font (size 0.75 0.75) (thickness 0.15)))
   )
@@
     (effects (font (size 0.75 0.75) (thickness 0.15)))
   )
-  (gr_text "7" (at 240.923 87.148) (layer "F.SilkS")
+  (gr_text "7" (at 240.45 87.4) (layer "F.SilkS")
     (effects (font (size 0.75 0.75) (thickness 0.15)))
   )
@@
     (effects (font (size 0.75 0.75) (thickness 0.15)))
   )
+  (gr_text "GREEN" (at 237.65 84.4) (layer "F.SilkS")
+    (effects (font (size 0.75 0.75) (thickness 0.15)))
+  )
   (gr_text "SN74ALS175N (КР1533ТМ8)" (at 256.671 132.106) (layer "F.SilkS")
     (effects (font (size 0.75 0.75) (thickness 0.15)))
   )
-  (gr_text "4" (at 228.477 84.354) (layer "F.SilkS")
+  (gr_text "4 BLUE" (at 229.25 84.7) (layer "F.SilkS")
     (effects (font (size 0.75 0.75) (thickness 0.15)))
   )

Commit message: Version 1.2 update
Parts:
- removed H2, H4, H5: MountingHole_3.2mm_M3, MountingHole:MountingHole_3.2mm_M3
- removed the H6 at (81.3, 211.0)
- added J8: USB_PORT, Connector_PinHeader_2.54mm:PinHeader_1x04_P2.54mm_Vertical, F.Cu at (216.3, 78.4)
- C1, C10, C11, C12, C13, C16, C17, C18, C19, C2, C20, C21, C22, C23, C24, C25, C26, C27, C28, C29, C3, C30, C31, C32, C4, C5, C6, C8, C9: footprint Delta_s_m_lib:C_Disc_D7.0mm_W2.5mm_P5.00mm -> Delta_sm_lib:C_Disc_D7.0mm_W2.5mm_P5.00mm
- C14: footprint Capacitor_THT:CP_Radial_D4.0mm_P2.00mm -> Delta_sm_lib:CP_Radial_D4.0mm_P2.00mm
- C15: footprint Capacitor_THT:CP_Radial_D10.0mm_P5.00mm -> Delta_sm_lib:CP_Radial_D10.0mm_P5.00mm
- D1, D10, D11, D12, D13, D14, D15, D16, D17, D18, D19, D2, D20, D21, D22, D23, D24, D25, D26, D27, D28, D29, D3, D30, D31, D4, D5, D6, D7, D8, D9: footprint Delta_s_m_lib:D_DO-35_SOD27_P10.16mm_Horizontal -> Delta_sm_lib:D_DO-35_SOD27_P10.16mm_Horizontal
- DA1, DA2: footprint Resistor_THT:R_Array_SIP10 -> Delta_sm_lib:R_Array_SIP10
- H1: footprint MountingHole:MountingHole_3mm -> Delta_sm_lib:MountingHole_3mm
- H6: footprint MountingHole:MountingHole_3.5mm -> Delta_sm_lib:MountingHole_3.5mm
- J1: footprint Delta_s_m_lib:snp59_96_female_angle_3 -> Delta_sm_lib:snp59_96_female_angle_3
- J2, J6, J7: footprint Delta_s_m_lib:DIN-7-Variable -> Delta_sm_lib:DIN-7-Variable
- J3, J4: footprint Delta_s_m_lib:DIN-5-Variable -> Delta_sm_lib:DIN-5-Variable
- J5: footprint Delta_s_m_lib:IDC-Header_2x12_P2.54mm_Vertical -> Delta_sm_lib:IDC-Header_2x12_P2.54mm_Vertical
- JP1, JP2: footprint Connector_PinHeader_2.54mm:PinHeader_1x03_P2.54mm_Vertical -> Delta_sm_lib:PinHeader_1x03_P2.54mm_Vertical
- JP3, JP4, JP5: footprint Connector_PinHeader_2.54mm:PinHeader_1x02_P2.54mm_Vertical -> Delta_sm_lib:PinHeader_1x02_P2.54mm_Vertical
- JP6: footprint Delta_s_m_lib:PinHeader_2x03_P2.54mm_Vertical -> Delta_sm_lib:PinHeader_2x03_P2.54mm_Vertical
- LS1: footprint delta:ZM-Piezo Buzzer-2207T2 -> Delta_sm_lib:ZM-Piezo Buzzer-2207T2
- Log1: footprint Symbol:KiCad-Logo2_6mm_SilkScreen -> Delta_sm_lib:KiCad-Logo2_6mm_SilkScreen
- Log2: footprint Symbol:OSHW-Logo2_14.6x12mm_SilkScreen -> Delta_sm_lib:OSHW-Logo2_14.6x12mm_SilkScreen
- Q1, Q3, Q4, Q5, Q6, Q7, Q8: footprint Delta_s_m_lib:TO-92_Inline -> Delta_sm_lib:TO-92_Inline
- R1, R10, R11, R12, R13, R14, R15, R16, R19, R20, R21, R22, R23, R24, R25, R26, R28, R30, R32, R33, R34, R35, R36, R37, R38, R39, R4, R40, R41, R45, R46, R47, R48, R49, R5, R50, R51, R52, R53, R54, R55, R56, R57, R58, R59, R6, R7, R8, R9: footprint Delta_s_m_lib:R_Axial_DIN0207_L6.3mm_D2.5mm_P10.16mm_Horizontal -> Delta_sm_lib:R_Axial_DIN0207_L6.3mm_D2.5mm_P10.16mm_Horizontal
- R2: value 430 -> 470; footprint Delta_s_m_lib:R_Axial_DIN0207_L6.3mm_D2.5mm_P10.16mm_Horizontal -> Delta_sm_lib:R_Axial_DIN0207_L6.3mm_D2.5mm_P10.16mm_Horizontal
- RV42, RV43, RV44: footprint Delta_s_m_lib:Potentiometer_Bourns_3299X_Horizontal -> Delta_sm_lib:Potentiometer_Bourns_3299X_Horizontal
- SW1: footprint Button_Switch_THT:SW_Tactile_SPST_Angled_PTS645Vx83-2LFS -> Delta_sm_lib:SW_Tactile_SPST_Angled_PTS645Vx83-2LFS
- U1, U10, U11, U12, U13, U14, U18, U19, U2, U20, U21, U28, U29, U3, U30, U39, U40, U49, U5, U50, U51, U57, U58, U64, U65, U7, U73, U74, U75, U8, U9: footprint Delta_s_m_lib:DIP-14_W7.62mm_Socket -> Delta_sm_lib:DIP-14_W7.62mm_Socket
- U15, U16, U17, U22, U23, U24, U25, U26, U27, U31, U32, U33, U34, U35, U36, U37, U38, U4, U41, U42, U43, U44, U45, U46, U47, U48, U52, U53, U54, U55, U56, U59, U6, U60, U61, U62, U63, U66: footprint Delta_s_m_lib:DIP-16_W7.62mm_Socket -> Delta_sm_lib:DIP-16_W7.62mm_Socket
- U67: footprint Delta_s_m_lib:DIP-20_W7.62mm_Socket -> Delta_sm_lib:DIP-20_W7.62mm_Socket
- U68, U72: value КР556РТ2 -> 27C512
- U69: footprint Delta_s_m_lib:DIP-40_W15.24mm_Socket -> Delta_sm_lib:DIP-40_W15.24mm_Socket
- U70, U71: footprint Delta_s_m_lib:DIP-28_W15.24mm_Socket -> Delta_sm_lib:DIP-28_W15.24mm_Socket
- Y1: footprint Delta_s_m_lib:Crystal_HC49-U_Vertical -> Delta_sm_lib:Crystal_HC49-U_Vertical
- moved R7 11.9 mm to (105.8, 101.8), turned to 180 degrees
- moved U72 1.73 mm to (336.9, 161.0)
- moved U68 1.03 mm to (288.4, 209.8)
- moved DA1 0.93 mm to (291.9, 209.7)
Connections:
- R51 pad 2: Net-(U72-В1) -> Net-(U72-D0)
- U68 pad 10: KB7 -> KBD12
- U68 pad 11: unconnected-(U68-В7-Pad11) -> KB0
- U68 pad 12: KB5 -> KB1
- U68 pad 13: KB4 -> KB2
- U68 pad 16: KB2 -> KB4
- U68 pad 17: KB1 -> KB5
- U68 pad 18: KB0 -> unconnected-(U68-D6-Pad18)
- U68 pad 19: GND -> KB7
- U68 pad 2: JOY5 -> RA13
- U68 pad 21: unconnected-(U68-А15-Pad21) -> KBD2
- U68 pad 22: RA15 -> GND
- U68 pad 23: RA13 -> RA8
- U68 pad 24: RA8 -> JOY3
- U68 pad 25: KBD2 -> JOY4
- U68 pad 26: JOY3 -> RA15
- U68 pad 27: JOY4 -> unconnected-(U68-A14-Pad27)
- U68 pad 3: JOY6 -> JOY5
- U68 pad 4: JOY7 -> JOY6
- U68 pad 5: KBD8 -> JOY7
- U68 pad 6: KBD9 -> KBD8
- U68 pad 7: KBD10 -> KBD9
- U68 pad 8: KBD11 -> KBD10
- U68 pad 9: KBD12 -> KBD11
- U72 pad 10: B22_SNP -> A8
- U72 pad 11: B28_SNP -> Net-(U72-D0)
- U72 pad 12: A28_SNP -> Net-(U67-STB)
- U72 pad 13: B29_SNP -> Net-(U66-Cp)
- U72 pad 16: Net-(U66-Cp) -> B29_SNP
- U72 pad 17: Net-(U67-STB) -> A28_SNP
- U72 pad 18: Net-(U72-В1) -> B28_SNP
- U72 pad 19: GND -> B22_SNP
- U72 pad 2: A15 -> BUSY
- U72 pad 21: unconnected-(U72-А15-Pad21) -> ЗПL
- U72 pad 22: unconnected-(U72-А14-Pad22) -> GND
- U72 pad 23: BUSY -> A1
- U72 pad 24: A1 -> ЧТL
- U72 pad 25: ЗПL -> ВУL
- U72 pad 26: ЧТL -> unconnected-(U72-A13-Pad26)
- U72 pad 27: ВУL -> unconnected-(U72-A14-Pad27)
- U72 pad 3: A14 -> A15
- U72 pad 4: A13 -> A14
- U72 pad 5: A12 -> A13
- U72 pad 6: A11 -> A12
- U72 pad 7: A10 -> A11
- U72 pad 8: A9 -> A10
- U72 pad 9: A8 -> A9
Routing:
- net GND: track 1870.9 -> 0.00 mm, vias 1 -> 0
- net +5V: track 1641.4 -> 0.00 mm
- net A15: track 418.7 -> 0.00 mm, vias 2 -> 0
- net ПРL: track 410.5 -> 0.00 mm, vias 1 -> 0
- net 7MHZ: track 409.7 -> 0.00 mm, vias 1 -> 0
- net JOY3: track 399.1 -> 0.00 mm
- net A13: track 397.3 -> 0.00 mm, vias 2 -> 0
- net JOY5: track 387.0 -> 0.00 mm, vias 1 -> 0
- net JOY4: track 383.5 -> 0.00 mm
- net A14: track 381.4 -> 0.00 mm, vias 7 -> 0
- net A11: track 377.1 -> 0.00 mm, vias 6 -> 0
- net A1: track 374.4 -> 0.00 mm, vias 4 -> 0
- net A12: track 354.2 -> 0.00 mm, vias 3 -> 0
- net A10: track 346.6 -> 0.00 mm, vias 3 -> 0
- net A8: track 343.6 -> 0.00 mm, vias 5 -> 0
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Other:
- board text added: "GND"
- board text added: "RESET"
- board text added: "БПК {dblquote}Дельта-С{dblquote} Recreation Project Version 1.2 Board Design by MadCat, 2023 https://github.com/madcatse/Delta-S-M t.me/zx_delta_s https://www.youtube.com/@MadCatSE"
- board text removed: "БПК {dblquote}Дельта-С{dblquote} Recreation Project Version 1.1 Board Design by MadCat, 2023 https://github.com/madcatse/Delta-S-M t.me/zx_delta_s https://www.youtube.com/@MadCatSE"

Commit message: Topology for version 1.2
Parts:
- added H10: MountingHole_3.5mm, Delta_sm_lib:MountingHole_3.5mm, F.Cu at (111.3, 86.7)
- added H3: MountingHole_3.2mm_M3, Delta_sm_lib:MountingHole_3.2mm_M3, F.Cu at (72.6, 75.9)
- added H4: MountingHole_3.2mm_M3, Delta_sm_lib:MountingHole_3.2mm_M3, F.Cu at (81.3, 211.0)
- added H5: MountingHole_3.2mm_M3, Delta_sm_lib:MountingHole_3.2mm_M3, F.Cu at (339.6, 78.4)
- added H6: MountingHole_3.2mm_M3, Delta_sm_lib:MountingHole_3.2mm_M3, F.Cu at (353.6, 218.7)
- added H7: MountingHole_3.5mm, Delta_sm_lib:MountingHole_3.5mm, F.Cu at (118.9, 76.8)
- added H9: MountingHole_3.2mm_M3, Delta_sm_lib:MountingHole_3.2mm_M3, F.Cu at (321.6, 86.6)
- added J10: Conn_01x06, Connector_PinHeader_2.54mm:PinHeader_1x06_P2.54mm_Vertical, F.Cu at (156.3, 77.4)
- added J11: Conn_01x06, Connector_PinHeader_2.54mm:PinHeader_1x06_P2.54mm_Vertical, F.Cu at (239.7, 77.4)
- added J12: Conn_01x04, Connector_PinHeader_2.54mm:PinHeader_1x04_P2.54mm_Vertical, F.Cu at (195.4, 77.4)
- added J13: Conn_01x02, Connector_PinHeader_2.54mm:PinHeader_1x02_P2.54mm_Vertical, F.Cu at (99.2, 84.9)
- added J14: Conn_01x02, Connector_PinHeader_2.54mm:PinHeader_1x02_P2.54mm_Vertical, F.Cu at (340.1, 136.0)
- added J9: Conn_01x06, Connector_PinHeader_2.54mm:PinHeader_1x06_P2.54mm_Vertical, F.Cu at (177.2, 77.4)
- added LS2: 1407, Delta_sm_lib:1407 Piezoelectric Passive Buzzer, F.Cu at (85.2, 87.2)
- added R3: 4.7K, Delta_sm_lib:R_Axial_DIN0207_L6.3mm_D2.5mm_P10.16mm_Horizontal, F.Cu at (336.4, 139.9)
- added SW2: SW_SPST, Delta_sm_lib:onoffswitch, F.Cu at (303.9, 76.7)
- J8: footprint Connector_PinHeader_2.54mm:PinHeader_1x04_P2.54mm_Vertical -> Delta_sm_lib:USB-C Power board
- LS1: value Speaker -> 2207
- U70: value 27C64 -> 27C256
- moved Log2 211.6 mm to (330.5, 77.6)
- moved Log1 178.0 mm to (309.4, 83.8)
- moved D1 15.3 mm to (138.7, 88.2)
- moved RV44 13.3 mm to (294.0, 80.7)
- moved C10 11.4 mm to (154.1, 95.5), turned to 180 degrees
- moved D6 7.11 mm to (138.7, 90.8)
- moved D10 7.11 mm to (138.7, 100.9)
- moved D7 7.11 mm to (138.7, 93.3)
- moved D8 7.11 mm to (138.7, 95.9)
- moved D9 7.11 mm to (138.7, 98.4)
- moved D2 7.11 mm to (126.4, 93.3)
- moved D3 7.11 mm to (126.4, 95.9)
- moved D4 7.11 mm to (126.4, 98.4)
- moved D5 7.11 mm to (126.4, 100.9)
- moved RV43 6.91 mm to (284.0, 80.7)
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- renumbered H6 to H1, H1 to H8
Connections:
- U70 pad 27: unconnected-(U70-~{PGM}-Pad27) -> Extra_A14
Routing:
- net GND: track 0.00 -> 2741.8 mm, vias 0 -> 9
- net +5V: track 0.00 -> 2418.0 mm, vias 0 -> 5
- net A14: track 0.00 -> 445.2 mm, vias 0 -> 13
- net A13: track 0.00 -> 409.7 mm, vias 0 -> 4
- net A15: track 0.00 -> 405.5 mm, vias 0 -> 5
- net ПРL: track 0.00 -> 398.8 mm, vias 0 -> 4
- net A8: track 0.00 -> 370.3 mm, vias 0 -> 9
- net A11: track 0.00 -> 364.1 mm, vias 0 -> 4
- net D0: track 0.00 -> 354.9 mm, vias 0 -> 5
- net A1: track 0.00 -> 349.5 mm, vias 0 -> 10
- net A10: track 0.00 -> 345.0 mm, vias 0 -> 3
- net 7MHZ: track 0.00 -> 336.3 mm, vias 0 -> 4
- net D4: track 0.00 -> 333.2 mm, vias 0 -> 7
- net A12: track 0.00 -> 331.4 mm, vias 0 -> 2
- net A9: track 0.00 -> 329.1 mm, vias 0 -> 2
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Other:
- board text added: "2207 Piezobuzzer"
- board text added: "27C256 (if DoubleROM is used) or 27C64 (К573РФ4)"
- board text added: "27C512 Keyboard ROM"
- board text added: "27C512 Printer ROM (Optional)"
- board text added: "27C64 (К573РФ4) Do not place if 27C256 is used"
- board text added: "Blue"
- board text added: "Delta S-M {dblquote}Дельта-С{dblquote} Recreation Project Version 1.2"
- board text added: "Green"
- board text added: "ROM SWITCH"
- board text added: "Red"
- board text removed: "27C128 or 27C64 (К573РФ4)"
- board text removed: "27C64 (К573РФ4)"
- board text removed: "КР556РТ2"
