File: delta48m.kicad_pcb (KiCad board)
At the start: 2 copper layers, 287 x 150 mm, 236 parts, among them J1 SNP, J10 Conn_01x06, J11 Conn_01x06, J12 Conn_01x04, J13 Conn_01x02, J14 Conn_01x02, J2 DIN-7 Video, J3 DIN-5 Audio, J4 DIN-5 Power, J5 Keyboard Connector, J6 Joystick 1, J7 Joystick 2, J8 USB_PORT, J9 Conn_01x06, Q1 BC547B, Q3 BC547B, Q4 BC547B, Q5 BC547B, Q6 BC547B, Q7 BC547B, Q8 BC547B, SW1 Reset button, SW2 SW_SPST, U1 SN74ALS08 (КР1533ЛИ1), U10 SN74ALS08 (КР1533ЛИ1), U11 IN74ALS00N (КР1533ЛА3), U12 IN74ALS02N (КР1533ЛЕ1), U13 SN74ALS10 (КР1533ЛА4), U14 SN74ALS86N (КР1533ЛП5), U15 CD4520АN (К561ИЕ10A), U16 SN74ALS257N_(КР1533КП11А), U17 CD4520АN (К561ИЕ10A), U18 CD4011 (К561ЛА7), U19 SN74ALS04 (КР1533ЛН1), U2 SN74ALS04 (КР1533ЛН1), U20 SN74ALS74AN (КР1533ТМ2), U21 SN74ALS04 (КР1533ЛН1), U22 74LS257 (КР1533КП11А), U23 SN74ALS253N (КР1533КП12), U24 SN74ALS253N (КР1533КП12), U25 74LS257 (КР1533КП11А), U26 SN74ALS253N (КР1533КП12), U27 SN74ALS253N (КР1533КП12), U28 IN74ALS32N (КР1533ЛЛ1), U29 IN74ALS32N (КР1533ЛЛ1), U3 SN74ALS74AN (КР1533ТМ2), U30 IN74ALS02N (КР1533ЛЕ1), U31 RU5D1, U32 RU5D1, U33 RU5D1, U34 RU5D1, U35 RU5D1, U36 RU5D1, U37 RU5D1, U38 RU5D1, U39 IN74ALS32N (КР1533ЛЛ1), U4 SN74ALS193N_(КР1533ИЕ7), U40 IN74ALS00N (КР1533ЛА3), U41 2118 (КР565РУ6), U42 2118 (КР565РУ6), U43 2118 (КР565РУ6), U44 2118 (КР565РУ6), U45 2118 (КР565РУ6), U46 2118 (КР565РУ6), U47 2118 (КР565РУ6), U48 2118 (КР565РУ6), U49 SN74ALS04 (КР1533ЛН1), U5 СD4013АN_(К561ТМ2), U50 SN74ALS86N (КР1533ЛП5), U51 SN7486N (К155ЛП5), U52 SN74ALS175N (КР1533ТМ8), U53 SN74ALS153N (КР1533КП2), U54 SN74ALS298N (КР1533КП13), U55 74LS257 (КР1533КП11А), U56 SN74ALS175N (КР1533ТМ8), U57 SN74LS295N_(К555ИР16), U58 SN74LS295N_(К555ИР16), U59 SN74ALS175N (КР1533ТМ8), U6 CD4015A (К561ИР2), U60 SN74ALS153N (КР1533КП2)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

Commit message: Gerbers update
Parts:
- moved Log2 279.0 mm to (81.0, 202.2)
- moved Log1 52.6 mm to (256.8, 85.4)
Other:
- board text added: "Short 1-2 for 2x 27C64 Short 2-3 for 1x 27C128/256"
- board text removed: "Short 1-2 for 2x 27C64 Short 2-3 for 1x 27C128"
Changed lines of the file:
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@@
     (property "ki_keywords" "R res resistor")
     (attr through_hole)
-    (fp_text reference "R56" (at 4.699 -2.54 270) (layer "F.SilkS")
+    (fp_text reference "R56" (at 7.587 -2.245 270) (layer "F.SilkS")
         (effects (font (size 1 1) (thickness 0.15)))
     )
@@
   )
   (footprint "Delta_sm_lib:KiCad-Logo2_6mm_SilkScreen" (layer "F.Cu")
-    (at 309.3778 83.7628)
+    (at 256.842514 85.404848)
     (descr "KiCad Logo")
     (tags "Logo KiCad")
@@
   )
   (footprint "Delta_sm_lib:OSHW-Logo2_14.6x12mm_SilkScreen" (layer "F.Cu")
-    (at 330.536 77.616)
+    (at 80.95 202.2)
     (descr "Open Source Hardware Symbol")
     (tags "Logo Symbol OSHW")
@@
     (property "ki_keywords" "TTL and2")
     (attr through_hole)
-    (fp_text reference "U74" (at -2.5968 7.7526 270) (layer "F.SilkS")
+    (fp_text reference "U74" (at -2.472 3.987 270) (layer "F.SilkS")
         (effects (font (size 1 1) (thickness 0.15)))
     )
@@
     (effects (font (size 0.75 0.75) (thickness 0.15)))
   )
-  (gr_text "Short 1-2 for 2x 27C64\nShort 2-3 for 1x 27C128\n" (at 341.4268 210.2104) (layer "F.SilkS" knockout)
+  (gr_text "Short 1-2 for 2x 27C64\nShort 2-3 for 1x 27C128/256\n" (at 341.45 209) (layer "F.SilkS" knockout)
     (effects (font (size 0.75 0.75) (thickness 0.15)))
   )
@@
   (segment locked (start 284.0023 75.6348) (end 284.0023 71.7749) (width 0.4) (layer "B.Cu") (net 3))
   (segment (start 298.1167 163.8712) (end 298.1167 173.7183) (width 0.4) (layer "B.Cu") (net 3))
-  (segment (start 351.207 185.769) (end 351.2072 185.7692) (width 0.4) (layer "B.Cu") (net 3))
   (segment (start 280.3652 120.4468) (end 280.3652 117.9445) (width 0.4) (layer "B.Cu") (net 3))
   (segment (start 212.612 155.9154) (end 212.612 155.3145) (width 0.4) (layer "B.Cu") (net 3))
@@
   (segment (start 141.0593 199.0803) (end 143.387 201.408) (width 0.4) (layer "B.Cu") (net 3))
   (segment locked (start 95.1234 90.7442) (end 96.9586 92.5794) (width 0.4) (layer "B.Cu") (net 3))
-  (segment (start 308.1074 75.3527) (end 308.1072 75.3525) (width 0.4) (layer "B.Cu") (net 3))
   (segment (start 101.1791 147.3673) (end 100.3389 146.5271) (width 0.4) (layer "B.Cu") (net 3))
   (segment (start 143.397 136.8833) (end 143.397 136.2824) (width 0.4) (layer "B.Cu") (net 3))

Commit message: Fixes
Parts:
- added C7: 4.7µF 16V, Delta_sm_lib:CP_Radial_D4.0mm_P2.00mm, F.Cu at (170.7, 95.7)
- added R17: 220, Delta_sm_lib:R_Axial_DIN0207_L6.3mm_D2.5mm_P10.16mm_Horizontal, F.Cu at (248.5, 90.6)
- added R18: 220, Delta_sm_lib:R_Axial_DIN0207_L6.3mm_D2.5mm_P10.16mm_Horizontal, F.Cu at (245.3, 90.6)
- added R27: 220, Delta_sm_lib:R_Axial_DIN0207_L6.3mm_D2.5mm_P10.16mm_Horizontal, F.Cu at (251.6, 90.6)
- moved Log1 182.2 mm to (78.9, 124.8)
Connections:
- D11 pad 2: YB -> YR
- D12 pad 2: YG -> YB
- D13 pad 2: YR -> YG
- J11 pad 4: BLUE -> GREEN
- J11 pad 5: GREEN -> BLUE
- J13 pad 1: AUDIO -> Net-(J13-Pin_1)
- J2 pad 4: BLUE -> GREEN
- J2 pad 5: GREEN -> BLUE
- J2 pad 6: unconnected-(J2-Pad6) -> AUDIO
- JP6 pad 2: YR -> YG
- JP6 pad 4: YB -> YR
- JP6 pad 6: YG -> YB
- LS1 pad 1: AUDIO -> Net-(J13-Pin_1)
- LS2 pad 1: AUDIO -> Net-(J13-Pin_1)
- Q1 pad 3: AUDIO -> Net-(J13-Pin_1)
- Q4 pad 3: BLUE -> Net-(Q4-E)
- Q5 pad 3: RED -> Net-(Q5-E)
- Q6 pad 3: GREEN -> Net-(Q6-E)
- R26 pad 1: BLUE -> RED
- R28 pad 1: RED -> GREEN
- R30 pad 1: GREEN -> BLUE
- R32 pad 2: YB -> YR
- R36 pad 2: YG -> YB
- R39 pad 2: YR -> YG
- R7 pad 1: AUDIO -> Net-(J13-Pin_1)
- RV42 pad 1: YG -> YB
- RV43 pad 1: YB -> YR
- RV44 pad 1: YR -> YG
Routing:
- net Net-(J13-Pin_1): track 0.00 -> 111.3 mm, vias 0 -> 3
- net AUDIO: track 148.1 -> 71.9 mm, vias 0 -> 2
- net Net-(Q5-E): track 0.00 -> 30.2 mm, vias 0 -> 3
- net Net-(Q4-E): track 0.00 -> 26.7 mm, vias 0 -> 1
- net BLUE: track 30.6 -> 52.8 mm, vias 0 -> 2
- net YB: track 56.5 -> 40.5 mm, vias 1 -> 0
- net GREEN: track 37.8 -> 52.3 mm, vias 1 -> 3
- net RED: track 33.8 -> 48.1 mm
- net Net-(Q6-E): track 0.00 -> 12.6 mm, vias 0 -> 1
- net YR: track 45.3 -> 56.5 mm, vias 0 -> 1
- net YG: track 40.5 -> 45.3 mm
- net Net-(Q4-B): track 64.8 -> 67.6 mm
- net Left1: track 58.3 -> 59.6 mm
- net Contact2: track 301.2 -> 302.5 mm
- net Net-(Q6-B): track 39.6 -> 40.6 mm
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Other:
- board text added: "+5"
- board text added: "4 GREEN"
- board text added: "5 BLUE"
- board text added: "B"
- board text added: "G"
- board text added: "R"
- board text added: "S"
- board text removed: "4 BLUE"
- board text removed: "GREEN"

Commit message: Gerbers 05042024
Other:
- board text added: "27C64 (К573РФ4) Do not place if 27C128/256 is used"
- board text added: "27С128(27C256 if DoubleROM is used) or 27C64 (К573РФ4)"
- board text removed: "27C64 (К573РФ4) Do not place if 27C256 is used"
Changed lines of the file:
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@@
     (effects (font (size 0.75 0.75) (thickness 0.15)))
   )
-  (gr_text "27C256 \n(if DoubleROM is used)\nor\n27C64 (К573РФ4)" (at 313.0354 126.8412) (layer "F.SilkS")
+  (gr_text "27С128(27C256 if \nDoubleROM is used)\nor\n27C64 (К573РФ4)" (at 313.0354 126.9174) (layer "F.SilkS")
     (effects (font (size 2 2) (thickness 0.3)))
   )
@@
     (effects (font (size 0.75 0.75) (thickness 0.15)))
   )
-  (gr_text "27C64 (К573РФ4)\nDo not place if\n27C256 is used" (at 314.075 147.346) (layer "F.SilkS")
+  (gr_text "27C64 (К573РФ4)\nDo not place if\n27C128/256 is used" (at 314.075 147.346) (layer "F.SilkS")
     (effects (font (size 2 2) (thickness 0.3)))
   )

Commit message: Gerbers 08042024
Other:
- board text added: "БПК {dblquote}Дельта-С{dblquote} Recreation Project Version 1.2 Board Design by MadCat, 2023-24 https://github.com/madcatse/Delta-S-M t.me/zx_delta_s https://www.youtube.com/@MadCatSE"
- board text removed: "БПК {dblquote}Дельта-С{dblquote} Recreation Project Version 1.2 Board Design by MadCat, 2023 https://github.com/madcatse/Delta-S-M t.me/zx_delta_s https://www.youtube.com/@MadCatSE"
Changed lines of the file:
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@@
   )
   (footprint "Delta_sm_lib:R_Axial_DIN0207_L6.3mm_D2.5mm_P10.16mm_Horizontal" (layer "F.Cu")
-    (at 245.319 90.6462 90)
+    (at 245.319 90.6208 90)
     (descr "Resistor, Axial_DIN0207 series, Axial, Horizontal, pin pitch=10.16mm, 0.25W = 1/4W, length*diameter=6.3*2.5mm^2, http://cdn-reichelt.de/documents/datenblatt/B400/1_4W%23YAG.pdf")
     (tags "Resistor Axial_DIN0207 series Axial Horizontal pin pitch 10.16mm 0.25W = 1/4W length 6.3mm diameter 2.5mm")
@@
   )
   (footprint "Delta_sm_lib:R_Axial_DIN0207_L6.3mm_D2.5mm_P10.16mm_Horizontal" (layer "F.Cu")
-    (at 248.5067 90.6462 90)
+    (at 248.4686 90.6208 90)
     (descr "Resistor, Axial_DIN0207 series, Axial, Horizontal, pin pitch=10.16mm, 0.25W = 1/4W, length*diameter=6.3*2.5mm^2, http://cdn-reichelt.de/documents/datenblatt/B400/1_4W%23YAG.pdf")
     (tags "Resistor Axial_DIN0207 series Axial Horizontal pin pitch 10.16mm 0.25W = 1/4W length 6.3mm diameter 2.5mm")
@@
     (effects (font (size 1 1) (thickness 0.15)) (justify mirror))
   )
-  (gr_text "БПК {dblquote}Дельта-С{dblquote}\nRecreation Project\nVersion 1.2\nBoard Design by MadCat, 2023\nhttps://github.com/madcatse/Delta-S-M\nt.me/zx_delta_s\nhttps://www.youtube.com/@MadCatSE" (at 293.0964 89.7572) (layer "B.SilkS")
+  (gr_text "БПК {dblquote}Дельта-С{dblquote}\nRecreation Project\nVersion 1.2\nBoard Design by MadCat, 2023-24\nhttps://github.com/madcatse/Delta-S-M\nt.me/zx_delta_s\nhttps://www.youtube.com/@MadCatSE" (at 293.0964 89.7572) (layer "B.SilkS")
     (effects (font (size 1.5 1.5) (thickness 0.1875)) (justify mirror))
   )
