File: logic.kicad_sch (KiCad schematic)
At the start: 42 parts, among them U1 SN74ALS08 (КР1533ЛИ1), U10 SN74ALS08 (КР1533ЛИ1), U11 IN74ALS00N (КР1533ЛА3), U12 IN74ALS02N (КР1533ЛЕ1), U13 SN74ALS10 (КР1533ЛА4), U14 SN74ALS86N (КР1533ЛП5), U15 CD4520АN_(К561ИЕ10), U16 SN74ALS257N_(КР1533КП11А), U17 CD4520АN_(К561ИЕ10), U18 CD4011 (К561ЛА7)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

Commit message: 28th march ver2
Parts:
- added unit 1 of U49
Connections:
- net ТАКТ: now also U49.2; no longer U49.4
- net at U49.3: no longer U10.3
- net at U13.12, U3.12 (D): now also U1.12; no longer U1.13
- net at R8.1, U14.8: now also U1.13; no longer U1.12
- new net: U10.3, U49.1
- no-connect marks 31 -> 33
Changed lines of the file:
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@@
   (no_connect (at 108.585 -245.745))
   (no_connect (at 161.29 52.07))
+  (no_connect (at 176.53 -215.265))
   (no_connect (at 248.285 183.515))
   (no_connect (at 158.75 -214.63))
@@
   (no_connect (at 104.14 126.365))
   (no_connect (at 142.875 -266.7))
+  (no_connect (at 191.77 -215.265))
   (no_connect (at 161.29 49.53))
   (no_connect (at 104.14 128.905))
@@
     (pin "1")
   )
+  (symbol (lib_id "74xx:74LS08") (at 234.95 128.905 0) (mirror x) (unit 4)
+    (in_bom yes) (on_board yes)
+    (property "Reference" "U1" (id 0) (at 234.95 128.905 0))
+    (property "Value" "SN74ALS08 (КР1533ЛИ1)" (id 1) (at 234.4166 122.3551 0))
+    (property "Footprint" "Package_DIP:DIP-14_W7.62mm_Socket" (id 2) (at 234.95 128.905 0)
+      (effects (font (size 1.27 1.27)) hide)
+    )
+    (property "Datasheet" "http://www.ti.com/lit/gpn/sn74LS08" (id 3) (at 234.95 128.905 0)
+      (effects (font (size 1.27 1.27)) hide)
+    )
+    (pin "1")
+    (pin "2")
+    (pin "3")
+    (pin "4")
+    (pin "5")
+    (pin "6")
+    (pin "10")
+    (pin "8")
+    (pin "9")
+    (pin "11")
+    (pin "12")
+    (pin "13")
+    (pin "14")
+    (pin "7")
+  )
   (symbol (lib_id "74xx:74LS32") (at 116.84 -214.63 0) (unit 4)
     (in_bom yes) (on_board yes) (fields_autoplaced)
@@
     (pin "7")
   )
-  (symbol (lib_id "74xx:74LS04") (at 312.42 95.885 0) (unit 2)
+  (symbol (lib_id "74xx:74LS08") (at 177.165 149.225 0) (mirror x) (unit 2)
     (in_bom yes) (on_board yes)
-    (property "Reference" "U49" (id 0) (at 311.785 95.885 0))
-    (property "Value" "SN74ALS04 (КР1533ЛН1)" (id 1) (at 312.42 100.965 0))
-    (property "Footprint" "Package_DIP:DIP-14_W7.62mm_Socket" (id 2) (at 312.42 95.885 0)
+    (property "Reference" "U10" (id 0) (at 177.8 149.225 0))
+    (property "Value" "SN74ALS08 (КР1533ЛИ1)" (id 1) (at 175.895 141.605 0))
+    (property "Footprint" "Package_DIP:DIP-14_W7.62mm_Socket" (id 2) (at 177.165 149.225 0)
       (effects (font (size 1.27 1.27)) hide)
     )
-    (property "Datasheet" "http://www.ti.com/lit/gpn/sn74LS04" (id 3) (at 312.42 95.885 0)
+    (property "Datasheet" "http://www.ti.com/lit/gpn/sn74LS08" (id 3) (at 177.165 149.225 0)
       (effects (font (size 1.27 1.27)) hide)
     )
@@
     (pin "5")
     (pin "6")
+    (pin "10")
     (pin "8")
     (pin "9")
-    (pin "10")
     (pin "11")
     (pin "12")
@@
     (pin "7")
   )
-  (symbol (lib_id "74xx:74LS08") (at 177.165 149.225 0) (mirror x) (unit 2)
+  (symbol (lib_id "4xx:4001") (at 266.065 177.165 0) (mirror x) (unit 1)
     (in_bom yes) (on_board yes)
-    (property "Reference" "U10" (id 0) (at 177.8 149.225 0))
-    (property "Value" "SN74ALS08 (КР1533ЛИ1)" (id 1) (at 175.895 141.605 0))
-    (property "Footprint" "Package_DIP:DIP-14_W7.62mm_Socket" (id 2) (at 177.165 149.225 0)
+    (property "Reference" "U9" (id 0) (at 266.065 177.165 0))
+    (property "Value" "СD4001АN (К561ЛЕ5)" (id 1) (at 266.065 172.085 0))
+    (property "Footprint" "Package_DIP:DIP-14_W7.62mm_Socket" (id 2) (at 266.065 177.165 0)
       (effects (font (size 1.27 1.27)) hide)
     )
-    (property "Datasheet" "http://www.ti.com/lit/gpn/sn74LS08" (id 3) (at 177.165 149.225 0)
+    (property "Datasheet" "http://www.intersil.com/content/dam/Intersil/documents/cd40/cd4000bms-01bms-02bms-25bms.pdf" (id 3) (at 266.065 177.165 0)
       (effects (font (size 1.27 1.27)) hide)
     )
@@
     (pin "7")
   )
-  (symbol (lib_id "4xx:4001") (at 266.065 177.165 0) (mirror x) (unit 1)
+  (symbol (lib_id "74xx:74LS04") (at 87.63 156.21 0) (unit 1)
     (in_bom yes) (on_board yes)
-    (property "Reference" "U9" (id 0) (at 266.065 177.165 0))
-    (property "Value" "СD4001АN (К561ЛЕ5)" (id 1) (at 266.065 172.085 0))
-    (property "Footprint" "Package_DIP:DIP-14_W7.62mm_Socket" (id 2) (at 266.065 177.165 0)
+    (property "Reference" "U7" (id 0) (at 86.995 156.21 0))
+    (property "Value" "SN74ALS04 (КР1533ЛН1)" (id 1) (at 87.63 151.13 0))
+    (property "Footprint" "Package_DIP:DIP-14_W7.62mm_Socket" (id 2) (at 87.63 156.21 0)
       (effects (font (size 1.27 1.27)) hide)
     )
-    (property "Datasheet" "http://www.intersil.com/content/dam/Intersil/documents/cd40/cd4000bms-01bms-02bms-25bms.pdf" (id 3) (at 266.065 177.165 0)
+    (property "Datasheet" "http://www.ti.com/lit/gpn/sn74LS04" (id 3) (at 87.63 156.21 0)
       (effects (font (size 1.27 1.27)) hide)
     )
@@
     (pin "5")
     (pin "6")
-    (pin "10")
     (pin "8")
     (pin "9")
+    (pin "10")
     (pin "11")
     (pin "12")
@@
     (pin "7")
   )
-  (symbol (lib_id "74xx:74LS04") (at 87.63 156.21 0) (unit 1)
+  (symbol (lib_id "74xx:74LS04") (at 184.15 -215.265 0) (unit 2)
     (in_bom yes) (on_board yes)
-    (property "Reference" "U7" (id 0) (at 86.995 156.21 0))
-    (property "Value" "SN74ALS04 (КР1533ЛН1)" (id 1) (at 87.63 151.13 0))
-    (property "Footprint" "Package_DIP:DIP-14_W7.62mm_Socket" (id 2) (at 87.63 156.21 0)
+    (property "Reference" "U49" (id 0) (at 183.515 -215.265 0))
+    (property "Value" "SN74ALS04 (КР1533ЛН1)" (id 1) (at 184.15 -210.185 0))
+    (property "Footprint" "Package_DIP:DIP-14_W7.62mm_Socket" (id 2) (at 184.15 -215.265 0)
       (effects (font (size 1.27 1.27)) hide)
     )
-    (property "Datasheet" "http://www.ti.com/lit/gpn/sn74LS04" (id 3) (at 87.63 156.21 0)
+    (property "Datasheet" "http://www.ti.com/lit/gpn/sn74LS04" (id 3) (at 184.15 -215.265 0)
       (effects (font (size 1.27 1.27)) hide)
     )
@@
     (pin "1")
   )
+  (symbol (lib_id "74xx:74LS04") (at 312.42 95.885 0) (unit 1)
+    (in_bom yes) (on_board yes)
+    (property "Reference" "U49" (id 0) (at 311.785 95.885 0))
+    (property "Value" "SN74ALS04 (КР1533ЛН1)" (id 1) (at 312.42 88.9 0))
+    (property "Footprint" "Package_DIP:DIP-14_W7.62mm_Socket" (id 2) (at 312.42 95.885 0)
+      (effects (font (size 1.27 1.27)) hide)
+    )
+    (property "Datasheet" "http://www.ti.com/lit/gpn/sn74LS04" (id 3) (at 312.42 95.885 0)
+      (effects (font (size 1.27 1.27)) hide)
+    )
+    (pin "1")
+    (pin "2")
+    (pin "3")
+    (pin "4")
+    (pin "5")
+    (pin "6")
+    (pin "8")
+    (pin "9")
+    (pin "10")
+    (pin "11")
+    (pin "12")
+    (pin "13")
+    (pin "14")
+    (pin "7")
+  )
   (symbol (lib_id "74xx:74LS08") (at 290.195 95.885 0) (mirror x) (unit 1)
     (in_bom yes) (on_board yes)
@@
       (effects (font (size 1.27 1.27)) hide)
     )
-    (pin "1")
-    (pin "2")
-    (pin "3")
-    (pin "4")
-    (pin "5")
-    (pin "6")
-    (pin "10")
-    (pin "8")
-    (pin "9")
-    (pin "11")
-    (pin "12")
-    (pin "13")
-    (pin "14")
-    (pin "7")
-  )
-  (symbol (lib_id "74xx:74LS08") (at 234.95 128.905 0) (unit 4)
-    (in_bom yes) (on_board yes)
-    (property "Reference" "U1" (id 0) (at 234.95 128.905 0))
-    (property "Value" "SN74ALS08 (КР1533ЛИ1)" (id 1) (at 234.95 121.92 0))
-    (property "Footprint" "Package_DIP:DIP-14_W7.62mm_Socket" (id 2) (at 234.95 128.905 0)
-      (effects (font (size 1.27 1.27)) hide)
-    )
-    (property "Datasheet" "http://www.ti.com/lit/gpn/sn74LS08" (id 3) (at 234.95 128.905 0)
-      (effects (font (size 1.27 1.27)) hide)
-    )

Commit message: 29th march 2023 Update 1
Connections:
- net CT9: now also U16.2 (I0a), U17.6 (Q4), U18.6; no longer U16.13 (I1c), U16.5 (I0b), U17.5 (Q3), U18.5
- new net: U16.13 (I1c), U16.5 (I0b), U17.5 (Q3), U18.5
Changed lines of the file:
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@@
   (junction (at 128.905 53.34) (diameter 0) (color 0 0 0 0)
   )
+  (junction (at 147.955 232.41) (diameter 0) (color 0 0 0 0)
+  )
   (junction (at 105.41 81.28) (diameter 0) (color 0 0 0 0)
   )
@@
   )
   (junction (at 163.83 42.545) (diameter 0) (color 0 0 0 0)
-  )
-  (junction (at 161.29 213.995) (diameter 0) (color 0 0 0 0)
   )
   (junction (at 99.695 43.18) (diameter 0) (color 0 0 0 0)
@@
     (stroke (width 0) (type default) (color 0 0 0 0))
   )
+  (wire (pts (xy 147.955 232.41) (xy 141.605 232.41))
+    (stroke (width 0) (type default) (color 0 0 0 0))
+  )
   (wire (pts (xy 206.375 42.545) (xy 206.375 47.625))
     (stroke (width 0) (type default) (color 0 0 0 0))
@@
   )
   (wire (pts (xy 323.215 95.885) (xy 326.39 95.885))
-    (stroke (width 0) (type default) (color 0 0 0 0))
-  )
-  (wire (pts (xy 161.29 213.995) (xy 167.64 213.995))
     (stroke (width 0) (type default) (color 0 0 0 0))
   )
@@
     )
   )
-  (global_label "CT9" (shape input) (at 167.64 213.995 0) (fields_autoplaced)
-    (effects (font (size 1.27 1.27)) (justify left))
-    (property "Intersheet References" "${INTERSHEET_REFS}" (id 0) (at 173.5002 213.9156 0)
-      (effects (font (size 1.27 1.27)) (justify left) hide)
-    )
-  )
   (global_label "CT9" (shape input) (at 299.085 123.825 180) (fields_autoplaced)
     (effects (font (size 1.27 1.27)) (justify right))
@@
     )
   )
+  (global_label "CT9" (shape input) (at 141.605 232.41 180) (fields_autoplaced)
+    (effects (font (size 1.27 1.27)) (justify right))
+    (property "Intersheet References" "${INTERSHEET_REFS}" (id 0) (at 135.7448 232.4894 0)
+      (effects (font (size 1.27 1.27)) (justify right) hide)
+    )
+  )

Commit message: March 31st final update (for today)
Parts:
- U15, U17: value CD4520АN_(К561ИЕ10) -> CD4520АN (К561ИЕ10A)
Changed lines of the file:
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@@
       (effects (font (size 1.27 1.27)) (justify left))
     )
-    (property "Value" "CD4520АN_(К561ИЕ10)" (id 1) (at 87.63 -166.3701 0)
+    (property "Value" "CD4520АN (К561ИЕ10A)" (id 1) (at 87.63 -166.3701 0)
       (effects (font (size 1.27 1.27)) (justify left))
     )
@@
     (in_bom yes) (on_board yes)
     (property "Reference" "U17" (id 0) (at 135.255 208.915 0))
-    (property "Value" "CD4520АN_(К561ИЕ10)" (id 1) (at 135.255 204.47 0))
+    (property "Value" "CD4520АN (К561ИЕ10A)" (id 1) (at 135.255 204.47 0))
     (property "Footprint" "Package_DIP:DIP-16_W7.62mm_Socket" (id 2) (at 135.255 222.885 0)
       (effects (font (size 1.27 1.27)) hide)
@@
     (in_bom yes) (on_board yes)
     (property "Reference" "U15" (id 0) (at 52.705 81.28 0))
-    (property "Value" "CD4520АN_(К561ИЕ10)" (id 1) (at 52.705 76.2 0))
+    (property "Value" "CD4520АN (К561ИЕ10A)" (id 1) (at 52.705 76.2 0))
     (property "Footprint" "Package_DIP:DIP-16_W7.62mm_Socket" (id 2) (at 52.705 95.25 0)
       (effects (font (size 1.27 1.27)) hide)
@@
     (in_bom yes) (on_board yes)
     (property "Reference" "U17" (id 0) (at 102.87 186.055 0))
-    (property "Value" "CD4520АN_(К561ИЕ10)" (id 1) (at 102.87 180.975 0))
+    (property "Value" "CD4520АN (К561ИЕ10A)" (id 1) (at 102.87 180.975 0))
     (property "Footprint" "Package_DIP:DIP-16_W7.62mm_Socket" (id 2) (at 102.87 200.025 0)
       (effects (font (size 1.27 1.27)) hide)
