File: logic.kicad_sch (KiCad schematic)
At the start: 42 parts, among them U1 SN74ALS08 (КР1533ЛИ1), U10 SN74ALS08 (КР1533ЛИ1), U11 IN74ALS00N (КР1533ЛА3), U12 IN74ALS02N (КР1533ЛЕ1), U13 SN74ALS10 (КР1533ЛА4), U14 SN74ALS86N (КР1533ЛП5), U15 CD4520АN (К561ИЕ10A), U16 SN74ALS257N_(КР1533КП11А), U17 CD4520АN (К561ИЕ10A), U18 CD4011 (К561ЛА7)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

Commit message: Version 1.0 schematics and PCB complete
Parts:
- C1, C12, C3, C32, C4, C5, C6, C8: symbol Device:C -> Delta_s_m_Lib:C
- R1, R10, R13, R15, R19, R2, R4, R5, R6, R8, R9: symbol Device:R -> Delta_s_m_Lib:R
- U1, U10: symbol 74xx:74LS08 -> Delta_s_m_Lib:74LS08
- U11: symbol 74xx:74LS00 -> Delta_s_m_Lib:74LS00
- U12: symbol 74xx:74LS02 -> Delta_s_m_Lib:74LS02
- U13: symbol 74xx:74LS10 -> Delta_s_m_Lib:74LS10_1
- U13: symbol 74xx:74LS10 -> Delta_s_m_Lib:74LS10
- U13: symbol 74xx:74LS10 -> Delta_s_m_Lib:74LS10_2
- U14: symbol 74xx:74LS86 -> Delta_s_m_Lib:74LS86
- U15, U17: symbol w_connectors:CD4520АN_(К561ИЕ10) -> Delta_s_m_Lib:CD4520АN_(К561ИЕ10)
- U16: symbol w_connectors:SN74ALS257N_(КР1533КП11А) -> Delta_s_m_Lib:SN74ALS257N_(КР1533КП11А)
- U18: symbol 4xx:4011 -> Delta_s_m_Lib:4011
- U19, U2, U49, U7: symbol 74xx:74LS04 -> Delta_s_m_Lib:74LS04
- U20: symbol 74xx:74LS74 -> Delta_s_m_Lib:74LS74_1
- U20, U3: symbol 74xx:74LS74 -> Delta_s_m_Lib:74LS74
- U28: symbol 74xx:74LS32 -> Delta_s_m_Lib:74LS32
- U4: symbol w_connectors:SN74ALS193N_(КР1533ИЕ7) -> Delta_s_m_Lib:SN74ALS193N_(КР1533ИЕ7)
- U5: symbol w_connectors:СD4013АN_(К561ТМ2) -> Delta_s_m_Lib:СD4013АN_(К561ТМ2)
- U6: symbol 4xxx_IEEE:4015 -> Delta_s_m_Lib:4015
- U6: symbol 4xxx_IEEE:4015 -> Delta_s_m_Lib:4015_1
- U8, U9: symbol 4xx:4001 -> Delta_s_m_Lib:4001
- Y1: symbol Device:Crystal -> Delta_s_m_Lib:Crystal

Commit message: Version 1.2 update
Parts:
- C1, C12, C3, C32, C4, C5, C6, C8: footprint Capacitor_THT:C_Disc_D7.0mm_W2.5mm_P5.00mm -> Delta_sm_lib:C_Disc_D7.0mm_W2.5mm_P5.00mm
- R1, R10, R13, R15, R19, R4, R5, R6, R8, R9: footprint Resistor_THT:R_Axial_DIN0207_L6.3mm_D2.5mm_P10.16mm_Horizontal -> Delta_sm_lib:R_Axial_DIN0207_L6.3mm_D2.5mm_P10.16mm_Horizontal
- R2: value 430 -> 470; footprint Resistor_THT:R_Axial_DIN0207_L6.3mm_D2.5mm_P10.16mm_Horizontal -> Delta_sm_lib:R_Axial_DIN0207_L6.3mm_D2.5mm_P10.16mm_Horizontal
- U1, U10, U11, U12, U13, U14, U18, U19, U2, U20, U28, U3, U49, U5, U7, U8, U9: footprint Package_DIP:DIP-14_W7.62mm_Socket -> Delta_sm_lib:DIP-14_W7.62mm_Socket
- U15, U16, U17, U4, U6: footprint Package_DIP:DIP-16_W7.62mm_Socket -> Delta_sm_lib:DIP-16_W7.62mm_Socket
- Y1: footprint Crystal:Crystal_HC49-U_Vertical -> Delta_sm_lib:Crystal_HC49-U_Vertical
