File: logic2.kicad_sch (KiCad schematic)
At the start: 45 parts, among them U12 IN74ALS02N (КР1533ЛЕ1), U14 SN74ALS86N (КР1533ЛП5), U15 CD4520АN_(К561ИЕ10), U21 SN74ALS14 (КР1533ТЛ2), U29 IN74ALS32N (КР1533ЛЛ1), U30 IN74ALS02N (КР1533ЛЕ1), U40 IN74ALS00N (КР1533ЛА3), U49 SN74ALS04 (КР1533ЛН1), U50 SN74ALS86N (КР1533ЛП5), U51 SN7486N (К155ЛП5)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

Commit message: March 26th update
Parts:
- U12, U14, U21, U29, U30, U40, U49, U50, U51, U57, U58, U64, U65: footprint Package_DIP:DIP-14_W7.62mm_Socket_LongPads -> Package_DIP:DIP-14_W7.62mm_Socket
- U15, U52, U53, U54, U55, U56, U59, U60, U61, U62, U63: footprint Package_DIP:DIP-16_W7.62mm_Socket_LongPads -> Package_DIP:DIP-16_W7.62mm_Socket

Commit message: 28th march ver2
Parts:
- removed unit 1 of U49
Connections:
- no-connect marks 61 -> 59
Changed lines of the file:
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@@
   )
   (no_connect (at 768.35 175.895))
-  (no_connect (at 720.09 206.375))
   (no_connect (at 193.675 102.235))
   (no_connect (at 783.59 206.375))
@@
   (no_connect (at 297.18 191.77))
   (no_connect (at 127.635 98.425))
-  (no_connect (at 704.85 206.375))
   (no_connect (at 127.635 40.64))
   (no_connect (at 127.635 35.56))
@@
     (pin "1")
   )
-  (symbol (lib_id "74xx:74LS04") (at 712.47 206.375 0) (unit 1)
-    (in_bom yes) (on_board yes)
-    (property "Reference" "U49" (id 0) (at 711.835 206.375 0))
-    (property "Value" "SN74ALS04 (КР1533ЛН1)" (id 1) (at 712.47 199.39 0))
-    (property "Footprint" "Package_DIP:DIP-14_W7.62mm_Socket" (id 2) (at 712.47 206.375 0)
-      (effects (font (size 1.27 1.27)) hide)
-    )
-    (property "Datasheet" "http://www.ti.com/lit/gpn/sn74LS04" (id 3) (at 712.47 206.375 0)
-      (effects (font (size 1.27 1.27)) hide)
-    )
-    (pin "1")
-    (pin "2")
-    (pin "3")
-    (pin "4")
-    (pin "5")
-    (pin "6")
-    (pin "8")
-    (pin "9")
-    (pin "10")
-    (pin "11")
-    (pin "12")
-    (pin "13")
-    (pin "14")
-    (pin "7")
-  )
   (symbol (lib_name "74LS257_1") (lib_id "74xx:74LS257") (at 366.395 243.205 0) (unit 1)

Commit message: March 31st Update
Connections:
- net at U54.1 (I1b): now also U56.15 (Q3); no longer U56.10 (Q2)
- net at U54.5 (I1c): now also U56.10 (Q2); no longer U56.15 (Q3)
Changed lines of the file:
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@@
-    (stroke (width 0) (type default) (color 0 0 0 0))
-  )
-  (wire (pts (xy 195.58 104.775) (xy 195.58 113.03))
     (stroke (width 0) (type default) (color 0 0 0 0))
   )
@@
     (stroke (width 0) (type default) (color 0 0 0 0))
   )
-  (wire (pts (xy 193.675 104.775) (xy 195.58 104.775))
-    (stroke (width 0) (type default) (color 0 0 0 0))
-  )
   (wire (pts (xy 848.36 139.065) (xy 864.87 139.065))
     (stroke (width 0) (type default) (color 0 0 0 0))
@@
     (stroke (width 0) (type default) (color 0 0 0 0))
   )
+  (wire (pts (xy 224.79 107.95) (xy 198.755 107.95))
+    (stroke (width 0) (type default) (color 0 0 0 0))
+  )
   (wire (pts (xy 257.81 88.9) (xy 257.81 135.89))
     (stroke (width 0) (type default) (color 0 0 0 0))
   )
+  (wire (pts (xy 198.755 104.775) (xy 193.675 104.775))
+    (stroke (width 0) (type default) (color 0 0 0 0))
+  )
   (wire (pts (xy 39.37 222.885) (xy 51.435 222.885))
     (stroke (width 0) (type default) (color 0 0 0 0))
@@
     (stroke (width 0) (type default) (color 0 0 0 0))
   )
-  (wire (pts (xy 195.58 113.03) (xy 224.79 113.03))
-    (stroke (width 0) (type default) (color 0 0 0 0))
-  )
   (wire (pts (xy 215.265 38.1) (xy 224.79 38.1))
     (stroke (width 0) (type default) (color 0 0 0 0))
@@
     (stroke (width 0) (type default) (color 0 0 0 0))
   )
-  (wire (pts (xy 198.12 99.695) (xy 198.12 107.95))
-    (stroke (width 0) (type default) (color 0 0 0 0))
-  )
   (wire (pts (xy 203.2 49.53) (xy 224.79 49.53))
     (stroke (width 0) (type default) (color 0 0 0 0))
@@
     (stroke (width 0) (type default) (color 0 0 0 0))
   )
-  (wire (pts (xy 198.12 107.95) (xy 224.79 107.95))
-    (stroke (width 0) (type default) (color 0 0 0 0))
-  )
   (wire (pts (xy 252.095 99.06) (xy 252.095 130.81))
     (stroke (width 0) (type default) (color 0 0 0 0))
@@
     (stroke (width 0) (type default) (color 0 0 0 0))
   )
+  (wire (pts (xy 198.755 107.95) (xy 198.755 104.775))
+    (stroke (width 0) (type default) (color 0 0 0 0))
+  )
   (wire (pts (xy 201.93 94.615) (xy 201.93 102.87))
     (stroke (width 0) (type default) (color 0 0 0 0))
@@
     (stroke (width 0) (type default) (color 0 0 0 0))
   )
-  (wire (pts (xy 193.675 99.695) (xy 198.12 99.695))
-    (stroke (width 0) (type default) (color 0 0 0 0))
-  )
   (wire (pts (xy 64.135 193.04) (xy 71.12 193.04))
     (stroke (width 0) (type default) (color 0 0 0 0))
@@
     (stroke (width 0) (type default) (color 0 0 0 0))
   )
+  (wire (pts (xy 224.79 113.03) (xy 200.025 113.03))
+    (stroke (width 0) (type default) (color 0 0 0 0))
+  )
   (wire (pts (xy 128.905 133.35) (xy 128.905 147.955))
     (stroke (width 0) (type default) (color 0 0 0 0))
@@
     (stroke (width 0) (type default) (color 0 0 0 0))
   )
+  (wire (pts (xy 200.025 113.03) (xy 200.025 99.695))
+    (stroke (width 0) (type default) (color 0 0 0 0))
+  )
   (wire (pts (xy 205.74 89.535) (xy 205.74 97.79))
     (stroke (width 0) (type default) (color 0 0 0 0))
@@
     (stroke (width 0) (type default) (color 0 0 0 0))
   )
+  (wire (pts (xy 200.025 99.695) (xy 193.675 99.695))
+    (stroke (width 0) (type default) (color 0 0 0 0))
+  )

Commit message: Version 0.1 (March 31st)
Parts:
- U56: value SN74ALS175N_U56 -> SN74ALS175N (КР1533ТМ8)
- U63: value SN74ALS175N_U63 -> SN74ALS175N (КР1533ТМ8)
Changed lines of the file:
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@@
       (effects (font (size 1.27 1.27)) (justify left))
     )
-    (property "Value" "SN74ALS175N_U63" (id 1) (at 182.9944 34.925 0)
+    (property "Value" "SN74ALS175N (КР1533ТМ8)" (id 1) (at 182.9944 34.925 0)
       (effects (font (size 1.27 1.27)) (justify left))
     )
@@
       (effects (font (size 1.27 1.27)) (justify left))
     )
-    (property "Value" "SN74ALS175N_U56" (id 1) (at 182.9944 83.82 0)
-      (effects (font (size 1.27 1.27)) (justify left))
-    )
+    (property "Value" "SN74ALS175N (КР1533ТМ8)" (id 1) (at 182.9944 83.82 0)
+      (effects (font (size 1.27 1.27)) (justify left))
+    )

Commit message: March 31st final update (for today)
Parts:
- U15: value CD4520АN_(К561ИЕ10) -> CD4520АN (К561ИЕ10A)
Changed lines of the file:
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@@
       (effects (font (size 1.27 1.27)) (justify left))
     )
-    (property "Value" "CD4520АN_(К561ИЕ10)" (id 1) (at 906.78 127.6349 0)
+    (property "Value" "CD4520АN (К561ИЕ10A)" (id 1) (at 906.78 127.6349 0)
       (effects (font (size 1.27 1.27)) (justify left))
     )
@@
     (in_bom yes) (on_board yes) (fields_autoplaced)
     (property "Reference" "U15" (id 0) (at 284.48 182.245 0))
-    (property "Value" "CD4520АN_(К561ИЕ10)" (id 1) (at 284.48 184.785 0))
+    (property "Value" "CD4520АN (К561ИЕ10A)" (id 1) (at 284.48 184.785 0))
     (property "Footprint" "Package_DIP:DIP-16_W7.62mm_Socket" (id 2) (at 284.48 203.2 0)
       (effects (font (size 1.27 1.27)) hide)
