File: SNP.kicad_sch (KiCad schematic)
At the start: 12 parts, among them J1 SNP, SW1 Reset button, U75 IN74ALS32N (КР1533ЛЛ1)

Commit message: Version 1.0 schematics and PCB complete
Parts:
- C25, C26, C27, C28: symbol Device:C -> Delta_s_m_Lib:C
- DA2: symbol Device:R_Network09 -> Delta_s_m_Lib:R_Network09
- J1: symbol w_connectors:SNP -> Delta_s_m_Lib:SNP
- R47, R48, R49, R53: symbol Device:R -> Delta_s_m_Lib:R
- SW1: symbol Switch:SW_Push -> Delta_s_m_Lib:SW_Push
- U75: symbol 74xx:74LS32 -> Delta_s_m_Lib:74LS32
Changed lines of the file:
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@@
     )
   )
-  (symbol (lib_id "Device:R") (at 161.29 134.62 90) (unit 1)
+  (symbol (lib_id "Delta_s_m_Lib:R") (at 161.29 134.62 90) (unit 1)
     (in_bom yes) (on_board yes) (dnp no)
     (property "Reference" "R53" (at 162.56 132.08 90)
@@
     )
   )
-  (symbol (lib_id "Device:C") (at 167.005 42.545 0) (unit 1)
+  (symbol (lib_id "Delta_s_m_Lib:C") (at 167.005 42.545 0) (unit 1)
     (in_bom yes) (on_board yes) (dnp no) (fields_autoplaced)
     (property "Reference" "C26" (at 170.18 41.2749 0)
@@
     )
   )
-  (symbol (lib_id "Device:R") (at 195.58 42.545 0) (unit 1)
+  (symbol (lib_id "Delta_s_m_Lib:R") (at 195.58 42.545 0) (unit 1)
     (in_bom yes) (on_board yes) (dnp no)
     (property "Reference" "R47" (at 196.85 41.275 0)
@@
     )
   )
-  (symbol (lib_id "Device:R") (at 203.835 42.545 0) (unit 1)
+  (symbol (lib_id "Delta_s_m_Lib:R") (at 203.835 42.545 0) (unit 1)
     (in_bom yes) (on_board yes) (dnp no)
     (property "Reference" "R48" (at 205.105 41.275 0)
@@
     )
   )
-  (symbol (lib_id "74xx:74LS32") (at 149.86 134.62 0) (unit 3)
+  (symbol (lib_id "Delta_s_m_Lib:74LS32") (at 149.86 134.62 0) (unit 3)
     (in_bom yes) (on_board yes) (dnp no)
     (property "Reference" "U75" (at 150.495 134.62 0)
@@
     )
   )
-  (symbol (lib_id "Device:C") (at 178.435 42.545 0) (unit 1)
+  (symbol (lib_id "Delta_s_m_Lib:C") (at 178.435 42.545 0) (unit 1)
     (in_bom yes) (on_board yes) (dnp no) (fields_autoplaced)
     (property "Reference" "C27" (at 181.61 41.2749 0)
@@
     )
   )
-  (symbol (lib_id "Device:C") (at 212.09 67.31 0) (unit 1)
+  (symbol (lib_id "Delta_s_m_Lib:C") (at 212.09 67.31 0) (unit 1)
     (in_bom yes) (on_board yes) (dnp no) (fields_autoplaced)
     (property "Reference" "C25" (at 215.265 66.0399 0)
@@
     )
   )
-  (symbol (lib_id "w_connectors:SNP") (at 53.34 69.85 0) (mirror y) (unit 1)
+  (symbol (lib_id "Delta_s_m_Lib:SNP") (at 53.34 69.85 0) (mirror y) (unit 1)
     (in_bom yes) (on_board yes) (dnp no) (fields_autoplaced)
     (property "Reference" "J1" (at 53.34 26.035 0)
@@
     )
   )
-  (symbol (lib_id "Device:C") (at 155.575 42.545 0) (unit 1)
+  (symbol (lib_id "Delta_s_m_Lib:C") (at 155.575 42.545 0) (unit 1)
     (in_bom yes) (on_board yes) (dnp no) (fields_autoplaced)
     (property "Reference" "C28" (at 158.75 41.2749 0)
@@
     )
   )
-  (symbol (lib_id "Device:R") (at 212.09 42.545 0) (unit 1)
+  (symbol (lib_id "Delta_s_m_Lib:R") (at 212.09 42.545 0) (unit 1)
     (in_bom yes) (on_board yes) (dnp no)
     (property "Reference" "R49" (at 213.36 41.275 0)
@@
     )
   )
-  (symbol (lib_id "74xx:74LS32") (at 130.175 132.08 0) (unit 2)
+  (symbol (lib_id "Delta_s_m_Lib:74LS32") (at 130.175 132.08 0) (unit 2)
     (in_bom yes) (on_board yes) (dnp no)
     (property "Reference" "U75" (at 130.175 132.08 0)
@@
     )
   )
-  (symbol (lib_id "Switch:SW_Push") (at 224.79 67.31 270) (unit 1)
+  (symbol (lib_id "Delta_s_m_Lib:SW_Push") (at 224.79 67.31 270) (unit 1)
     (in_bom yes) (on_board yes) (dnp no) (fields_autoplaced)
     (property "Reference" "SW1" (at 228.6 66.0399 90)
@@
     )
   )
-  (symbol (lib_id "Device:R_Network09") (at 138.43 41.275 0) (unit 1)
+  (symbol (lib_id "Delta_s_m_Lib:R_Network09") (at 138.43 41.275 0) (unit 1)
     (in_bom yes) (on_board yes) (dnp no) (fields_autoplaced)
     (property "Reference" "DA2" (at 125.73 40.2589 0)

Commit message: Version 1.2 update
Parts:
- C25, C26, C27, C28: footprint Capacitor_THT:C_Disc_D7.0mm_W2.5mm_P5.00mm -> Delta_sm_lib:C_Disc_D7.0mm_W2.5mm_P5.00mm
- DA2: footprint Resistor_THT:R_Array_SIP10 -> Delta_sm_lib:R_Array_SIP10
- J1: footprint delta:snp59_96_female_angle_3 -> Delta_sm_lib:snp59_96_female_angle_3
- R47, R48, R49, R53: footprint Resistor_THT:R_Axial_DIN0207_L6.3mm_D2.5mm_P10.16mm_Horizontal -> Delta_sm_lib:R_Axial_DIN0207_L6.3mm_D2.5mm_P10.16mm_Horizontal
- SW1: footprint Button_Switch_THT:SW_Tactile_SPST_Angled_PTS645Vx83-2LFS -> Delta_sm_lib:SW_Tactile_SPST_Angled_PTS645Vx83-2LFS
- U75: footprint Package_DIP:DIP-14_W7.62mm_Socket -> Delta_sm_lib:DIP-14_W7.62mm_Socket
Changed lines of the file:
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@@
       (effects (font (size 1.27 1.27)) (justify left))
     )
-    (property "Footprint" "Resistor_THT:R_Axial_DIN0207_L6.3mm_D2.5mm_P10.16mm_Horizontal" (at 161.29 136.398 90)
+    (property "Footprint" "Delta_sm_lib:R_Axial_DIN0207_L6.3mm_D2.5mm_P10.16mm_Horizontal" (at 161.29 136.398 90)
       (effects (font (size 1.27 1.27)) hide)
     )
@@
       (effects (font (size 1.27 1.27)) (justify left))
     )
-    (property "Footprint" "Capacitor_THT:C_Disc_D7.0mm_W2.5mm_P5.00mm" (at 167.9702 46.355 0)
+    (property "Footprint" "Delta_sm_lib:C_Disc_D7.0mm_W2.5mm_P5.00mm" (at 167.9702 46.355 0)
       (effects (font (size 1.27 1.27)) hide)
     )
@@
       (effects (font (size 1.27 1.27)) (justify left))
     )
-    (property "Footprint" "Resistor_THT:R_Axial_DIN0207_L6.3mm_D2.5mm_P10.16mm_Horizontal" (at 193.802 42.545 90)
+    (property "Footprint" "Delta_sm_lib:R_Axial_DIN0207_L6.3mm_D2.5mm_P10.16mm_Horizontal" (at 193.802 42.545 90)
       (effects (font (size 1.27 1.27)) hide)
     )
@@
       (effects (font (size 1.27 1.27)) (justify left))
     )
-    (property "Footprint" "Resistor_THT:R_Axial_DIN0207_L6.3mm_D2.5mm_P10.16mm_Horizontal" (at 202.057 42.545 90)
+    (property "Footprint" "Delta_sm_lib:R_Axial_DIN0207_L6.3mm_D2.5mm_P10.16mm_Horizontal" (at 202.057 42.545 90)
       (effects (font (size 1.27 1.27)) hide)
     )
@@
       (effects (font (size 1.27 1.27)))
     )
-    (property "Footprint" "Package_DIP:DIP-14_W7.62mm_Socket" (at 149.86 134.62 0)
+    (property "Footprint" "Delta_sm_lib:DIP-14_W7.62mm_Socket" (at 149.86 134.62 0)
       (effects (font (size 1.27 1.27)) hide)
     )
@@
       (effects (font (size 1.27 1.27)) (justify left))
     )
-    (property "Footprint" "Capacitor_THT:C_Disc_D7.0mm_W2.5mm_P5.00mm" (at 179.4002 46.355 0)
+    (property "Footprint" "Delta_sm_lib:C_Disc_D7.0mm_W2.5mm_P5.00mm" (at 179.4002 46.355 0)
       (effects (font (size 1.27 1.27)) hide)
     )
@@
       (effects (font (size 1.27 1.27)) (justify left))
     )
-    (property "Footprint" "Capacitor_THT:C_Disc_D7.0mm_W2.5mm_P5.00mm" (at 213.0552 71.12 0)
+    (property "Footprint" "Delta_sm_lib:C_Disc_D7.0mm_W2.5mm_P5.00mm" (at 213.0552 71.12 0)
       (effects (font (size 1.27 1.27)) hide)
     )
@@
       (effects (font (size 1.27 1.27)))
     )
-    (property "Footprint" "delta:snp59_96_female_angle_3" (at 53.34 27.94 0)
+    (property "Footprint" "Delta_sm_lib:snp59_96_female_angle_3" (at 53.34 27.94 0)
       (effects (font (size 1.27 1.27)) hide)
     )
@@
       (effects (font (size 1.27 1.27)) (justify left))
     )
-    (property "Footprint" "Capacitor_THT:C_Disc_D7.0mm_W2.5mm_P5.00mm" (at 156.5402 46.355 0)
+    (property "Footprint" "Delta_sm_lib:C_Disc_D7.0mm_W2.5mm_P5.00mm" (at 156.5402 46.355 0)
       (effects (font (size 1.27 1.27)) hide)
     )
@@
       (effects (font (size 1.27 1.27)) (justify left))
     )
-    (property "Footprint" "Resistor_THT:R_Axial_DIN0207_L6.3mm_D2.5mm_P10.16mm_Horizontal" (at 210.312 42.545 90)
+    (property "Footprint" "Delta_sm_lib:R_Axial_DIN0207_L6.3mm_D2.5mm_P10.16mm_Horizontal" (at 210.312 42.545 90)
       (effects (font (size 1.27 1.27)) hide)
     )
@@
       (effects (font (size 1.27 1.27)))
     )
-    (property "Footprint" "Package_DIP:DIP-14_W7.62mm_Socket" (at 130.175 132.08 0)
+    (property "Footprint" "Delta_sm_lib:DIP-14_W7.62mm_Socket" (at 130.175 132.08 0)
       (effects (font (size 1.27 1.27)) hide)
     )
@@
       (effects (font (size 1.27 1.27)) (justify left))
     )
-    (property "Footprint" "Button_Switch_THT:SW_Tactile_SPST_Angled_PTS645Vx83-2LFS" (at 229.87 67.31 0)
+    (property "Footprint" "Delta_sm_lib:SW_Tactile_SPST_Angled_PTS645Vx83-2LFS" (at 229.87 67.31 0)
       (effects (font (size 1.27 1.27)) hide)
     )
@@
       (effects (font (size 1.27 1.27)) (justify right))
     )
-    (property "Footprint" "Resistor_THT:R_Array_SIP10" (at 153.035 41.275 90)
-      (effects (font (size 1.27 1.27)) hide)
-    )
+    (property "Footprint" "Delta_sm_lib:R_Array_SIP10" (at 153.035 41.275 90)
+      (effects (font (size 1.27 1.27)) hide)
+    )
