File: power.kicad_sch (KiCad schematic)
At the start: 19 parts, among them U19 SN74ALS04 (КР1533ЛН1), U21 SN74ALS14 (КР1533ТЛ2), U39 IN74ALS32N (КР1533ЛЛ1), U40 IN74ALS00N (КР1533ЛА3), U75 IN74ALS32N (КР1533ЛЛ1)

Commit message: Update for U21 fix (tape loading works now)
Parts:
- U21: value SN74ALS14 (КР1533ТЛ2) -> SN74ALS04 (КР1533ЛН1)
Changed lines of the file:
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@@
       (effects (font (size 1.27 1.27)) (justify left))
     )
-    (property "Value" "SN74ALS14 (КР1533ТЛ2)" (at 114.3 43.1799 0)
+    (property "Value" "SN74ALS04 (КР1533ЛН1)" (at 114.3 43.1799 0)
       (effects (font (size 1.27 1.27)) (justify left))
     )

Commit message: Version 1.0 schematics and PCB complete
Parts:
- C13, C16, C17, C18, C19, C2, C20, C23, C24, C29, C30, C31, C9: symbol Device:C -> Delta_s_m_Lib:C
- C15: symbol Device:C_Polarized -> Delta_s_m_Lib:C_Polarized
- U19: symbol 74xx:74LS04 -> Delta_s_m_Lib:74LS04
- U21: symbol 74xx:74LS14 -> Delta_s_m_Lib:74LS14
- U39, U75: symbol 74xx:74LS32 -> Delta_s_m_Lib:74LS32
- U40: symbol 74xx:74LS00 -> Delta_s_m_Lib:74LS00
Changed lines of the file:
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@@
     (stroke (width 0) (type default))
   )
-  (symbol (lib_id "Device:C") (at 240.665 41.91 0) (unit 1)
+  (symbol (lib_id "Delta_s_m_Lib:C") (at 240.665 41.91 0) (unit 1)
     (in_bom yes) (on_board yes) (dnp no) (fields_autoplaced)
     (property "Reference" "C24" (at 243.84 40.6399 0)
@@
     )
   )
-  (symbol (lib_id "74xx:74LS32") (at 54.61 41.91 0) (unit 5)
+  (symbol (lib_id "Delta_s_m_Lib:74LS32") (at 54.61 41.91 0) (unit 5)
     (in_bom yes) (on_board yes) (dnp no) (fields_autoplaced)
     (property "Reference" "U39" (at 61.595 40.6399 0)
@@
     )
   )
-  (symbol (lib_id "Device:C") (at 231.14 41.91 0) (unit 1)
+  (symbol (lib_id "Delta_s_m_Lib:C") (at 231.14 41.91 0) (unit 1)
     (in_bom yes) (on_board yes) (dnp no) (fields_autoplaced)
     (property "Reference" "C20" (at 234.315 40.6399 0)
@@
     )
   )
-  (symbol (lib_id "Device:C") (at 171.45 41.91 0) (unit 1)
+  (symbol (lib_id "Delta_s_m_Lib:C") (at 171.45 41.91 0) (unit 1)
     (in_bom yes) (on_board yes) (dnp no) (fields_autoplaced)
     (property "Reference" "C16" (at 174.625 40.6399 0)
@@
     )
   )
-  (symbol (lib_id "74xx:74LS14") (at 107.95 41.91 0) (unit 7)
+  (symbol (lib_id "Delta_s_m_Lib:74LS14") (at 107.95 41.91 0) (unit 7)
     (in_bom yes) (on_board yes) (dnp no) (fields_autoplaced)
     (property "Reference" "U21" (at 114.3 40.6399 0)
@@
     )
   )
-  (symbol (lib_id "Device:C") (at 160.655 41.91 0) (unit 1)
+  (symbol (lib_id "Delta_s_m_Lib:C") (at 160.655 41.91 0) (unit 1)
     (in_bom yes) (on_board yes) (dnp no) (fields_autoplaced)
     (property "Reference" "C9" (at 163.83 40.6399 0)
@@
     )
   )
-  (symbol (lib_id "Device:C") (at 222.25 41.91 0) (unit 1)
+  (symbol (lib_id "Delta_s_m_Lib:C") (at 222.25 41.91 0) (unit 1)
     (in_bom yes) (on_board yes) (dnp no) (fields_autoplaced)
     (property "Reference" "C23" (at 225.425 40.6399 0)
@@
     )
   )
-  (symbol (lib_id "74xx:74LS04") (at 37.465 41.91 0) (unit 7)
+  (symbol (lib_id "Delta_s_m_Lib:74LS04") (at 37.465 41.91 0) (unit 7)
     (in_bom yes) (on_board yes) (dnp no) (fields_autoplaced)
     (property "Reference" "U19" (at 43.815 40.6399 0)
@@
     )
   )
-  (symbol (lib_id "74xx:74LS32") (at 89.535 41.91 0) (unit 5)
+  (symbol (lib_id "Delta_s_m_Lib:74LS32") (at 89.535 41.91 0) (unit 5)
     (in_bom yes) (on_board yes) (dnp no) (fields_autoplaced)
     (property "Reference" "U75" (at 96.52 40.6399 0)
@@
     )
   )
-  (symbol (lib_id "Device:C") (at 269.24 41.91 0) (unit 1)
+  (symbol (lib_id "Delta_s_m_Lib:C") (at 269.24 41.91 0) (unit 1)
     (in_bom yes) (on_board yes) (dnp no) (fields_autoplaced)
     (property "Reference" "C30" (at 272.415 40.6399 0)
@@
     )
   )
-  (symbol (lib_id "Device:C") (at 250.19 41.91 0) (unit 1)
+  (symbol (lib_id "Delta_s_m_Lib:C") (at 250.19 41.91 0) (unit 1)
     (in_bom yes) (on_board yes) (dnp no) (fields_autoplaced)
     (property "Reference" "C29" (at 253.365 40.6399 0)
@@
     )
   )
-  (symbol (lib_id "74xx:74LS00") (at 72.39 41.91 0) (unit 5)
+  (symbol (lib_id "Delta_s_m_Lib:74LS00") (at 72.39 41.91 0) (unit 5)
     (in_bom yes) (on_board yes) (dnp no) (fields_autoplaced)
     (property "Reference" "U40" (at 79.375 40.6399 0)
@@
     )
   )
-  (symbol (lib_id "Device:C") (at 259.715 41.91 0) (unit 1)
+  (symbol (lib_id "Delta_s_m_Lib:C") (at 259.715 41.91 0) (unit 1)
     (in_bom yes) (on_board yes) (dnp no) (fields_autoplaced)
     (property "Reference" "C17" (at 262.89 40.6399 0)
@@
     )
   )
-  (symbol (lib_id "Device:C") (at 202.565 41.91 0) (unit 1)
+  (symbol (lib_id "Delta_s_m_Lib:C") (at 202.565 41.91 0) (unit 1)
     (in_bom yes) (on_board yes) (dnp no) (fields_autoplaced)
     (property "Reference" "C18" (at 205.74 40.6399 0)
@@
     )
   )
-  (symbol (lib_id "Device:C_Polarized") (at 26.67 40.64 0) (unit 1)
+  (symbol (lib_id "Delta_s_m_Lib:C_Polarized") (at 26.67 40.64 0) (unit 1)
     (in_bom yes) (on_board yes) (dnp no) (fields_autoplaced)
     (property "Reference" "C15" (at 30.48 38.4809 0)
@@
     )
   )
-  (symbol (lib_id "Device:C") (at 192.405 41.91 0) (unit 1)
+  (symbol (lib_id "Delta_s_m_Lib:C") (at 192.405 41.91 0) (unit 1)
     (in_bom yes) (on_board yes) (dnp no) (fields_autoplaced)
     (property "Reference" "C13" (at 195.58 40.6399 0)
@@
     )
   )
-  (symbol (lib_id "Device:C") (at 182.245 41.91 0) (unit 1)
+  (symbol (lib_id "Delta_s_m_Lib:C") (at 182.245 41.91 0) (unit 1)
     (in_bom yes) (on_board yes) (dnp no) (fields_autoplaced)
     (property "Reference" "C31" (at 185.42 40.6399 0)
@@
     )
   )
-  (symbol (lib_id "Device:C") (at 212.725 41.91 0) (unit 1)
+  (symbol (lib_id "Delta_s_m_Lib:C") (at 212.725 41.91 0) (unit 1)
     (in_bom yes) (on_board yes) (dnp no) (fields_autoplaced)
     (property "Reference" "C19" (at 215.9 40.6399 0)
@@
     )
   )
-  (symbol (lib_id "Device:C") (at 148.59 41.91 0) (unit 1)
+  (symbol (lib_id "Delta_s_m_Lib:C") (at 148.59 41.91 0) (unit 1)
     (in_bom yes) (on_board yes) (dnp no) (fields_autoplaced)
     (property "Reference" "C2" (at 151.765 40.6399 0)

Commit message: Version 1.2 update
Parts:
- C13, C16, C17, C18, C19, C2, C20, C23, C24, C29, C30, C31, C9: footprint Capacitor_THT:C_Disc_D7.0mm_W2.5mm_P5.00mm -> Delta_sm_lib:C_Disc_D7.0mm_W2.5mm_P5.00mm
- C15: value 470µF -> 470µF 16V; footprint Capacitor_THT:CP_Radial_D10.0mm_P5.00mm -> Delta_sm_lib:CP_Radial_D10.0mm_P5.00mm
- U19, U21, U39, U40, U75: footprint Package_DIP:DIP-14_W7.62mm_Socket -> Delta_sm_lib:DIP-14_W7.62mm_Socket
Changed lines of the file:
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@@
       (effects (font (size 1.27 1.27)) (justify left))
     )
-    (property "Footprint" "Capacitor_THT:C_Disc_D7.0mm_W2.5mm_P5.00mm" (at 241.6302 45.72 0)
+    (property "Footprint" "Delta_sm_lib:C_Disc_D7.0mm_W2.5mm_P5.00mm" (at 241.6302 45.72 0)
       (effects (font (size 1.27 1.27)) hide)
     )
@@
       (effects (font (size 1.27 1.27)) (justify left))
     )
-    (property "Footprint" "Package_DIP:DIP-14_W7.62mm_Socket" (at 54.61 41.91 0)
+    (property "Footprint" "Delta_sm_lib:DIP-14_W7.62mm_Socket" (at 54.61 41.91 0)
       (effects (font (size 1.27 1.27)) hide)
     )
@@
       (effects (font (size 1.27 1.27)) (justify left))
     )
-    (property "Footprint" "Capacitor_THT:C_Disc_D7.0mm_W2.5mm_P5.00mm" (at 232.1052 45.72 0)
+    (property "Footprint" "Delta_sm_lib:C_Disc_D7.0mm_W2.5mm_P5.00mm" (at 232.1052 45.72 0)
       (effects (font (size 1.27 1.27)) hide)
     )
@@
       (effects (font (size 1.27 1.27)) (justify left))
     )
-    (property "Footprint" "Capacitor_THT:C_Disc_D7.0mm_W2.5mm_P5.00mm" (at 172.4152 45.72 0)
+    (property "Footprint" "Delta_sm_lib:C_Disc_D7.0mm_W2.5mm_P5.00mm" (at 172.4152 45.72 0)
       (effects (font (size 1.27 1.27)) hide)
     )
@@
       (effects (font (size 1.27 1.27)) (justify left))
     )
-    (property "Footprint" "Package_DIP:DIP-14_W7.62mm_Socket" (at 107.95 41.91 0)
+    (property "Footprint" "Delta_sm_lib:DIP-14_W7.62mm_Socket" (at 107.95 41.91 0)
       (effects (font (size 1.27 1.27)) hide)
     )
@@
       (effects (font (size 1.27 1.27)) (justify left))
     )
-    (property "Footprint" "Capacitor_THT:C_Disc_D7.0mm_W2.5mm_P5.00mm" (at 161.6202 45.72 0)
+    (property "Footprint" "Delta_sm_lib:C_Disc_D7.0mm_W2.5mm_P5.00mm" (at 161.6202 45.72 0)
       (effects (font (size 1.27 1.27)) hide)
     )
@@
       (effects (font (size 1.27 1.27)) (justify left))
     )
-    (property "Footprint" "Capacitor_THT:C_Disc_D7.0mm_W2.5mm_P5.00mm" (at 223.2152 45.72 0)
+    (property "Footprint" "Delta_sm_lib:C_Disc_D7.0mm_W2.5mm_P5.00mm" (at 223.2152 45.72 0)
       (effects (font (size 1.27 1.27)) hide)
     )
@@
       (effects (font (size 1.27 1.27)) (justify left))
     )
-    (property "Footprint" "Package_DIP:DIP-14_W7.62mm_Socket" (at 37.465 41.91 0)
+    (property "Footprint" "Delta_sm_lib:DIP-14_W7.62mm_Socket" (at 37.465 41.91 0)
       (effects (font (size 1.27 1.27)) hide)
     )
@@
       (effects (font (size 1.27 1.27)) (justify left))
     )
-    (property "Footprint" "Package_DIP:DIP-14_W7.62mm_Socket" (at 89.535 41.91 0)
+    (property "Footprint" "Delta_sm_lib:DIP-14_W7.62mm_Socket" (at 89.535 41.91 0)
       (effects (font (size 1.27 1.27)) hide)
     )
@@
       (effects (font (size 1.27 1.27)) (justify left))
     )
-    (property "Footprint" "Capacitor_THT:C_Disc_D7.0mm_W2.5mm_P5.00mm" (at 270.2052 45.72 0)
+    (property "Footprint" "Delta_sm_lib:C_Disc_D7.0mm_W2.5mm_P5.00mm" (at 270.2052 45.72 0)
       (effects (font (size 1.27 1.27)) hide)
     )
@@
       (effects (font (size 1.27 1.27)) (justify left))
     )
-    (property "Footprint" "Capacitor_THT:C_Disc_D7.0mm_W2.5mm_P5.00mm" (at 251.1552 45.72 0)
+    (property "Footprint" "Delta_sm_lib:C_Disc_D7.0mm_W2.5mm_P5.00mm" (at 251.1552 45.72 0)
       (effects (font (size 1.27 1.27)) hide)
     )
@@
       (effects (font (size 1.27 1.27)) (justify left))
     )
-    (property "Footprint" "Package_DIP:DIP-14_W7.62mm_Socket" (at 72.39 41.91 0)
+    (property "Footprint" "Delta_sm_lib:DIP-14_W7.62mm_Socket" (at 72.39 41.91 0)
       (effects (font (size 1.27 1.27)) hide)
     )
@@
       (effects (font (size 1.27 1.27)) (justify left))
     )
-    (property "Footprint" "Capacitor_THT:C_Disc_D7.0mm_W2.5mm_P5.00mm" (at 260.6802 45.72 0)
+    (property "Footprint" "Delta_sm_lib:C_Disc_D7.0mm_W2.5mm_P5.00mm" (at 260.6802 45.72 0)
       (effects (font (size 1.27 1.27)) hide)
     )
@@
       (effects (font (size 1.27 1.27)) (justify left))
     )
-    (property "Footprint" "Capacitor_THT:C_Disc_D7.0mm_W2.5mm_P5.00mm" (at 203.5302 45.72 0)
+    (property "Footprint" "Delta_sm_lib:C_Disc_D7.0mm_W2.5mm_P5.00mm" (at 203.5302 45.72 0)
       (effects (font (size 1.27 1.27)) hide)
     )
@@
       (effects (font (size 1.27 1.27)) (justify left))
     )
-    (property "Value" "470µF" (at 30.48 41.0209 0)
-      (effects (font (size 1.27 1.27)) (justify left))
-    )
-    (property "Footprint" "Capacitor_THT:CP_Radial_D10.0mm_P5.00mm" (at 27.6352 44.45 0)
+    (property "Value" "470µF 16V" (at 30.48 41.0209 0)
+      (effects (font (size 1.27 1.27)) (justify left))
+    )
+    (property "Footprint" "Delta_sm_lib:CP_Radial_D10.0mm_P5.00mm" (at 27.6352 44.45 0)
       (effects (font (size 1.27 1.27)) hide)
     )
@@
       (effects (font (size 1.27 1.27)) (justify left))
     )
-    (property "Footprint" "Capacitor_THT:C_Disc_D7.0mm_W2.5mm_P5.00mm" (at 193.3702 45.72 0)
+    (property "Footprint" "Delta_sm_lib:C_Disc_D7.0mm_W2.5mm_P5.00mm" (at 193.3702 45.72 0)
       (effects (font (size 1.27 1.27)) hide)
     )
@@
       (effects (font (size 1.27 1.27)) (justify left))
     )
-    (property "Footprint" "Capacitor_THT:C_Disc_D7.0mm_W2.5mm_P5.00mm" (at 183.2102 45.72 0)
+    (property "Footprint" "Delta_sm_lib:C_Disc_D7.0mm_W2.5mm_P5.00mm" (at 183.2102 45.72 0)
       (effects (font (size 1.27 1.27)) hide)
     )
@@
       (effects (font (size 1.27 1.27)) (justify left))
     )
-    (property "Footprint" "Capacitor_THT:C_Disc_D7.0mm_W2.5mm_P5.00mm" (at 213.6902 45.72 0)
+    (property "Footprint" "Delta_sm_lib:C_Disc_D7.0mm_W2.5mm_P5.00mm" (at 213.6902 45.72 0)
       (effects (font (size 1.27 1.27)) hide)
     )
@@
       (effects (font (size 1.27 1.27)) (justify left))
     )
-    (property "Footprint" "Capacitor_THT:C_Disc_D7.0mm_W2.5mm_P5.00mm" (at 149.5552 45.72 0)
-      (effects (font (size 1.27 1.27)) hide)
-    )
+    (property "Footprint" "Delta_sm_lib:C_Disc_D7.0mm_W2.5mm_P5.00mm" (at 149.5552 45.72 0)
+      (effects (font (size 1.27 1.27)) hide)
+    )
