File: ramd41d48.kicad_sch (KiCad schematic)
At the start: 14 parts, among them U23 SN74ALS253N (КР1533КП12), U24 SN74ALS253N (КР1533КП12), U26 SN74ALS253N (КР1533КП12), U27 SN74ALS253N (КР1533КП12), U41 2118 (КР565РУ6), U42 2118 (КР565РУ6), U43 2118 (КР565РУ6), U44 2118 (КР565РУ6), U45 2118 (КР565РУ6), U46 2118 (КР565РУ6)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

Commit message: Version 1.0 schematics and PCB complete
Parts:
- JP3: symbol Jumper:Jumper_2_Open -> Delta_s_m_Lib:Jumper_2_Open
- R14: symbol Device:R -> Delta_s_m_Lib:R
- U23: symbol w_connectors:SN74ALS253N_(КР1533КП12)_U23 -> Delta_s_m_Lib:SN74ALS253N_(КР1533КП12)_U23
- U24: symbol w_connectors:SN74ALS253N_(КР1533КП12)_U24 -> Delta_s_m_Lib:SN74ALS253N_(КР1533КП12)_U24
- U26: symbol w_connectors:SN74ALS253N_(КР1533КП12)_U26 -> Delta_s_m_Lib:SN74ALS253N_(КР1533КП12)_U26
- U27: symbol w_connectors:SN74ALS253N_(КР1533КП12)_U27 -> Delta_s_m_Lib:SN74ALS253N_(КР1533КП12)_U27
- U41, U42, U43, U44, U45, U46, U47, U48: symbol w_connectors:RU6 -> Delta_s_m_Lib:RU6
Changed lines of the file:
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@@
     )
   )
-  (symbol (lib_id "w_connectors:RU6") (at 264.795 84.455 0) (unit 1)
+  (symbol (lib_id "Delta_s_m_Lib:RU6") (at 264.795 84.455 0) (unit 1)
     (in_bom yes) (on_board yes) (dnp no)
     (property "Reference" "U48" (at 268.605 84.455 0)
@@
     )
   )
-  (symbol (lib_id "w_connectors:RU6") (at 165.1 26.67 0) (unit 1)
+  (symbol (lib_id "Delta_s_m_Lib:RU6") (at 165.1 26.67 0) (unit 1)
     (in_bom yes) (on_board yes) (dnp no)
     (property "Reference" "U42" (at 168.91 26.67 0)
@@
     )
   )
-  (symbol (lib_id "w_connectors:RU6") (at 264.795 26.67 0) (unit 1)
+  (symbol (lib_id "Delta_s_m_Lib:RU6") (at 264.795 26.67 0) (unit 1)
     (in_bom yes) (on_board yes) (dnp no)
     (property "Reference" "U44" (at 268.605 26.67 0)
@@
     )
   )
-  (symbol (lib_id "w_connectors:SN74ALS253N_(КР1533КП12)_U24") (at 187.96 155.575 0) (unit 1)
+  (symbol (lib_id "Delta_s_m_Lib:SN74ALS253N_(КР1533КП12)_U24") (at 187.96 155.575 0) (unit 1)
     (in_bom yes) (on_board yes) (dnp no) (fields_autoplaced)
     (property "Reference" "U24" (at 189.9794 129.54 0)
@@
     )
   )
-  (symbol (lib_id "w_connectors:RU6") (at 115.57 84.455 0) (unit 1)
+  (symbol (lib_id "Delta_s_m_Lib:RU6") (at 115.57 84.455 0) (unit 1)
     (in_bom yes) (on_board yes) (dnp no)
     (property "Reference" "U45" (at 119.38 84.455 0)
@@
     )
   )
-  (symbol (lib_id "w_connectors:RU6") (at 214.63 84.455 0) (unit 1)
+  (symbol (lib_id "Delta_s_m_Lib:RU6") (at 214.63 84.455 0) (unit 1)
     (in_bom yes) (on_board yes) (dnp no)
     (property "Reference" "U47" (at 218.44 84.455 0)
@@
     )
   )
-  (symbol (lib_id "w_connectors:SN74ALS253N_(КР1533КП12)_U26") (at 59.69 53.975 0) (unit 1)
+  (symbol (lib_id "Delta_s_m_Lib:SN74ALS253N_(КР1533КП12)_U26") (at 59.69 53.975 0) (unit 1)
     (in_bom yes) (on_board yes) (dnp no) (fields_autoplaced)
     (property "Reference" "U26" (at 61.7094 27.94 0)
@@
     )
   )
-  (symbol (lib_id "w_connectors:SN74ALS253N_(КР1533КП12)_U23") (at 121.285 150.495 0) (unit 1)
+  (symbol (lib_id "Delta_s_m_Lib:SN74ALS253N_(КР1533КП12)_U23") (at 121.285 150.495 0) (unit 1)
     (in_bom yes) (on_board yes) (dnp no) (fields_autoplaced)
     (property "Reference" "U23" (at 123.3044 124.46 0)
@@
     )
   )
-  (symbol (lib_id "w_connectors:RU6") (at 115.57 27.305 0) (unit 1)
+  (symbol (lib_id "Delta_s_m_Lib:RU6") (at 115.57 27.305 0) (unit 1)
     (in_bom yes) (on_board yes) (dnp no)
     (property "Reference" "U41" (at 119.38 27.305 0)
@@
     )
   )
-  (symbol (lib_id "Jumper:Jumper_2_Open") (at 38.1 134.62 0) (unit 1)
+  (symbol (lib_id "Delta_s_m_Lib:Jumper_2_Open") (at 38.1 134.62 0) (unit 1)
     (in_bom yes) (on_board yes) (dnp no) (fields_autoplaced)
     (property "Reference" "JP3" (at 38.1 128.27 0)
@@
     )
   )
-  (symbol (lib_id "Device:R") (at 38.1 127 90) (unit 1)
+  (symbol (lib_id "Delta_s_m_Lib:R") (at 38.1 127 90) (unit 1)
     (in_bom yes) (on_board yes) (dnp no)
     (property "Reference" "R14" (at 38.1 124.46 90)
@@
     )
   )
-  (symbol (lib_id "w_connectors:RU6") (at 165.1 84.455 0) (unit 1)
+  (symbol (lib_id "Delta_s_m_Lib:RU6") (at 165.1 84.455 0) (unit 1)
     (in_bom yes) (on_board yes) (dnp no)
     (property "Reference" "U46" (at 168.91 84.455 0)
@@
     )
   )
-  (symbol (lib_id "w_connectors:SN74ALS253N_(КР1533КП12)_U27") (at 59.69 115.57 0) (unit 1)
+  (symbol (lib_id "Delta_s_m_Lib:SN74ALS253N_(КР1533КП12)_U27") (at 59.69 115.57 0) (unit 1)
     (in_bom yes) (on_board yes) (dnp no) (fields_autoplaced)
     (property "Reference" "U27" (at 61.7094 89.535 0)
@@
     )
   )
-  (symbol (lib_id "w_connectors:RU6") (at 213.995 26.67 0) (unit 1)
+  (symbol (lib_id "Delta_s_m_Lib:RU6") (at 213.995 26.67 0) (unit 1)
     (in_bom yes) (on_board yes) (dnp no)
     (property "Reference" "U43" (at 217.805 26.67 0)

Commit message: Version 1.2 update
Parts:
- JP3: footprint Connector_PinHeader_2.54mm:PinHeader_1x02_P2.54mm_Vertical -> Delta_sm_lib:PinHeader_1x02_P2.54mm_Vertical
- R14: footprint Resistor_THT:R_Axial_DIN0207_L6.3mm_D2.5mm_P10.16mm_Horizontal -> Delta_sm_lib:R_Axial_DIN0207_L6.3mm_D2.5mm_P10.16mm_Horizontal
- U23, U24, U26, U27, U41, U42, U43, U44, U45, U46, U47, U48: footprint Package_DIP:DIP-16_W7.62mm_Socket -> Delta_sm_lib:DIP-16_W7.62mm_Socket
Changed lines of the file:
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@@
       (effects (font (size 1.27 1.27)))
     )
-    (property "Footprint" "Package_DIP:DIP-16_W7.62mm_Socket" (at 255.905 75.565 0)
+    (property "Footprint" "Delta_sm_lib:DIP-16_W7.62mm_Socket" (at 255.905 75.565 0)
       (effects (font (size 1.27 1.27)) hide)
     )
@@
       (effects (font (size 1.27 1.27)))
     )
-    (property "Footprint" "Package_DIP:DIP-16_W7.62mm_Socket" (at 156.21 17.78 0)
+    (property "Footprint" "Delta_sm_lib:DIP-16_W7.62mm_Socket" (at 156.21 17.78 0)
       (effects (font (size 1.27 1.27)) hide)
     )
@@
       (effects (font (size 1.27 1.27)))
     )
-    (property "Footprint" "Package_DIP:DIP-16_W7.62mm_Socket" (at 255.905 17.78 0)
+    (property "Footprint" "Delta_sm_lib:DIP-16_W7.62mm_Socket" (at 255.905 17.78 0)
       (effects (font (size 1.27 1.27)) hide)
     )
@@
       (effects (font (size 1.27 1.27)) (justify left))
     )
-    (property "Footprint" "Package_DIP:DIP-16_W7.62mm_Socket" (at 186.69 159.385 0)
+    (property "Footprint" "Delta_sm_lib:DIP-16_W7.62mm_Socket" (at 186.69 159.385 0)
       (effects (font (size 1.27 1.27)) hide)
     )
@@
       (effects (font (size 1.27 1.27)))
     )
-    (property "Footprint" "Package_DIP:DIP-16_W7.62mm_Socket" (at 106.68 75.565 0)
+    (property "Footprint" "Delta_sm_lib:DIP-16_W7.62mm_Socket" (at 106.68 75.565 0)
       (effects (font (size 1.27 1.27)) hide)
     )
@@
       (effects (font (size 1.27 1.27)))
     )
-    (property "Footprint" "Package_DIP:DIP-16_W7.62mm_Socket" (at 205.74 75.565 0)
+    (property "Footprint" "Delta_sm_lib:DIP-16_W7.62mm_Socket" (at 205.74 75.565 0)
       (effects (font (size 1.27 1.27)) hide)
     )
@@
       (effects (font (size 1.27 1.27)) (justify left))
     )
-    (property "Footprint" "Package_DIP:DIP-16_W7.62mm_Socket" (at 59.69 53.975 0)
+    (property "Footprint" "Delta_sm_lib:DIP-16_W7.62mm_Socket" (at 59.69 53.975 0)
       (effects (font (size 1.27 1.27)) hide)
     )
@@
       (effects (font (size 1.27 1.27)) (justify left))
     )
-    (property "Footprint" "Package_DIP:DIP-16_W7.62mm_Socket" (at 121.285 150.495 0)
+    (property "Footprint" "Delta_sm_lib:DIP-16_W7.62mm_Socket" (at 121.285 150.495 0)
       (effects (font (size 1.27 1.27)) hide)
     )
@@
       (effects (font (size 1.27 1.27)))
     )
-    (property "Footprint" "Package_DIP:DIP-16_W7.62mm_Socket" (at 106.68 18.415 0)
+    (property "Footprint" "Delta_sm_lib:DIP-16_W7.62mm_Socket" (at 106.68 18.415 0)
       (effects (font (size 1.27 1.27)) hide)
     )
@@
       (effects (font (size 1.27 1.27)))
     )
-    (property "Footprint" "Connector_PinHeader_2.54mm:PinHeader_1x02_P2.54mm_Vertical" (at 38.1 134.62 0)
+    (property "Footprint" "Delta_sm_lib:PinHeader_1x02_P2.54mm_Vertical" (at 38.1 134.62 0)
       (effects (font (size 1.27 1.27)) hide)
     )
@@
       (effects (font (size 1.27 1.27)))
     )
-    (property "Footprint" "Resistor_THT:R_Axial_DIN0207_L6.3mm_D2.5mm_P10.16mm_Horizontal" (at 38.1 128.778 90)
+    (property "Footprint" "Delta_sm_lib:R_Axial_DIN0207_L6.3mm_D2.5mm_P10.16mm_Horizontal" (at 38.1 128.778 90)
       (effects (font (size 1.27 1.27)) hide)
     )
@@
       (effects (font (size 1.27 1.27)))
     )
-    (property "Footprint" "Package_DIP:DIP-16_W7.62mm_Socket" (at 156.21 75.565 0)
+    (property "Footprint" "Delta_sm_lib:DIP-16_W7.62mm_Socket" (at 156.21 75.565 0)
       (effects (font (size 1.27 1.27)) hide)
     )
@@
       (effects (font (size 1.27 1.27)) (justify left))
     )
-    (property "Footprint" "Package_DIP:DIP-16_W7.62mm_Socket" (at 58.42 119.38 0)
+    (property "Footprint" "Delta_sm_lib:DIP-16_W7.62mm_Socket" (at 58.42 119.38 0)
       (effects (font (size 1.27 1.27)) hide)
     )
@@
       (effects (font (size 1.27 1.27)))
     )
-    (property "Footprint" "Package_DIP:DIP-16_W7.62mm_Socket" (at 205.105 17.78 0)
-      (effects (font (size 1.27 1.27)) hide)
-    )
+    (property "Footprint" "Delta_sm_lib:DIP-16_W7.62mm_Socket" (at 205.105 17.78 0)
+      (effects (font (size 1.27 1.27)) hide)
+    )
