File: video.kicad_sch (KiCad schematic)
At the start: 31 parts, among them J11 Conn_01x06, J12 Conn_01x04, J13 Conn_01x02, J2 DIN-7 Video, J3 DIN-5 Audio, J4 DIN-5 Power, J8 USB_PORT, Q1 BC547B, Q3 BC547B, Q4 BC547B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

Commit message: Update
Connections:
- net BLUE: now also J11.4 (Pin_4), J2.4, R17.2, R28.1; no longer J11.5 (Pin_5), J2.5, R27.2, R30.1
- net GREEN: now also J11.5 (Pin_5), J2.5, R27.2, R30.1; no longer J11.4 (Pin_4), J2.4, R17.2, R28.1
- net YB: now also JP6.2 (Pin_2), RV44.1; no longer JP6.6 (Pin_6), RV42.1
- net YG: now also JP6.6 (Pin_6), RV42.1; no longer JP6.2 (Pin_2), RV44.1
Other:
- note added: "ПРОВЕРИТЬ!"
- moved on the sheet: J11, J2
