File: keyboard/keyboard.kicad_pcb (KiCad board)
At the start: 2 copper layers, 273.4 x 132.9 mm, 61 parts, among them J1 Conn_02x12_Odd_Even, SW1 true video, SW10 8, SW11 9, SW12 0, SW13 Break, SW14 delete, SW15 q, SW16 w, SW17 e, SW18 r, SW19 t, SW2 inverted video, SW20 y, SW21 u, SW22 i, SW23 o, SW24 p, SW25 graph, SW26 extended mode, SW27 edit, SW28 a, SW29 s, SW3 1, SW30 d, SW31 f, SW32 g, SW33 h, SW34 j, SW35 k, SW36 l, SW37 enter, SW38 caps shift left, SW39 caps lock, SW4 2, SW40 z, SW41 x, SW42 c, SW43 v, SW44 b, SW45 n, SW46 m, SW47 dot, SW48 caps shift right, SW49 symbol shift left, SW5 3, SW50 semicolon, SW51 quotes, SW52 left, SW53 right, SW54 left space, SW55 right space, SW56 up, SW57 down, SW58 comma, SW59 symbol shift right, SW6 4, SW60 rus-lat, SW7 5, SW8 6, SW9 7

Commit message: Update 20092023
Connections:
- J1 pad 7: unconnected-(J1-Pin_7-Pad7) -> Net-(J1-Pin_7)
- SW12 pad 1: unconnected-(SW12-Pad1) -> Net-(J1-Pin_7)
- SW15 pad 1: unconnected-(SW15-Pad1) -> Net-(J1-Pin_7)
- SW24 pad 1: unconnected-(SW24-Pad1) -> Net-(J1-Pin_7)
- SW28 pad 1: unconnected-(SW28-Pad1) -> Net-(J1-Pin_7)
- SW3 pad 1: unconnected-(SW3-Pad1) -> Net-(J1-Pin_7)
- SW37 pad 1: unconnected-(SW37-Pad1) -> Net-(J1-Pin_7)
- SW38 pad 1: unconnected-(SW38-Pad1) -> Net-(J1-Pin_7)
- SW48 pad 2: unconnected-(SW48-Pad2) -> Net-(J1-Pin_7)
- SW54 pad 1: unconnected-(SW54-Pad1) -> Net-(J1-Pin_7)
- SW55 pad 1: unconnected-(SW55-Pad1) -> Net-(J1-Pin_7)
Routing:
- net Net-(J1-Pin_6): track 0.00 -> 405.2 mm
- net Net-(J1-Pin_7): track 0.00 -> 387.4 mm
- net Net-(J1-Pin_3): track 0.00 -> 239.5 mm
- net Net-(J1-Pin_4): track 0.00 -> 162.7 mm
- net Net-(J1-Pin_5): track 0.00 -> 140.5 mm
- net Net-(J1-Pin_1): track 0.00 -> 117.8 mm
- net Net-(J1-Pin_2): track 0.00 -> 112.1 mm
