File: keyboard_test/keyboard_test.kicad_pcb (KiCad board)
At the start: 2 copper layers, 133 x 67 mm, 65 parts, among them J1 Conn_02x12_Odd_Even, SW1 true video, SW10 8, SW11 9, SW12 0, SW13 Break, SW14 DELETE, SW15 Q, SW16 Q, SW17 E, SW18 R, SW19 T, SW2 inverted video, SW20 Y, SW21 U, SW22 I, SW23 O, SW24 P, SW25 GRAPH, SW26 Extended Mode, SW27 EDIT, SW28 A, SW29 S, SW3 1, SW30 D, SW31 F, SW32 G, SW33 H, SW34 J, SW35 K, SW36 L, SW37 ENTER, SW38 Caps Shift, SW39 Caps Lock, SW4 2, SW40 Z, SW41 X, SW42 C, SW43 V, SW44 B, SW45 N, SW46 M, SW47 ., SW48 Caps Shift, SW49 Symbol Shift, SW5 3, SW50 ;, SW51 ", SW52 ←, SW53 →, SW54 Space (L), SW55 Space (R), SW56 ↑, SW57 ↓, SW58 ,, SW59 Symbol Shift, SW6 4, SW60 RUS/LAT, SW7 5, SW8 6, SW9 7

Commit message: Added silkscreen to test keyboard
Parts:
- added G***: LOGO, kbd_test:logo_early, F.Cu at (159.0, 84.7)
Other:
- board text added: "Delta-S-M Test Keyboard Ver.0.1 Made by MadCat, 2023 https://t.me/madcatse https://www.youtube.com/@MadCatSE https://github.com/madcatse/Delta-S-M"

Commit message: Gerbers
Parts:
- moved G*** 1.42 mm to (160.4, 84.8)
Other:
- board text added: "Delta-S-M Mini-Test Keyboard Ver.0.1 Made by MadCat, 2023 https://t.me/madcatse https://www.youtube.com/@MadCatSE https://github.com/madcatse/Delta-S-M"
- board text removed: "Delta-S-M Test Keyboard Ver.0.1 Made by MadCat, 2023 https://t.me/madcatse https://www.youtube.com/@MadCatSE https://github.com/madcatse/Delta-S-M"
