File: keyboard_cherry/keyboard_cherry.kicad_sch (KiCad schematic)
At the start: 60 parts, among them J1 Conn_02x12_Odd_Even, SW1 true video, SW10 8, SW11 9, SW12 0, SW13 Break, SW14 delete, SW15 q, SW16 w, SW17 e, SW18 r, SW19 t, SW2 inverted video, SW20 y, SW21 u, SW22 i, SW23 o, SW24 p, SW25 graph, SW26 extended mode, SW27 edit, SW28 a, SW29 s, SW3 1, SW30 d, SW31 f, SW32 g, SW33 h, SW34 j, SW35 k, SW36 l, SW37 enter, SW38 caps shift left, SW39 caps lock, SW4 2, SW40 z, SW41 x, SW42 c, SW43 v, SW44 b, SW45 n, SW46 m, SW47 dot, SW48 caps shift right, SW49 symbol shift left, SW5 3, SW50 semicolon, SW51 quotes, SW52 left, SW53 right, SW54 left space, SW56 up, SW57 down, SW58 comma, SW59 symbol shift right, SW6 4, SW60 rus-lat, SW7 5, SW8 6, SW9 7

Commit message: Rev2 Update
Parts:
- SW14, SW49: footprint Button_Switch_Keyboard:SW_Cherry_MX_2.25u_PCB -> Button_Switch_Keyboard:SW_Cherry_MX_2.00u_PCB
- SW25: footprint Button_Switch_Keyboard:SW_Cherry_MX_2.00u_PCB -> Button_Switch_Keyboard:SW_Cherry_MX_1.00u_PCB
- SW26: footprint Button_Switch_Keyboard:SW_Cherry_MX_2.00u_PCB -> Button_Switch_Keyboard:SW_Cherry_MX_1.75u_PCB
- SW37: footprint Button_Switch_Keyboard:SW_Cherry_MX_1.50u_PCB -> Button_Switch_Keyboard:SW_Cherry_MX_1.75u_PCB
- SW38: footprint Button_Switch_Keyboard:SW_Cherry_MX_1.50u_PCB -> Button_Switch_Keyboard:SW_Cherry_MX_2.25u_PCB
- SW48: footprint Button_Switch_Keyboard:SW_Cherry_MX_2.00u_PCB -> Button_Switch_Keyboard:SW_Cherry_MX_2.25u_PCB
- SW59: footprint Button_Switch_Keyboard:SW_Cherry_MX_1.00u_PCB -> Button_Switch_Keyboard:SW_Cherry_MX_1.25u_PCB
- SW60: footprint Button_Switch_Keyboard:SW_Cherry_MX_1.25u_PCB -> Button_Switch_Keyboard:SW_Cherry_MX_1.50u_PCB
Changed lines of the file:
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@@
       (effects (font (size 1.27 1.27)) (justify right))
     )
-    (property "Footprint" "Button_Switch_Keyboard:SW_Cherry_MX_1.25u_PCB" (at 300.355 193.675 0)
+    (property "Footprint" "Button_Switch_Keyboard:SW_Cherry_MX_1.50u_PCB" (at 300.355 193.675 0)
       (effects (font (size 1.27 1.27)) hide)
     )
@@
       (effects (font (size 1.27 1.27)) (justify right))
     )
-    (property "Footprint" "Button_Switch_Keyboard:SW_Cherry_MX_1.50u_PCB" (at 92.71 170.18 0)
+    (property "Footprint" "Button_Switch_Keyboard:SW_Cherry_MX_2.25u_PCB" (at 92.71 170.18 0)
       (effects (font (size 1.27 1.27)) hide)
     )
@@
       (effects (font (size 1.27 1.27)) (justify right))
     )
-    (property "Footprint" "Button_Switch_Keyboard:SW_Cherry_MX_2.25u_PCB" (at 92.71 120.65 0)
+    (property "Footprint" "Button_Switch_Keyboard:SW_Cherry_MX_2.00u_PCB" (at 92.71 120.65 0)
       (effects (font (size 1.27 1.27)) hide)
     )
@@
       (effects (font (size 1.27 1.27)) (justify right))
     )
-    (property "Footprint" "Button_Switch_Keyboard:SW_Cherry_MX_1.50u_PCB" (at 308.61 144.78 0)
+    (property "Footprint" "Button_Switch_Keyboard:SW_Cherry_MX_1.75u_PCB" (at 308.61 144.78 0)
       (effects (font (size 1.27 1.27)) hide)
     )
@@
       (effects (font (size 1.27 1.27)) (justify right))
     )
-    (property "Footprint" "Button_Switch_Keyboard:SW_Cherry_MX_2.00u_PCB" (at 312.42 120.65 0)
+    (property "Footprint" "Button_Switch_Keyboard:SW_Cherry_MX_1.00u_PCB" (at 312.42 120.65 0)
       (effects (font (size 1.27 1.27)) hide)
     )
@@
       (effects (font (size 1.27 1.27)) (justify right))
     )
-    (property "Footprint" "Button_Switch_Keyboard:SW_Cherry_MX_1.00u_PCB" (at 281.94 194.31 0)
+    (property "Footprint" "Button_Switch_Keyboard:SW_Cherry_MX_1.25u_PCB" (at 281.94 194.31 0)
       (effects (font (size 1.27 1.27)) hide)
     )
@@
       (effects (font (size 1.27 1.27)) (justify right))
     )
-    (property "Footprint" "Button_Switch_Keyboard:SW_Cherry_MX_2.00u_PCB" (at 92.71 144.78 0)
+    (property "Footprint" "Button_Switch_Keyboard:SW_Cherry_MX_1.75u_PCB" (at 92.71 144.78 0)
       (effects (font (size 1.27 1.27)) hide)
     )
@@
       (effects (font (size 1.27 1.27)) (justify right))
     )
-    (property "Footprint" "Button_Switch_Keyboard:SW_Cherry_MX_2.00u_PCB" (at 290.83 170.18 0)
+    (property "Footprint" "Button_Switch_Keyboard:SW_Cherry_MX_2.25u_PCB" (at 290.83 170.18 0)
       (effects (font (size 1.27 1.27)) hide)
     )
@@
       (effects (font (size 1.27 1.27)) (justify right))
     )
-    (property "Footprint" "Button_Switch_Keyboard:SW_Cherry_MX_2.25u_PCB" (at 83.82 193.04 0)
-      (effects (font (size 1.27 1.27)) hide)
-    )
+    (property "Footprint" "Button_Switch_Keyboard:SW_Cherry_MX_2.00u_PCB" (at 83.82 193.04 0)
+      (effects (font (size 1.27 1.27)) hide)
+    )
