File: keyboard_cherry/keyboard_cherry.kicad_pcb (KiCad board)
At the start: 2 copper layers, 291.6 x 112.5 mm, 62 parts, among them J1 Conn_02x12_Odd_Even, SW1 true video, SW10 8, SW11 9, SW12 0, SW13 Break, SW14 delete, SW15 q, SW16 w, SW17 e, SW18 r, SW19 t, SW2 inverted video, SW20 y, SW21 u, SW22 i, SW23 o, SW24 p, SW25 graph, SW26 extended mode, SW27 edit, SW28 a, SW29 s, SW3 1, SW30 d, SW31 f, SW32 g, SW33 h, SW34 j, SW35 k, SW36 l, SW37 enter, SW38 caps shift left, SW39 caps lock, SW4 2, SW40 z, SW41 x, SW42 c, SW43 v, SW44 b, SW45 n, SW46 m, SW47 dot, SW48 caps shift right, SW49 symbol shift left, SW5 3, SW50 semicolon, SW51 quotes, SW52 left, SW53 right, SW54 left space, SW56 up, SW57 down, SW58 comma, SW59 symbol shift right, SW6 4, SW60 rus-lat, SW7 5, SW8 6, SW9 7

Commit message: Keyboard models update
Parts:
- H1, H2: footprint MountingHole:MountingHole_3.2mm_M3 -> Library_mx:MountingHole_3.2mm_M3
- J1: footprint Connector_IDC:IDC-Header_2x12_P2.54mm_Vertical -> Library_mx:IDC-Header_2x12_P2.54mm_Vertical
- SW1, SW2, SW27, SW37, SW38: footprint Button_Switch_Keyboard:SW_Cherry_MX_1.50u_PCB -> Library_mx:SW_Cherry_MX_1.50u_PCB
- SW10, SW11, SW12, SW13, SW15, SW16, SW17, SW18, SW19, SW20, SW21, SW22, SW23, SW24, SW28, SW29, SW3, SW30, SW31, SW32, SW33, SW34, SW35, SW36, SW39, SW4, SW40, SW41, SW42, SW43, SW44, SW45, SW46, SW47, SW5, SW50, SW51, SW52, SW53, SW56, SW57, SW58, SW59, SW6, SW7, SW8, SW9: footprint Button_Switch_Keyboard:SW_Cherry_MX_1.00u_PCB -> Library_mx:SW_Cherry_MX_1.00u_PCB
- SW14, SW49: footprint Button_Switch_Keyboard:SW_Cherry_MX_2.25u_PCB -> Library_mx:SW_Cherry_MX_2.25u_PCB
- SW25, SW26, SW48: footprint Button_Switch_Keyboard:SW_Cherry_MX_2.00u_PCB -> Library_mx:SW_Cherry_MX_2.00u_PCB
- SW54: footprint Button_Switch_Keyboard:SW_Cherry_MX_6.25u_PCB -> Library_mx:SW_Cherry_MX_6.25u_PCB
- SW60: footprint Button_Switch_Keyboard:SW_Cherry_MX_1.25u_PCB -> Library_mx:SW_Cherry_MX_1.25u_PCB
- moved SW1 69.6 mm to (305.8, 114.9)
- moved H1 69.5 mm to (63.3, 96.0)
- moved J1 69.5 mm to (289.0, 82.7)
- moved SW10 69.5 mm to (232.7, 95.4)
- moved SW11 69.5 mm to (252.2, 95.4)
- moved SW12 69.5 mm to (271.7, 95.4)
- moved SW13 69.5 mm to (76.7, 95.4)
- moved SW15 69.5 mm to (105.9, 114.9)
- moved SW16 69.5 mm to (125.4, 114.9)
- moved SW17 69.5 mm to (144.9, 114.9)
- moved SW18 69.5 mm to (164.4, 114.9)
- moved SW19 69.5 mm to (183.9, 114.9)
- moved SW20 69.5 mm to (203.4, 114.9)
- moved SW21 69.5 mm to (222.9, 114.9)
- moved SW22 69.5 mm to (242.4, 114.9)
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Routing:
- net Net-(J1-Pin_7): track 463.9 -> 0.00 mm, vias 2 -> 0
- net Net-(J1-Pin_6): track 447.1 -> 0.00 mm, vias 3 -> 0
- net Net-(J1-Pin_13): track 389.0 -> 0.00 mm
- net Net-(J1-Pin_20): track 379.9 -> 0.00 mm, vias 1 -> 0
- net Net-(J1-Pin_24): track 343.3 -> 0.00 mm
- net Net-(J1-Pin_11): track 337.5 -> 0.00 mm
- net Net-(J1-Pin_18): track 320.0 -> 0.00 mm
- net Net-(J1-Pin_5): track 300.9 -> 0.00 mm, vias 2 -> 0
- net Net-(J1-Pin_12): track 283.7 -> 0.00 mm, vias 1 -> 0
- net Net-(J1-Pin_14): track 275.9 -> 0.00 mm
- net Net-(J1-Pin_4): track 273.8 -> 0.00 mm, vias 1 -> 0
- net Net-(J1-Pin_23): track 246.4 -> 0.00 mm
- net Net-(J1-Pin_3): track 237.9 -> 0.00 mm, vias 1 -> 0
- net Net-(J1-Pin_21): track 233.8 -> 0.00 mm, vias 2 -> 0
- net Net-(J1-Pin_22): track 228.7 -> 0.00 mm, vias 1 -> 0
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
Commit message: Adding plate to keyboard
Parts:
- moved J1 58.3 mm to (274.4, 26.2)
- moved SW49 57.5 mm to (94.6, 116.1)
- moved SW25 57.5 mm to (135.1, 116.1)
- moved SW54 57.3 mm to (213.7, 116.1)
- moved SW52 57.2 mm to (282.7, 116.1)
- moved SW57 57.2 mm to (301.8, 116.1)
- moved SW59 57.2 mm to (339.9, 116.1)
- moved SW53 57.2 mm to (320.8, 116.1)
- moved SW38 57.1 mm to (87.4, 97.1)
- moved SW39 57.0 mm to (111.3, 97.1)
- moved SW40 57.0 mm to (130.3, 97.1)
- moved SW41 56.9 mm to (149.4, 97.1)
- moved SW42 56.9 mm to (168.4, 97.1)
- moved SW43 56.9 mm to (187.5, 97.1)
- moved SW44 56.9 mm to (206.5, 97.1)
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Routing:
- net Net-(J1-Pin_7): track 0.00 -> 436.1 mm, vias 0 -> 2
- net Net-(J1-Pin_6): track 0.00 -> 429.7 mm, vias 0 -> 1
- net Net-(J1-Pin_13): track 0.00 -> 416.5 mm
- net Net-(J1-Pin_20): track 0.00 -> 372.9 mm, vias 0 -> 1
- net Net-(J1-Pin_24): track 0.00 -> 350.4 mm, vias 0 -> 1
- net Net-(J1-Pin_11): track 0.00 -> 331.6 mm, vias 0 -> 2
- net Net-(J1-Pin_18): track 0.00 -> 323.9 mm
- net Net-(J1-Pin_12): track 0.00 -> 284.3 mm, vias 0 -> 1
- net Net-(J1-Pin_5): track 0.00 -> 283.6 mm, vias 0 -> 1
- net Net-(J1-Pin_21): track 0.00 -> 277.3 mm
- net Net-(J1-Pin_14): track 0.00 -> 259.0 mm
- net Net-(J1-Pin_4): track 0.00 -> 258.5 mm, vias 0 -> 1
- net Net-(J1-Pin_23): track 0.00 -> 236.1 mm
- net Net-(J1-Pin_22): track 0.00 -> 230.5 mm
- net Net-(J1-Pin_3): track 0.00 -> 222.6 mm, vias 0 -> 1
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Other:
- board size 291.6 x 112.5 mm -> 293.1 x 225.6 mm

Commit message: Update 16.10.2023 (3D stuff)
Parts:
- added H2: MountingHole_3.2mm_M3, MountingHole:MountingHole_3.2mm_M3, F.Cu at (170.7, 68.2)
- added H4: MountingHole_3.2mm, MountingHole:MountingHole_3.2mm_M3, F.Cu at (43.9, 169.2)
- added H5: MountingHole_3.2mm_M3, MountingHole:MountingHole_3.2mm_M3, F.Cu at (206.9, 155.2)
- added H6: MountingHole_3.2mm_M3, MountingHole:MountingHole_3.2mm_M3, F.Cu at (329.0, 169.2)
- moved SW10 47.9 mm to (213.1, 82.5)
- moved SW26 47.9 mm to (70.2, 120.6)
- moved SW29 47.9 mm to (117.8, 120.6)
- moved SW31 47.9 mm to (155.9, 120.6)
- moved SW32 47.9 mm to (175.0, 120.6)
- moved SW33 47.9 mm to (194.0, 120.6)
- moved SW34 47.9 mm to (213.1, 120.6)
- moved SW37 47.9 mm to (313.1, 120.6)
- moved SW49 47.9 mm to (72.6, 158.7)
- moved SW5 47.9 mm to (117.8, 82.5)
- moved SW50 47.9 mm to (270.2, 120.6)
- moved SW51 47.9 mm to (289.3, 120.6)
- moved SW52 47.9 mm to (260.7, 158.7)
- moved SW57 47.9 mm to (279.7, 158.7)
- moved SW59 47.9 mm to (317.8, 158.7)
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- renumbered H2 to H3
Other:
- board size 293.1 x 225.6 mm -> 293.1 x 115.4 mm
- board text added: "Клавиатура БПК {dblquote}Дельта-С{dblquote} / Delta-S Keyboard (PCB) Version 0.1 Board Design by MadCat, 2023 https://github.com/madcatse/Delta-S-M t.me/zx_delta_s https://www.youtube.com/@MadCatSE"
- board text removed: "Д1-02.00.00.001 ИЗМ.1"

Commit message: Keyboard gerbers and 3d modelling of top case
Parts:
- added H7: MountingHole_3.2mm_M3, MountingHole:MountingHole_3.2mm_M3, F.Cu at (186.6, 113.3)
- added H8: MountingHole_3.2mm_M3, MountingHole:MountingHole_3.2mm_M3, F.Cu at (289.5, 110.0)
- moved H4 290.9 mm to (289.5, 13.5)
- moved H6 229.3 mm to (106.6, 113.3)
- moved H5 208.4 mm to (3.44, 110.0)
- moved H3 159.9 mm to (186.6, 8.70)
- moved H2 87.4 mm to (106.6, 8.70)
- moved H1 79.6 mm to (3.44, 13.5)
- moved SW1 76.0 mm to (243.8, 37.4)
- moved SW10 76.0 mm to (172.4, 18.3)
- moved SW11 76.0 mm to (191.4, 18.3)
- moved SW12 76.0 mm to (210.5, 18.3)
- moved SW13 76.0 mm to (20.0, 18.3)
- moved SW14 76.0 mm to (265.3, 18.3)
- moved SW16 76.0 mm to (67.6, 37.4)
- moved SW17 76.0 mm to (86.7, 37.4)
- moved SW19 76.0 mm to (124.8, 37.4)
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Routing:
- net Net-(J1-Pin_12): track 284.3 -> 288.7 mm
- net Net-(J1-Pin_14): track 259.0 -> 262.4 mm
- net Net-(J1-Pin_4): track 258.5 -> 259.7 mm
Other:
- board size 293.1 x 115.4 mm -> 293.1 x 117 mm

Commit message: Rev2 Update
Parts:
- removed H7, H8: MountingHole_3.2mm_M3, MountingHole:MountingHole_3.2mm_M3
- J1: footprint Library_mx:IDC-Header_2x12_P2.54mm_Vertical -> Connector_IDC:IDC-Header_2x12_P2.54mm_Vertical
- SW1, SW2, SW27: footprint Library_mx:SW_Cherry_MX_1.50u_PCB -> Button_Switch_Keyboard:SW_Cherry_MX_1.50u_PCB
- SW10, SW11, SW12, SW13, SW15, SW16, SW17, SW18, SW19, SW20, SW21, SW22, SW23, SW24, SW28, SW29, SW3, SW30, SW31, SW32, SW33, SW34, SW35, SW36, SW39, SW4, SW40, SW41, SW42, SW43, SW44, SW45, SW46, SW47, SW5, SW50, SW51, SW52, SW53, SW56, SW57, SW58, SW6, SW7, SW8, SW9: footprint Library_mx:SW_Cherry_MX_1.00u_PCB -> Button_Switch_Keyboard:SW_Cherry_MX_1.00u_PCB
- SW14, SW49: footprint Library_mx:SW_Cherry_MX_2.25u_PCB -> Button_Switch_Keyboard:SW_Cherry_MX_2.00u_PCB
- SW25: footprint Library_mx:SW_Cherry_MX_2.00u_PCB -> Button_Switch_Keyboard:SW_Cherry_MX_1.00u_PCB
- SW26: footprint Library_mx:SW_Cherry_MX_2.00u_PCB -> Button_Switch_Keyboard:SW_Cherry_MX_1.75u_PCB
- SW37: footprint Library_mx:SW_Cherry_MX_1.50u_PCB -> Button_Switch_Keyboard:SW_Cherry_MX_1.75u_PCB
- SW38: footprint Library_mx:SW_Cherry_MX_1.50u_PCB -> Button_Switch_Keyboard:SW_Cherry_MX_2.25u_PCB
- SW48: footprint Library_mx:SW_Cherry_MX_2.00u_PCB -> Button_Switch_Keyboard:SW_Cherry_MX_2.25u_PCB
- SW54: footprint Library_mx:SW_Cherry_MX_6.25u_PCB -> Button_Switch_Keyboard:SW_Cherry_MX_6.25u_PCB
- SW59: footprint Library_mx:SW_Cherry_MX_1.00u_PCB -> Button_Switch_Keyboard:SW_Cherry_MX_1.25u_PCB
- SW60: footprint Library_mx:SW_Cherry_MX_1.25u_PCB -> Button_Switch_Keyboard:SW_Cherry_MX_1.50u_PCB
- moved SW39 21.3 mm to (58.1, 94.5)
- moved SW38 7.14 mm to (31.9, 75.5)
- moved SW32 4.76 mm to (129.5, 56.4)
- moved SW35 4.76 mm to (186.7, 56.4)
- moved SW44 4.76 mm to (139.1, 75.5)
- moved SW46 4.76 mm to (177.2, 75.5)
- moved SW50 4.76 mm to (224.8, 56.4)
- moved SW53 4.76 mm to (253.4, 94.5)
- moved SW54 4.76 mm to (146.2, 94.5)
- moved SW56 4.76 mm to (234.3, 75.5)
- moved SW57 4.76 mm to (234.3, 94.5)
- moved SW25 4.76 mm to (77.1, 94.5)
- moved SW28 4.76 mm to (53.3, 56.4)
- moved SW29 4.76 mm to (72.4, 56.4)
- moved SW31 4.76 mm to (110.5, 56.4)
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Routing:
- net Net-(J1-Pin_21): track 277.3 -> 213.5 mm, vias 0 -> 1
- net Net-(J1-Pin_10): track 144.3 -> 178.6 mm, vias 0 -> 1
- net Net-(J1-Pin_6): track 429.7 -> 459.5 mm, vias 1 -> 2
- net Net-(J1-Pin_24): track 350.4 -> 323.0 mm, vias 1 -> 0
- net Net-(J1-Pin_8): track 153.3 -> 134.1 mm, vias 0 -> 1
- net Net-(J1-Pin_11): track 331.6 -> 348.1 mm, vias 2 -> 0
- net Net-(J1-Pin_13): track 416.5 -> 401.3 mm, vias 0 -> 1
- net Net-(J1-Pin_12): track 288.7 -> 300.6 mm
- net Net-(J1-Pin_18): track 323.9 -> 334.3 mm
- net Net-(J1-Pin_22): track 230.5 -> 220.6 mm, vias 0 -> 1
- net Net-(J1-Pin_23): track 236.4 -> 229.2 mm, vias 0 -> 1
- net Net-(J1-Pin_5): track 283.6 -> 290.3 mm
- net Net-(J1-Pin_14): track 262.4 -> 257.0 mm
- net Net-(J1-Pin_7): track 436.1 -> 441.1 mm, vias 2 -> 1
- net Net-(J1-Pin_9): track 182.3 -> 177.7 mm, vias 1 -> 2
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
Commit message: Routing rev2
Routing:
- net Net-(J1-Pin_17): track 143.8 -> 188.4 mm, vias 3 -> 0
- net Net-(J1-Pin_10): track 178.6 -> 145.5 mm, vias 1 -> 0
- net Net-(J1-Pin_6): track 459.5 -> 437.3 mm, vias 2 -> 0
- net Net-(J1-Pin_24): track 323.0 -> 343.5 mm
- net Net-(J1-Pin_12): track 300.6 -> 283.5 mm
- net Net-(J1-Pin_21): track 213.5 -> 227.6 mm, vias 1 -> 2
- net Net-(J1-Pin_15): track 203.5 -> 217.0 mm, vias 0 -> 1
- net Net-(J1-Pin_5): track 290.3 -> 277.7 mm
- net Net-(J1-Pin_7): track 441.1 -> 429.3 mm
- net Net-(J1-Pin_13): track 401.3 -> 390.5 mm
- net Net-(J1-Pin_4): track 261.2 -> 254.1 mm
- net Net-(J1-Pin_8): track 134.1 -> 128.5 mm, vias 1 -> 0
- net Net-(J1-Pin_9): track 177.7 -> 173.6 mm, vias 2 -> 1
- net Net-(J1-Pin_11): track 348.1 -> 352.1 mm, vias 0 -> 1
- net Net-(J1-Pin_14): track 257.0 -> 253.0 mm
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
Commit message: Cleanup
Parts:
- added H7: MountingHole_3.2mm_M3, Library_mx:MountingHole_3.2mm_M3, F.Cu at (186.6, 113.3)
- added H8: MountingHole_3.2mm, MountingHole:MountingHole_3.2mm_M3, F.Cu at (289.5, 113.3)
Changed lines of the file:
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@@
     )
   )
+  (footprint "MountingHole:MountingHole_3.2mm_M3" (layer "F.Cu")
+    (at 289.4933 113.2591)
+    (descr "Mounting Hole 3.2mm, no annular, M3")
+    (tags "mounting hole 3.2mm no annular m3")
+    (attr board_only exclude_from_pos_files exclude_from_bom)
+    (fp_text reference "H8" (at 0 -4.2) (layer "F.SilkS") hide
+        (effects (font (size 1 1) (thickness 0.15)))
+    )
+    (fp_text value "MountingHole_3.2mm" (at 0 4.2) (layer "F.Fab")
+        (effects (font (size 1 1) (thickness 0.15)))
+    )
+    (fp_text user "${REFERENCE}" (at 0 0) (layer "F.Fab")
+        (effects (font (size 1 1) (thickness 0.15)))
+    )
+    (fp_circle (center 0 0) (end 3.45 0)
+      (stroke (width 0.05) (type solid)) (fill none) (layer "F.CrtYd"))
+    (pad "" np_thru_hole circle (at 0 0) (size 3.2 3.2) (drill 3.2) (layers "*.Cu" "*.Mask"))
+  )
   (footprint "Button_Switch_Keyboard:SW_Cherry_MX_1.00u_PCB" (layer "F.Cu")
     (at 200.9679 37.35)
@@
     (tags "mounting hole 3.2mm no annular m3")
     (attr board_only exclude_from_pos_files exclude_from_bom)
-    (fp_text reference "H5" (at 0 -4.2) (layer "F.SilkS")
+    (fp_text reference "H5" (at 0 -4.2) (layer "F.SilkS") hide
         (effects (font (size 1 1) (thickness 0.15)))
     )
@@
     )
   )
+  (footprint "Library_mx:MountingHole_3.2mm_M3" (layer "F.Cu")
+    (at 186.628 113.2591)
+    (descr "Mounting Hole 3.2mm, no annular, M3")
+    (tags "mounting hole 3.2mm no annular m3")
+    (attr board_only exclude_from_pos_files exclude_from_bom)
+    (fp_text reference "H7" (at 0 -4.2) (layer "F.SilkS") hide
+        (effects (font (size 1 1) (thickness 0.15)))
+    )
+    (fp_text value "MountingHole_3.2mm_M3" (at -6.34235 -6.064) (layer "F.Fab")
+        (effects (font (size 1 1) (thickness 0.15)))
+    )
+    (fp_text user "${REFERENCE}" (at 0 0) (layer "F.Fab")
+        (effects (font (size 1 1) (thickness 0.15)))
+    )
+    (fp_circle (center 0 0) (end 3.45 0)
+      (stroke (width 0.05) (type solid)) (fill none) (layer "F.CrtYd"))
+    (pad "" np_thru_hole circle (at 0 0) (size 3.2 3.2) (drill 3.2) (layers "*.Cu" "*.Mask"))
+  )
   (footprint "Button_Switch_Keyboard:SW_Cherry_MX_1.00u_PCB" (layer "F.Cu")
     (at 110.4804 56.4)
@@
     (tags "mounting hole 3.2mm no annular m3")
     (attr board_only exclude_from_pos_files exclude_from_bom)
-    (fp_text reference "H6" (at -4.1376 2.7409) (layer "F.SilkS")
+    (fp_text reference "H6" (at -4.1376 2.7409) (layer "F.SilkS") hide
         (effects (font (size 1 1) (thickness 0.15)))
     )
