File: keyboard_cherry/keyboard_cherry.kicad_pcb (KiCad board)
At the start: 2 copper layers, 293.1 x 117 mm, 68 parts, among them J1 Conn_02x12_Odd_Even, SW1 true video, SW10 8, SW11 9, SW12 0, SW13 Break, SW14 delete, SW15 q, SW16 w, SW17 e, SW18 r, SW19 t, SW2 inverted video, SW20 y, SW21 u, SW22 i, SW23 o, SW24 p, SW25 graph, SW26 extended mode, SW27 edit, SW28 a, SW29 s, SW3 1, SW30 d, SW31 f, SW32 g, SW33 h, SW34 j, SW35 k, SW36 l, SW37 enter, SW38 caps shift left, SW39 caps lock, SW4 2, SW40 z, SW41 x, SW42 c, SW43 v, SW44 b, SW45 n, SW46 m, SW47 dot, SW48 caps shift right, SW49 symbol shift left, SW5 3, SW50 semicolon, SW51 quotes, SW52 left, SW53 right, SW54 left space, SW56 up, SW57 down, SW58 comma, SW59 symbol shift right, SW6 4, SW60 rus-lat, SW7 5, SW8 6, SW9 7

Commit message: Layout ver.2 finalised
Parts:
- SW1, SW2: footprint Button_Switch_Keyboard:SW_Cherry_MX_1.50u_PCB -> Library_mx:SW_Cherry_MX_1.00u_PCB
- SW10, SW11, SW12, SW13, SW15, SW16, SW17, SW18, SW19, SW20, SW21, SW22, SW23, SW24, SW28, SW29, SW3, SW30, SW31, SW32, SW33, SW34, SW35, SW36, SW4, SW40, SW41, SW42, SW43, SW44, SW45, SW46, SW47, SW5, SW50, SW51, SW52, SW53, SW56, SW57, SW58, SW6, SW7, SW8, SW9: footprint Button_Switch_Keyboard:SW_Cherry_MX_1.00u_PCB -> Library_mx:SW_Cherry_MX_1.00u_PCB
- SW14, SW49: footprint Button_Switch_Keyboard:SW_Cherry_MX_2.00u_PCB -> Library_mx:SW_Cherry_MX_2.00u_PCB
- SW25: footprint Button_Switch_Keyboard:SW_Cherry_MX_1.00u_PCB -> Library_mx:SW_Cherry_MX_1.50u_PCB
- SW26: footprint Button_Switch_Keyboard:SW_Cherry_MX_1.75u_PCB -> Library_mx:SW_Cherry_MX_1.50u_PCB
- SW27, SW60: footprint Button_Switch_Keyboard:SW_Cherry_MX_1.50u_PCB -> Library_mx:SW_Cherry_MX_1.50u_PCB
- SW37: footprint Button_Switch_Keyboard:SW_Cherry_MX_1.75u_PCB -> Library_mx:SW_Cherry_MX_1.75u_PCB
- SW38, SW48: footprint Button_Switch_Keyboard:SW_Cherry_MX_2.25u_PCB -> Library_mx:SW_Cherry_MX_2.25u_PCB
- SW39: footprint Button_Switch_Keyboard:SW_Cherry_MX_1.00u_PCB -> Library_mx:SW_Cherry_MX_1.75u_PCB
- SW54: footprint Button_Switch_Keyboard:SW_Cherry_MX_6.25u_PCB -> Library_mx:SW_Cherry_MX_6.25u_PCB
- SW59: footprint Button_Switch_Keyboard:SW_Cherry_MX_1.25u_PCB -> Library_mx:SW_Cherry_MX_1.25u_PCB
- moved SW27 247.6 mm to (272.4, 37.4)
- moved SW2 203.5 mm to (77.1, 94.5)
- moved SW1 194.3 mm to (58.1, 94.5)
- moved SW25 174.7 mm to (234.3, 18.3)
- moved SW39 49.1 mm to (27.1, 56.4)
- moved SW60 21.3 mm to (243.8, 37.4)
- moved SW26 19.2 mm to (24.8, 37.4)
Routing:
- net Net-(J1-Pin_18): track 333.8 -> 182.3 mm
- net Net-(J1-Pin_10): track 145.5 -> 280.2 mm, vias 0 -> 1
- net Net-(J1-Pin_9): track 173.6 -> 261.9 mm
- net Net-(J1-Pin_17): track 188.4 -> 139.7 mm
- net Net-(J1-Pin_11): track 352.1 -> 304.9 mm, vias 1 -> 0
- net Net-(J1-Pin_6): track 437.3 -> 468.2 mm, vias 0 -> 1
- net Net-(J1-Pin_2): track 24.1 -> 48.3 mm
- net Net-(J1-Pin_1): track 32.6 -> 54.3 mm
- net Net-(J1-Pin_8): track 128.5 -> 149.4 mm
- net Net-(J1-Pin_13): track 390.5 -> 371.9 mm
- net Net-(J1-Pin_14): track 253.0 -> 236.1 mm
- net Net-(J1-Pin_21): track 227.6 -> 214.1 mm, vias 2 -> 1
- net Net-(J1-Pin_12): track 283.5 -> 296.7 mm
- net Net-(J1-Pin_7): track 429.3 -> 439.8 mm
- net Net-(J1-Pin_22): track 217.5 -> 208.8 mm, vias 1 -> 0
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Other:
- board text added: "Grid Size for Placement - 4.7625 Upper Left corner with {dblquote}S{dblquote}"
- board text added: "Клавиатура БПК {dblquote}Дельта-С{dblquote} / Delta-S Keyboard (PCB) Revision 2 Board Design by MadCat, 2023 https://github.com/madcatse/Delta-S-M t.me/zx_delta_s https://www.youtube.com/@MadCatSE"
- board text removed: "Клавиатура БПК {dblquote}Дельта-С{dblquote} / Delta-S Keyboard (PCB) Version 0.1 Board Design by MadCat, 2023 https://github.com/madcatse/Delta-S-M t.me/zx_delta_s https://www.youtube.com/@MadCatSE"

Commit message: 3d design for ver2 final
Parts:
- moved H8 3.30 mm to (289.5, 110.0)
Changed lines of the file:
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@@
   )
   (footprint "MountingHole:MountingHole_3.2mm_M3" (layer "F.Cu")
-    (at 289.4933 113.2591)
+    (at 289.4933 109.9602)
     (descr "Mounting Hole 3.2mm, no annular, M3")
     (tags "mounting hole 3.2mm no annular m3")
