File: keyboard_cherry/keyboard_cherry_panel.kicad_pcb (KiCad board)
At the start: 2 copper layers, 293.1 x 115.4 mm, 6 parts

Commit message: Keyboard gerbers and 3d modelling of top case
Parts:
- added H7: MountingHole_3.2mm_M3, MountingHole:MountingHole_3.2mm_M3, F.Cu at (186.6, 113.3)
- added H8: MountingHole_3.2mm_M3, MountingHole:MountingHole_3.2mm_M3, F.Cu at (289.5, 110.0)
- moved H6 181.9 mm to (106.6, 113.3)
- moved H4 145.7 mm to (289.5, 13.5)
- moved H3 102.1 mm to (186.6, 8.70)
- moved H2 23.8 mm to (106.6, 8.70)
- moved H5 4.97 mm to (3.44, 110.0)
- moved H1 4.29 mm to (3.44, 13.5)
- renumbered H4 to H5
Other:
- board size 293.1 x 115.4 mm -> 293.1 x 117 mm

Commit message: Cleanup
Other:
- outline, holes or cut-outs redrawn
- board text added: "Клавиатура БПК {dblquote}Дельта-С{dblquote} / Delta-S Keyboard (Panel) Revision 2 Board Design by MadCat, 2023 https://github.com/madcatse/Delta-S-M t.me/zx_delta_s https://www.youtube.com/@MadCatSE"
- board text removed: "Клавиатура БПК {dblquote}Дельта-С{dblquote} / Delta-S Keyboard (Panel) Version 0.1 Board Design by MadCat, 2023 https://github.com/madcatse/Delta-S-M t.me/zx_delta_s https://www.youtube.com/@MadCatSE"
